File: CLK.sch (KiCad schematic (older format))
At the start: 5 parts, among them SW2 SW_DPST_x2, U8 8284, Y1 Crystal

Commit message: Some minor changes
Connections:
- net labels added: +5V
- net labels removed: VCC
- wire segments 24 -> 27
Changed lines of the file:
@@
 $EndComp
 $Comp
-L power:VCC #PWR0117
-U 1 1 60793A2C
-P 5650 2450
-F 0 "#PWR0117" H 5650 2300 50  0001 C CNN
-F 1 "VCC" H 5665 2623 50  0000 C CNN
-F 2 "" H 5650 2450 50  0001 C CNN
-F 3 "" H 5650 2450 50  0001 C CNN
-	1    5650 2450
+L power:+5V #PWR0117
+U 1 1 6078E239
+P 5350 2200
+F 0 "#PWR0117" H 5350 2050 50  0001 C CNN
+F 1 "+5V" H 5365 2373 50  0000 C CNN
+F 2 "" H 5350 2200 50  0001 C CNN
+F 3 "" H 5350 2200 50  0001 C CNN
+	1    5350 2200
 	1    0    0    -1
 $EndComp
+Wire Wire Line
+	5350 2200 5450 2200
+Wire Wire Line
+	5450 2200 5450 2450
+Wire Wire Line
+	5450 2450 5650 2450
+Connection ~ 5350 2200
 $EndSCHEMATC

Commit message: Add files via upload
Updated Hierarchical labels
Connections:
- net labels added: PCLK, READY
- wire segments 27 -> 29
- no-connect marks 9 -> 7
Changed lines of the file:
@@
 NoConn ~ 4950 3950
 NoConn ~ 6350 3450
-NoConn ~ 6350 3350
-NoConn ~ 6350 2950
 $Comp
 L power:GND #PWR0116
@@
 	5450 2450 5650 2450
 Connection ~ 5350 2200
+Wire Wire Line
+	6350 2950 6700 2950
+Text HLabel 6700 2950 2    50   Output ~ 0
+READY
+Wire Wire Line
+	6350 3350 6650 3350
+Text HLabel 6650 3350 2    50   Output ~ 0
+PCLK
 $EndSCHEMATC
