File: 8259Layout.sch (KiCad schematic (older format))
At the start: 4 parts

Commit message: Add files via upload
Connections:
- net labels added: A[2:15], D[0:7]
- net labels removed: AD[0:7], A[12:15], A[2:11]
Changed lines of the file:
@@
 8259INT_Out
 Text HLabel 6300 3000 0    50   BiDi ~ 0
-AD[0:7]
+D[0:7]
 Wire Wire Line
 	7050 3150 6850 3150
@@
 Entry Wire Line
 	3050 4050 3150 3950
-Wire Bus Line
-	3050 4050 2850 4050
-Text HLabel 2850 4050 0    50   Input ~ 0
-A[2:11]
 Entry Wire Line
 	5200 3500 5300 3600
@@
 	5200 3200 5300 3300
 NoConn ~ 4850 3700
-Text HLabel 5300 3850 2    50   Input ~ 0
-A[12:15]
 Wire Wire Line
 	5200 3500 4850 3500
@@
 	5200 3200 4850 3200
 NoConn ~ 4850 3100
-Wire Bus Line
-	5300 3200 5300 3850
-Wire Bus Line
-	6600 2150 6600 3000
-Wire Bus Line
-	3050 2700 3050 4050
 Text HLabel 4850 3600 2    50   Input ~ 0
 IO\~M
@@
 Text Label 3400 3950 0    50   ~ 0
 A11
+Entry Bus Bus
+	5300 4400 5200 4500
+Entry Bus Bus
+	3050 4400 3150 4500
+Text HLabel 4250 4500 3    50   Input ~ 0
+A[2:15]
+Wire Bus Line
+	3150 4500 5200 4500
+Wire Bus Line
+	3050 2700 3050 4400
+Wire Bus Line
+	5300 3200 5300 4400
+Wire Bus Line
+	6600 2150 6600 3000
 $EndSCHEMATC

Commit message: Add files via upload
Parts:
- removed R?: R, symbol Device:R
Connections:
- wire segments 52 -> 51
Changed lines of the file:
@@
 	0    1    1    0
 $EndComp
-$Comp
-L Device:R R?
-U 1 1 6078C718
-P 8500 3550
-F 0 "R?" V 8293 3550 50  0000 C CNN
-F 1 "R" V 8384 3550 50  0000 C CNN
-F 2 "" V 8430 3550 50  0001 C CNN
-F 3 "~" H 8500 3550 50  0001 C CNN
-	1    8500 3550
-	0    1    1    0
-$EndComp
-Wire Wire Line
-	8250 3550 8350 3550
-Wire Wire Line
-	8650 3550 8800 3550
 NoConn ~ 8250 3150
 NoConn ~ 8250 3250
@@
 Wire Bus Line
 	3150 4500 5200 4500
+Wire Wire Line
+	8250 3550 8800 3550
 Wire Bus Line
 	3050 2700 3050 4400
