File: Display.sch (KiCad schematic (older format))
At the start: 25 parts, among them U31 PAL16L8, U32 PAL16L8, U33 74LS374, U34 74LS374, U35 74LS374, U36 MAN71A, U37 MAN71A

Commit message: annotations
Parts:
- renumbered U33 to Display1, U34 to Display2, U35 to Display3, U31 to Display_Decode1, U32 to Display_Decode2, U36 to Seven_Seg1, U37 to Seven_Seg2
Connections:
- wire segments 141 -> 161
Other:
- moved on the sheet: R5
Changed lines of the file:
@@
 $EndDescr
 $Comp
-L 74xx:74LS374 U33
+L 74xx:74LS374 Display1
 U 1 1 607791B4
 P 7500 1450
-F 0 "U33" H 7500 2431 50  0000 C CNN
+F 0 "Display1" H 7500 2431 50  0000 C CNN
 F 1 "74LS374" H 7500 2340 50  0000 C CNN
 F 2 "" H 7500 1450 50  0001 C CNN
@@
 $EndComp
 $Comp
-L 74xx:74LS374 U34
+L 74xx:74LS374 Display2
 U 1 1 60775947
 P 7550 3500
-F 0 "U34" H 7550 4481 50  0000 C CNN
+F 0 "Display2" H 7550 4481 50  0000 C CNN
 F 1 "74LS374" H 7550 4390 50  0000 C CNN
 F 2 "" H 7550 3500 50  0001 C CNN
@@
 $EndComp
 $Comp
-L 74xx:74LS374 U35
+L 74xx:74LS374 Display3
 U 1 1 60778C07
 P 7600 5500
-F 0 "U35" H 7600 6481 50  0000 C CNN
+F 0 "Display3" H 7600 6481 50  0000 C CNN
 F 1 "74LS374" H 7600 6390 50  0000 C CNN
 F 2 "" H 7600 5500 50  0001 C CNN
@@
 Wire Wire Line
 	7100 5100 6900 5100
-$Comp
-L power:VCC #PWR057
-U 1 1 6079D8CA
-P 6850 2700
-F 0 "#PWR057" H 6850 2550 50  0001 C CNN
-F 1 "VCC" V 6865 2827 50  0000 L CNN
-F 2 "" H 6850 2700 50  0001 C CNN
-F 3 "" H 6850 2700 50  0001 C CNN
-	1    6850 2700
-	1    0    0    -1
-$EndComp
-$Comp
-L power:GND #PWR058
-U 1 1 607A1D53
-P 7600 6400
-F 0 "#PWR058" H 7600 6150 50  0001 C CNN
-F 1 "GND" H 7605 6227 50  0000 C CNN
-F 2 "" H 7600 6400 50  0001 C CNN
-F 3 "" H 7600 6400 50  0001 C CNN
-	1    7600 6400
-	1    0    0    -1
-$EndComp
 Wire Wire Line
 	7000 1950 7000 2250
@@
 	7050 4350 7550 4350
 $Comp
-L Display_Character:MAN71A U36
+L Display_Character:MAN71A Seven_Seg1
 U 1 1 6078B9DF
 P 9550 1350
-F 0 "U36" H 9550 2017 50  0000 C CNN
+F 0 "Seven_Seg1" H 9550 2017 50  0000 C CNN
 F 1 "MAN71A" H 9550 1926 50  0000 C CNN
 F 2 "Display_7Segment:MAN71A" H 9050 650 50  0001 L CNN
@@
 $EndComp
 $Comp
-L Display_Character:MAN71A U37
+L Display_Character:MAN71A Seven_Seg2
 U 1 1 6079109D
-P 9550 3500
-F 0 "U37" H 9550 4167 50  0000 C CNN
-F 1 "MAN71A" H 9550 4076 50  0000 C CNN
-F 2 "Display_7Segment:MAN71A" H 9050 2800 50  0001 L CNN
-F 3 "https://www.digchip.com/datasheets/parts/datasheet/161/MAN3640A-pdf.php" H 9560 3840 50  0001 L CNN
-	1    9550 3500
+P 9550 3400
+F 0 "Seven_Seg2" H 9550 4067 50  0000 C CNN
+F 1 "MAN71A" H 9550 3976 50  0000 C CNN
+F 2 "Display_7Segment:MAN71A" H 9050 2700 50  0001 L CNN
+F 3 "https://www.digchip.com/datasheets/parts/datasheet/161/MAN3640A-pdf.php" H 9560 3740 50  0001 L CNN
+	1    9550 3400
 	1    0    0    -1
 $EndComp
@@
 	5650 1850 7000 1850
 Wire Wire Line
-	3300 800  2900 800
-Wire Wire Line
-	2900 800  2900 750
+	3300 800  3100 800
 $Comp
 L power:VCC #PWR054
 U 1 1 607ECC89
-P 2900 750
-F 0 "#PWR054" H 2900 600 50  0001 C CNN
-F 1 "VCC" H 2915 923 50  0000 C CNN
-F 2 "" H 2900 750 50  0001 C CNN
-F 3 "" H 2900 750 50  0001 C CNN
-	1    2900 750
-	1    0    0    -1
-$EndComp
-$Comp
-L power:GND #PWR055
-U 1 1 607EDAEB
-P 3300 2150
-F 0 "#PWR055" H 3300 1900 50  0001 C CNN
-F 1 "GND" H 3305 1977 50  0000 C CNN
-F 2 "" H 3300 2150 50  0001 C CNN
-F 3 "" H 3300 2150 50  0001 C CNN
-	1    3300 2150
-	1    0    0    -1
+P 2900 600
+F 0 "#PWR054" H 2900 450 50  0001 C CNN
+F 1 "VCC" H 2915 773 50  0000 C CNN
+F 2 "" H 2900 600 50  0001 C CNN
+F 3 "" H 2900 600 50  0001 C CNN
+	1    2900 600
+	0    -1   -1   0
 $EndComp
 Wire Wire Line
 	2800 1100 2550 1100
 $Comp
-L Logic_Programmable:PAL16L8 U32
+L Logic_Programmable:PAL16L8 Display_Decode2
 U 1 1 607F2271
 P 3300 3350
-F 0 "U32" H 3300 4231 50  0000 C CNN
+F 0 "Display_Decode2" H 3300 4231 50  0000 C CNN
 F 1 "PAL16L8" H 3300 4140 50  0000 C CNN
 F 2 "" H 3300 3350 50  0001 C CNN
@@
 	2150 800  2900 800
 Connection ~ 2900 800
-Wire Wire Line
-	3300 2100 3300 2150
-Wire Wire Line
-	3300 3950 3300 4050
 $Comp
 L power:GND #PWR056
 U 1 1 607FE1E1
-P 3300 4050
-F 0 "#PWR056" H 3300 3800 50  0001 C CNN
-F 1 "GND" H 3305 3877 50  0000 C CNN
-F 2 "" H 3300 4050 50  0001 C CNN
-F 3 "" H 3300 4050 50  0001 C CNN
-	1    3300 4050
+P 3300 5150
+F 0 "#PWR056" H 3300 4900 50  0001 C CNN
+F 1 "GND" H 3305 4977 50  0000 C CNN
+F 2 "" H 3300 5150 50  0001 C CNN
+F 3 "" H 3300 5150 50  0001 C CNN
+	1    3300 5150
 	1    0    0    -1
 $EndComp
@@
 	2800 2950 2550 2950
 $Comp
-L Logic_Programmable:PAL16L8 U31
+L Logic_Programmable:PAL16L8 Display_Decode1
 U 1 1 607E2663
 P 3300 1500
-F 0 "U31" H 3300 2381 50  0000 C CNN
+F 0 "Display_Decode1" H 3300 2381 50  0000 C CNN
 F 1 "PAL16L8" H 3300 2290 50  0000 C CNN
 F 2 "" H 3300 1500 50  0001 C CNN
@@
 	10000 1650 10000 1550
 Wire Wire Line
-	9850 3800 10000 3800
-Wire Wire Line
-	10000 3800 10000 3650
+	9850 3700 10000 3700
+Wire Wire Line
+	10000 3700 10000 3550
 $Comp
 L Device:R R4
@@
 L Device:R R5
 U 1 1 607D65C2
-P 10000 3500
-F 0 "R5" H 10070 3546 50  0000 L CNN
-F 1 "R" H 10070 3455 50  0000 L CNN
-F 2 "" V 9930 3500 50  0001 C CNN
-F 3 "~" H 10000 3500 50  0001 C CNN
-	1    10000 3500
+P 10000 3400
+F 0 "R5" H 10070 3446 50  0000 L CNN
+F 1 "R" H 10070 3355 50  0000 L CNN
+F 2 "" V 9930 3400 50  0001 C CNN
+F 3 "~" H 10000 3400 50  0001 C CNN
+	1    10000 3400
 	1    0    0    -1
 $EndComp
@@
 	10000 1250 10000 1150
 Wire Wire Line
-	10000 3350 10000 3200
+	10000 3350 10000 3250
 $Comp
 L power:VCC #PWR059
@@
 NoConn ~ 3800 3550
 NoConn ~ 9850 1750
-NoConn ~ 9850 3900
 Wire Wire Line
 	5450 2950 5450 5900
@@
 	7550 4350 7550 4300
 Connection ~ 7550 4350
-$Comp
-L power:GND #PWR0101
-U 1 1 60A72376
-P 7550 4400
-F 0 "#PWR0101" H 7550 4150 50  0001 C CNN
-F 1 "GND" H 7555 4227 50  0000 C CNN
-F 2 "" H 7550 4400 50  0001 C CNN
-F 3 "" H 7550 4400 50  0001 C CNN
-	1    7550 4400
-	1    0    0    -1
-$EndComp
-$Comp
-L power:GND #PWR0102
-U 1 1 60A729AF
-P 7500 2350
-F 0 "#PWR0102" H 7500 2100 50  0001 C CNN
-F 1 "GND" H 7505 2177 50  0000 C CNN
-F 2 "" H 7500 2350 50  0001 C CNN
-F 3 "" H 7500 2350 50  0001 C CNN
-	1    7500 2350
-	1    0    0    -1
-$EndComp
-Wire Wire Line
-	7450 650  6500 650
-Wire Wire Line
-	7550 2700 6850 2700
-Wire Wire Line
-	7600 4700 6600 4700
-$Comp
-L power:VCC #PWR0103
-U 1 1 60A94EE1
-P 6600 4700
-F 0 "#PWR0103" H 6600 4550 50  0001 C CNN
-F 1 "VCC" H 6615 4873 50  0000 C CNN
-F 2 "" H 6600 4700 50  0001 C CNN
-F 3 "" H 6600 4700 50  0001 C CNN
-	1    6600 4700
-	1    0    0    -1
-$EndComp
-$Comp
-L power:VCC #PWR0104
-U 1 1 60A9BDC3
-P 6500 650
-F 0 "#PWR0104" H 6500 500 50  0001 C CNN
-F 1 "VCC" V 6515 777 50  0000 L CNN
-F 2 "" H 6500 650 50  0001 C CNN
-F 3 "" H 6500 650 50  0001 C CNN
-	1    6500 650
-	-1   0    0    1
-$EndComp
+Wire Wire Line
+	3300 3950 3300 4250
+Wire Wire Line
+	3300 2100 1900 2100
+Wire Wire Line
+	1900 2100 1900 4350
+Wire Wire Line
+	1900 4350 3300 4350
+Connection ~ 3300 4350
+Wire Wire Line
+	3300 4350 3300 4400
+Wire Wire Line
+	2900 600  2900 800
+Wire Wire Line
+	3100 650  3100 800
+Connection ~ 3100 800
+Wire Wire Line
+	3100 800  2900 800
+Wire Wire Line
+	3100 650  5950 650
+Wire Wire Line
+	7600 6400 3950 6400
+Wire Wire Line
+	3950 6400 3950 4500
+Wire Wire Line
+	3950 4500 3300 4500
+Connection ~ 3300 4500
+Wire Wire Line
+	7550 4400 3300 4400
+Connection ~ 3300 4400
+Wire Wire Line
+	3300 4400 3300 4500
+Wire Wire Line
+	7500 2350 4250 2350
+Wire Wire Line
+	4250 2350 4250 4250
+Wire Wire Line
+	4250 4250 3300 4250
+Connection ~ 3300 4250
+Wire Wire Line
+	3300 4250 3300 4350
+Wire Wire Line
+	3300 4500 3300 5150
+Wire Wire Line
+	6150 2700 6150 650
+Wire Wire Line
+	6150 2700 7550 2700
+Connection ~ 6150 650
+Wire Wire Line
+	6150 650  7500 650
+Wire Wire Line
+	5950 4700 5950 650
+Wire Wire Line
+	5950 4700 7600 4700
+Connection ~ 5950 650
+Wire Wire Line
+	5950 650  6150 650
+Connection ~ 10000 3250
+Wire Wire Line
+	10000 3250 10000 3200
+NoConn ~ 9850 3800
 $EndSCHEMATC
