File: 8259_updated.sch (KiCad schematic (older format))
At the start: 4 parts, among them SW3 SW_Push, U24 PAL16L8, U25 8259

Commit message: Add files via upload
Parts:
- removed R3: R, symbol Device:R
- renumbered U25 to 8259INTR, U24 to 8259Selector
Connections:
- net labels added: VCC
- wire segments 30 -> 29
Changed lines of the file:
@@
 $EndDescr
 $Comp
-L Interface:8259 U25
+L Interface:8259 8259INTR
 U 1 1 6078126B
 P 7650 3050
-F 0 "U25" H 7650 4331 50  0000 C CNN
+F 0 "8259INTR" H 7650 4331 50  0000 C CNN
 F 1 "8259" H 7650 4240 50  0000 C CNN
 F 2 "Package_DIP:DIP-28_W15.24mm" H 7650 3050 50  0001 C CIN
@@
 NoConn ~ 8250 2350
 NoConn ~ 8250 2250
-$Comp
-L power:+5V #PWR040
-U 1 1 6078B521
-P 8800 3550
-F 0 "#PWR040" H 8800 3400 50  0001 C CNN
-F 1 "+5V" V 8815 3678 50  0000 L CNN
-F 2 "" H 8800 3550 50  0001 C CNN
-F 3 "" H 8800 3550 50  0001 C CNN
-	1    8800 3550
-	0    1    1    0
-$EndComp
-$Comp
-L Device:R R3
-U 1 1 6078C718
-P 8500 3550
-F 0 "R3" V 8293 3550 50  0000 C CNN
-F 1 "R" V 8384 3550 50  0000 C CNN
-F 2 "" V 8430 3550 50  0001 C CNN
-F 3 "~" H 8500 3550 50  0001 C CNN
-	1    8500 3550
-	0    1    1    0
-$EndComp
 Wire Wire Line
 	8250 3550 8350 3550
-Wire Wire Line
-	8650 3550 8800 3550
 NoConn ~ 8250 3150
 NoConn ~ 8250 3250
@@
 	6850 3850 7050 3850
 $Comp
-L Logic_Programmable:PAL16L8 U24
+L Logic_Programmable:PAL16L8 8259Selector
 U 1 1 60799BF8
 P 4350 3500
-F 0 "U24" H 4350 4381 50  0000 C CNN
+F 0 "8259Selector" H 4350 4381 50  0000 C CNN
 F 1 "PAL16L8" H 4350 4290 50  0000 C CNN
 F 2 "" H 4350 3500 50  0001 C CNN
@@
 Text HLabel 7050 2950 0    50   Input ~ 0
 D7
+$Comp
+L power:VCC #PWR?
+U 1 1 6090AF2E
+P 8350 3550
+F 0 "#PWR?" H 8350 3400 50  0001 C CNN
+F 1 "VCC" V 8365 3678 50  0000 L CNN
+F 2 "" H 8350 3550 50  0001 C CNN
+F 3 "" H 8350 3550 50  0001 C CNN
+	1    8350 3550
+	0    1    1    0
+$EndComp
 $EndSCHEMATC
