File: 8279_updated.sch (KiCad schematic (older format))
At the start: 24 parts, among them SW10 SW_Push, SW11 SW_Push, SW12 SW_Push, SW13 SW_Push, SW14 SW_Push, SW15 SW_Push, SW16 SW_Push, SW17 SW_Push, SW18 SW_Push, SW19 SW_Push, SW20 SW_Push, SW21 SW_Push, SW22 SW_Push, SW23 SW_Push, SW24 SW_Push, SW25 SW_Push, SW4 SW_Push, SW5 SW_Push, SW6 SW_Push, SW7 SW_Push, SW8 SW_Push, SW9 SW_Push, U28 pkd8279, U29 PAL16L8

Commit message: Add files via upload
Parts:
- renumbered U28 to 8279Keyboard, U29 to KeyboardSelector
Changed lines of the file:
@@
 $EndDescr
 $Comp
-L pkd8279:pkd8279 U28
+L pkd8279:pkd8279 8279Keyboard
 U 1 1 60761D14
 P 1850 3300
-F 0 "U28" H 2875 3687 60  0000 C CNN
+F 0 "8279Keyboard" H 2875 3687 60  0000 C CNN
 F 1 "pkd8279" H 2875 3581 60  0000 C CNN
 F 2 "pkd8279" H 2850 3690 60  0001 C CNN
@@
 8086_A1
 $Comp
-L Logic_Programmable:PAL16L8 U29
+L Logic_Programmable:PAL16L8 KeyboardSelector
 U 1 1 607FB29D
 P 4900 6200
-F 0 "U29" H 4900 7081 50  0000 C CNN
+F 0 "KeyboardSelector" H 4900 7081 50  0000 C CNN
 F 1 "PAL16L8" H 4900 6990 50  0000 C CNN
 F 2 "" H 4900 6200 50  0001 C CNN
