File: SRAM.sch (KiCad schematic (older format))
At the start: 12 parts

Commit message: Add files via upload
Parts:
- removed U? (x2): CY7C199, symbol Memory_RAM:CY7C199
- removed U? (x2): 74LVC1GU04DRL, Package_TO_SOT_SMD:SOT-553, symbol 74xGxx:74LVC1GU04DRL
- added SRAMSelector: PAL16L8, symbol Logic_Programmable:PAL16L8
- added U17, U18: 74LS04, symbol 74xx:74LS04
- gave numbers to parts that had none: 8
Connections:
- net labels added: D10, D11, D12, D13, D14, D15, D8, D9
- net labels removed: A[0:14], A[0:19], A[15:19], D[0:7], D[8:15]
- wire segments 120 -> 108
Other:
- moved on the sheet: U16

Commit message: Add files via upload
Parts:
- removed U16: 74LS138, symbol 74xx:74LS138
- added U?: 74AHC1G08, symbol 74xGxx:74AHC1G08
Connections:
- net labels added: ~BHE
- net labels removed: A15, A16, A17, A18, A19
- wire segments 108 -> 117
- no-connect marks 6 -> 4
Other:
- moved on the sheet: U17A, U18A
Changed lines of the file:
@@
 	0    1    1    0
-$EndComp
-$Comp
-L power:VCC #PWR030
-U 1 1 6128184B
-P 13750 2950
-F 0 "#PWR030" H 13750 2800 50  0001 C CNN
-F 1 "VCC" V 13765 3078 50  0000 L CNN
-F 2 "" H 13750 2950 50  0001 C CNN
-F 3 "" H 13750 2950 50  0001 C CNN
-	1    13750 2950
-	0    1    1    0
-$EndComp
-$Comp
-L power:GND #PWR031
-U 1 1 61282FEE
-P 13750 4250
-F 0 "#PWR031" H 13750 4000 50  0001 C CNN
-F 1 "GND" H 13755 4077 50  0000 C CNN
-F 2 "" H 13750 4250 50  0001 C CNN
-F 3 "" H 13750 4250 50  0001 C CNN
-	1    13750 4250
-	1    0    0    -1
 $EndComp
 Text Notes 3100 6300 0    50   ~ 0
@@
 Text Label 4200 5400 0    50   ~ 0
 CE10
-Text Notes 13200 2650 0    50   ~ 0
+Text Notes 7800 3200 0    50   ~ 0
 CE ; lsb ; msb\nChipEnable ; left = 0, right = 1; low = 0, high = 1
 $Comp
 L 74xGxx:74AHC1G08 U19
 U 1 1 613019A2
-P 15300 3300
-F 0 "U19" H 15275 3567 50  0000 C CNN
-F 1 "74AHC1G08" H 15275 3476 50  0000 C CNN
-F 2 "" H 15300 3300 50  0001 C CNN
-F 3 "http://www.ti.com/lit/sg/scyt129e/scyt129e.pdf" H 15300 3300 50  0001 C CNN
-	1    15300 3300
+P 9900 3850
+F 0 "U19" H 9875 4117 50  0000 C CNN
+F 1 "74AHC1G08" H 9875 4026 50  0000 C CNN
+F 2 "" H 9900 3850 50  0001 C CNN
+F 3 "http://www.ti.com/lit/sg/scyt129e/scyt129e.pdf" H 9900 3850 50  0001 C CNN
+	1    9900 3850
 	1    0    0    -1
 $EndComp
@@
 L 74xGxx:74AHC1G08 U20
 U 1 1 61309321
-P 15300 4050
-F 0 "U20" H 15275 4317 50  0000 C CNN
-F 1 "74AHC1G08" H 15275 4226 50  0000 C CNN
-F 2 "" H 15300 4050 50  0001 C CNN
-F 3 "http://www.ti.com/lit/sg/scyt129e/scyt129e.pdf" H 15300 4050 50  0001 C CNN
-	1    15300 4050
+P 9900 4600
+F 0 "U20" H 9875 4867 50  0000 C CNN
+F 1 "74AHC1G08" H 9875 4776 50  0000 C CNN
+F 2 "" H 9900 4600 50  0001 C CNN
+F 3 "http://www.ti.com/lit/sg/scyt129e/scyt129e.pdf" H 9900 4600 50  0001 C CNN
+	1    9900 4600
 	1    0    0    -1
 $EndComp
@@
 L 74xGxx:74AHC1G08 U21
 U 1 1 613108D7
-P 15300 4800
-F 0 "U21" H 15275 5067 50  0000 C CNN
-F 1 "74AHC1G08" H 15275 4976 50  0000 C CNN
-F 2 "" H 15300 4800 50  0001 C CNN
-F 3 "http://www.ti.com/lit/sg/scyt129e/scyt129e.pdf" H 15300 4800 50  0001 C CNN
-	1    15300 4800
-	1    0    0    -1
-$EndComp
-NoConn ~ 14250 3450
-NoConn ~ 14250 3550
-NoConn ~ 14250 3650
-NoConn ~ 14250 3750
-NoConn ~ 14250 3850
-NoConn ~ 14250 3950
-Wire Wire Line
-	14250 3250 14550 3250
-Wire Wire Line
-	14250 3350 14350 3350
-Wire Wire Line
-	15550 3300 15900 3300
-Text Label 15900 3300 0    50   ~ 0
+P 9900 5350
+F 0 "U21" H 9875 5617 50  0000 C CNN
+F 1 "74AHC1G08" H 9875 5526 50  0000 C CNN
+F 2 "" H 9900 5350 50  0001 C CNN
+F 3 "http://www.ti.com/lit/sg/scyt129e/scyt129e.pdf" H 9900 5350 50  0001 C CNN
+	1    9900 5350
+	1    0    0    -1
+$EndComp
+Wire Wire Line
+	8850 3900 8950 3900
+Wire Wire Line
+	10150 3850 10500 3850
+Text Label 10500 3850 0    50   ~ 0
 CE11
 Wire Wire Line
-	15550 4050 15900 4050
-Text Label 15900 4050 0    50   ~ 0
+	10150 4600 10500 4600
+Text Label 10500 4600 0    50   ~ 0
 CE10
-Text Label 15900 4800 0    50   ~ 0
+Text Label 10500 5350 0    50   ~ 0
 CE01
 Wire Wire Line
-	15550 4800 15900 4800
-Wire Wire Line
-	14550 3250 14550 4000
-Connection ~ 14550 3250
-Wire Wire Line
-	14550 3250 15000 3250
-Wire Wire Line
-	14850 3850 14850 3950
-Wire Wire Line
-	14350 4850 15000 4850
-Connection ~ 14350 3350
-Wire Wire Line
-	14700 4750 15000 4750
+	10150 5350 10500 5350
+Wire Wire Line
+	9150 3800 9150 4550
+Connection ~ 9150 3800
+Wire Wire Line
+	9150 3800 9600 3800
+Wire Wire Line
+	9450 4400 9450 4500
+Wire Wire Line
+	8950 5400 9600 5400
+Connection ~ 8950 3900
+Wire Wire Line
+	9300 5300 9600 5300
 Text HLabel 9650 2200 0    50   Input ~ 0
 ~RD
@@
 L 74xx:74LS04 U18
 U 1 1 619E8FEB
-P 14850 3650
-F 0 "U18" V 14804 3830 50  0000 L CNN
-F 1 "74LS04" V 14895 3830 50  0000 L CNN
-F 2 "" H 14850 3650 50  0001 C CNN
-F 3 "http://www.ti.com/lit/gpn/sn74LS04" H 14850 3650 50  0001 C CNN
-	1    14850 3650
+P 9450 4200
+F 0 "U18" V 9404 4380 50  0000 L CNN
+F 1 "74LS04" V 9495 4380 50  0000 L CNN
+F 2 "" H 9450 4200 50  0001 C CNN
+F 3 "http://www.ti.com/lit/gpn/sn74LS04" H 9450 4200 50  0001 C CNN
+	1    9450 4200
 	0    1    1    0
 $EndComp
 Wire Wire Line
-	14350 3350 14850 3350
-Connection ~ 14850 3350
-Wire Wire Line
-	14850 3350 15000 3350
-Wire Wire Line
-	15000 4100 14850 4100
-Wire Wire Line
-	14850 4100 14850 3950
-Connection ~ 14850 3950
-Wire Wire Line
-	14550 4000 14700 4000
+	8950 3900 9450 3900
+Connection ~ 9450 3900
+Wire Wire Line
+	9450 3900 9600 3900
+Wire Wire Line
+	9600 4650 9450 4650
+Wire Wire Line
+	9450 4650 9450 4500
+Connection ~ 9450 4500
+Wire Wire Line
+	9150 4550 9300 4550
 $Comp
 L 74xx:74LS04 U17
 U 1 1 619F3CB3
-P 14700 4300
-F 0 "U17" V 14654 4480 50  0000 L CNN
-F 1 "74LS04" V 14745 4480 50  0000 L CNN
-F 2 "" H 14700 4300 50  0001 C CNN
-F 3 "http://www.ti.com/lit/gpn/sn74LS04" H 14700 4300 50  0001 C CNN
-	1    14700 4300
+P 9300 4850
+F 0 "U17" V 9254 5030 50  0000 L CNN
+F 1 "74LS04" V 9345 5030 50  0000 L CNN
+F 2 "" H 9300 4850 50  0001 C CNN
+F 3 "http://www.ti.com/lit/gpn/sn74LS04" H 9300 4850 50  0001 C CNN
+	1    9300 4850
 	0    1    1    0
 $EndComp
 Wire Wire Line
-	14700 4750 14700 4600
-Wire Wire Line
-	14350 3350 14350 4850
-$Comp
-L power:GND #PWR0132
-U 1 1 61A0948D
-P 13250 3750
-F 0 "#PWR0132" H 13250 3500 50  0001 C CNN
-F 1 "GND" V 13255 3622 50  0000 R CNN
-F 2 "" H 13250 3750 50  0001 C CNN
-F 3 "" H 13250 3750 50  0001 C CNN
-	1    13250 3750
-	0    1    1    0
-$EndComp
-Text HLabel 13250 3950 0    50   Input ~ 0
-A19
-Text HLabel 13250 3850 0    50   Input ~ 0
-A18
-Text HLabel 13250 3450 0    50   Input ~ 0
-A17
-Text HLabel 13250 3350 0    50   Input ~ 0
-A16
-Text HLabel 13250 3250 0    50   Input ~ 0
-A15
-$Comp
-L 74xx:74LS138 U16
-U 1 1 608F8DF6
-P 13750 3550
-F 0 "U16" H 13750 4331 50  0000 C CNN
-F 1 "74LS138" H 13750 4240 50  0000 C CNN
-F 2 "" H 13750 3550 50  0001 C CNN
-F 3 "http://www.ti.com/lit/gpn/sn74LS138" H 13750 3550 50  0001 C CNN
-	1    13750 3550
-	1    0    0    -1
-$EndComp
-Connection ~ 14700 4000
-Wire Wire Line
-	14700 4000 15000 4000
+	9300 5300 9300 5150
+Wire Wire Line
+	8950 3900 8950 5400
+Connection ~ 9300 4550
+Wire Wire Line
+	9300 4550 9600 4550
 $Comp
 L Logic_Programmable:PAL16L8 SRAMSelector
@@
 	1    0    0    -1
 $EndComp
+$Comp
+L power:GND #PWR?
+U 1 1 6090F38D
+P 7650 5200
+F 0 "#PWR?" H 7650 4950 50  0001 C CNN
+F 1 "GND" H 7655 5027 50  0000 C CNN
+F 2 "" H 7650 5200 50  0001 C CNN
+F 3 "" H 7650 5200 50  0001 C CNN
+	1    7650 5200
+	1    0    0    -1
+$EndComp
+$Comp
+L power:VCC #PWR?
+U 1 1 6090FE1F
+P 7650 3900
+F 0 "#PWR?" H 7650 3750 50  0001 C CNN
+F 1 "VCC" V 7665 4028 50  0000 L CNN
+F 2 "" H 7650 3900 50  0001 C CNN
+F 3 "" H 7650 3900 50  0001 C CNN
+	1    7650 3900
+	0    1    1    0
+$EndComp
+Text HLabel 7150 4100 0    50   Input ~ 0
+A1
+Text HLabel 7150 4200 0    50   Input ~ 0
+A2
+Text HLabel 7150 4300 0    50   Input ~ 0
+A3
+Text HLabel 7150 4400 0    50   Input ~ 0
+A4
+Text HLabel 7150 4500 0    50   Input ~ 0
+A5
+Text HLabel 7150 4600 0    50   Input ~ 0
+A6
+Text HLabel 7150 4700 0    50   Input ~ 0
+A7
+Text HLabel 7150 4800 0    50   Input ~ 0
+A8
+Text HLabel 7150 4900 0    50   Input ~ 0
+A9
+Text HLabel 7150 5000 0    50   Input ~ 0
+A10
+Text HLabel 8150 4300 2    50   Input ~ 0
+~BHE
+Text HLabel 8150 4400 2    50   Input ~ 0
+A0
+$Comp
+L 74xGxx:74AHC1G08 U?
+U 1 1 609251D1
+P 9900 5950
+F 0 "U?" H 9875 6217 50  0000 C CNN
+F 1 "74AHC1G08" H 9875 6126 50  0000 C CNN
+F 2 "" H 9900 5950 50  0001 C CNN
+F 3 "http://www.ti.com/lit/sg/scyt129e/scyt129e.pdf" H 9900 5950 50  0001 C CNN
+	1    9900 5950
+	1    0    0    -1
+$EndComp
+Wire Wire Line
+	9450 4650 9450 5900
+Wire Wire Line
+	9450 5900 9600 5900
+Connection ~ 9450 4650
+Wire Wire Line
+	9300 5300 9300 6000
+Wire Wire Line
+	9300 6000 9600 6000
+Connection ~ 9300 5300
+Wire Wire Line
+	10150 5950 10500 5950
+Text Label 10500 5950 0    50   ~ 0
+CE00
+Wire Wire Line
+	8150 4100 8400 4100
+Wire Wire Line
+	8400 4100 8400 3800
+Wire Wire Line
+	8400 3800 9150 3800
+Wire Wire Line
+	8150 4200 8850 4200
+Wire Wire Line
+	8850 4200 8850 3900
+NoConn ~ 8150 4500
+NoConn ~ 8150 4600
+NoConn ~ 8150 4700
+NoConn ~ 8150 4800
 $EndSCHEMATC
