File: 16550.sch (KiCad schematic (older format))
At the start: 1 part

Commit message: Add files via upload
Parts:
- added DSUB: DSUB-9, DSUB-9, symbol DSUB-9:DSUB-9
- added MAX235: max235cpg, max235cpg, symbol max235cpg:max235cpg
- added Resistor10K: Resistor, symbol Device:R
- added SIXTEENL8: PAL16L8, symbol Logic_Programmable:PAL16L8
- gave numbers to parts that had none: 1
Connections:
- net A0: now also SIXTEENL8.1 (I1)
- net A1: now also SIXTEENL8.2 (I2)
- net A2: now also SIXTEENL8.3 (I3)
- net GND1: no longer UART.14 (~CS2~)
- net SIN: now also MAX235.6 (R2OUT)
- net SOUT: now also MAX235.8 (T1IN)
- net VCC: now also MAX235.12 (VCC), Resistor10K.1, SIXTEENL8.20 (VCC); no longer UART.13 (CS1), UART.39 (~RI~)
- net CLK renamed PCLK
- net DDIS: no longer names the net of UART.23 (DDIS)
- net IO~M: no longer names the net of UART.12 (CS0)
- net IO~M: now also UART.13 (CS1), Resistor10K.2
- net XOUT: no longer names the net of UART.17 (XOUT)
- net ~OUT1: no longer names the net of UART.34 (~OUT1~)
- net ~OUT2: no longer names the net of UART.31 (~OUT2~)
- net ~RXRDY: no longer names the net of UART.29 (~RXRDY~)
- net ~TXRDY: no longer names the net of UART.24 (~TXRDY~)
- new net: SIXTEENL8.19 (IO1), UART.14 (~CS2~)
- new net A11: SIXTEENL8.18 (IO2)
- new net A12: SIXTEENL8.17 (I03)
- new net A13: SIXTEENL8.16 (IO4)
- new net A14: SIXTEENL8.15 (IO5)
- new net A15: SIXTEENL8.14 (IO6)
- new net A3: SIXTEENL8.4 (I4)
- new net A4: SIXTEENL8.5 (I5)
- new net A5: SIXTEENL8.6 (I6)
- new net A6: SIXTEENL8.7 (I7)
- new net A7: SIXTEENL8.8 (I8)
- new net A8: SIXTEENL8.9 (I9)
- new net A9: SIXTEENL8.11 (I10)
- new net CTR9: DSUB.8 (CTS), MAX235.18 (R4IN)
- new net CTS: MAX235.17 (R4OUT)
- new net DCD: MAX235.9 (R1OUT)
- new net DCD9: DSUB.1 (DCD), MAX235.10 (R1IN)
- new net DSR: MAX235.23 (R3OUT)
- new net DSR9: DSUB.6 (DSR), MAX235.24 (R3IN)
- new net DTR: MAX235.7 (T2IN)
- new net DTR9: DSUB.4 (DTR), MAX235.4 (T2OUT)
- new net GND: MAX235.11 (GND), MAX235.20 (*EN), MAX235.21 (SHDN), SIXTEENL8.10 (GND)
- new net RI: MAX235.14 (R5OUT), UART.39 (~RI~)
- new net RI9: DSUB.9 (RI), MAX235.13 (R5IN)
- new net RTS: MAX235.15 (T3IN)
- new net RTS9: DSUB.7 (RTS), MAX235.2 (T3OUT)
- new net RXD: DSUB.2 (RDX), MAX235.5 (R2IN)
- new net TXD: DSUB.3 (TDX), MAX235.3 (T1OUT)
- no-connect marks 0 -> 12

Commit message: Add files via upload
Connections:
- net ~CTS is gone; now on net CTS: UART.36 (~CTS~)
- net ~DCD is gone; now on net DCD: UART.38 (~DCD~)
- net ~DSR is gone; now on net DSR: UART.37 (~DSR~)
- net ~DTR is gone; now on net DTR: UART.33 (~DTR~)
- net ~RTS is gone; now on net RTS: UART.32 (~RTS~)
- net CTR9: no longer DSUB.8 (CTS)
- net CTS: now also DSUB.8 (CTS)
Changed lines of the file:
@@
 RI
 Text Label 6100 2550 0    50   ~ 0
-~DCD
+DCD
 Text Label 6100 2650 0    50   ~ 0
-~DSR
+DSR
 Text Label 6100 2750 0    50   ~ 0
-~CTS
+CTS
 Text Label 6100 3150 0    50   ~ 0
-~DTR
+DTR
 Text Label 6100 3250 0    50   ~ 0
-~RTS
+RTS
 Text Label 4950 5900 2    50   ~ 0
 DCD9
@@
 RTS9
 Text Label 4950 6600 2    50   ~ 0
-CTR9
+CTS
 Text Label 4950 6700 2    50   ~ 0
 RI9
