File: Final/8255(FINAL).sch (KiCad schematic (older format))
At the start: 0 parts

Commit message: New stuff
Parts:
- added J1: DB25_Female, symbol Connector:DB25_Female
- added U22: PAL16L8, symbol Logic_Programmable:PAL16L8
- added U23: 8255, Package_DIP:DIP-40_W15.24mm, symbol Interface:8255
Connections:
- new net: U22.12 (IO8), U23.6 (~CS~)
- new net A0: U22.1 (I1), U23.9 (A0)
- new net A1: U23.8 (A1)
- new net A10: U22.9 (I9)
- new net A11: U22.11 (I10)
- new net A3: U22.2 (I2)
- new net A4: U22.3 (I3)
- new net A5: U22.4 (I4)
- new net A6: U22.5 (I5)
- new net A7: U22.6 (I6)
- new net A8: U22.7 (I7)
- new net A9: U22.8 (I8)
- new net D0: U23.34 (D0)
- new net D1: U23.33 (D1)
- new net D2: U23.32 (D2)
- new net D3: U23.31 (D3)
- new net D4: U23.30 (D4)
- new net D5: U23.29 (D5)
- new net D6: U23.28 (D6)
- new net D7: U23.27 (D7)
- new net GND: U22.10 (GND), U23.7 (GND)
- new net IO~M: U22.13 (IO7)
- new net P0: J1.1, U23.4 (PA0)
- new net P1: J1.2, U23.3 (PA1)
- new net P10: J1.11, U23.20 (PB2)
- new net P11: J1.12, U23.21 (PB3)
- new net P12: J1.13, U23.22 (PB4)
- new net P13: J1.14 (P14), U23.23 (PB5)
- new net P14: J1.15 (P15), U23.24 (PB6)
- new net P15: J1.16 (P16), U23.25 (PB7)
- new net P16: J1.17 (P17), U23.14 (PC0)
- new net P17: J1.18 (P18), U23.15 (PC1)
- new net P18: J1.19 (P19), U23.16 (PC2)
- new net P19: J1.20 (P20), U23.17 (PC3)
- new net P2: J1.3, U23.2 (PA2)
- new net P20: J1.21 (P21), U23.13 (PC4)
- new net P21: J1.22 (P22), U23.12 (PC5)
- new net P22: J1.23 (P23), U23.11 (PC6)
- new net P23: J1.24 (P24), U23.10 (PC7)
- new net P24: J1.25 (P25)
- new net P3: J1.4, U23.1 (PA3)
- new net P4: J1.5, U23.40 (PA4)
- new net P5: J1.6, U23.39 (PA5)
- new net P6: J1.7, U23.38 (PA6)
- new net P7: J1.8, U23.37 (PA7)
- new net P8: J1.9, U23.18 (PB0)
- new net P9: J1.10, U23.19 (PB1)
- new net RESET: U23.35 (RESET)
- new net VCC: U22.20 (VCC), U23.26 (VCC)
- new net ~RD: U23.5 (~RD~)
- new net ~WR: U23.36 (~WR~)
- no-connect marks 0 -> 2
