File: Final/8255(FINAL).sch (KiCad schematic (older format))
At the start: 3 parts, among them J1 DB25_Female, U22 PAL16L8, U23 8255

Commit message: For Commenting
Parts:
- removed J1: DB25_Female, symbol Connector:DB25_Female
- added J1, J10, J11, J4, J5, J6, J7, J8, J9: Conn_01x08_Female, symbol Connector:Conn_01x08_Female
- added U42, U43: 8255, Package_DIP:DIP-40_W15.24mm, symbol Interface:8255
Connections:
- net A0: now also U42.9 (A0), U43.9 (A0); no longer U22.1 (I1)
- net A1: now also U42.8 (A1), U43.8 (A1)
- net A12: now also U22.13 (IO7)
- net A13: now also U22.14 (IO6)
- net A14: now also U22.15 (IO5)
- net A15: now also U22.16 (IO4)
- net D0: now also U42.34 (D0), U43.34 (D0)
- net D1: now also U42.33 (D1), U43.33 (D1)
- net D2: now also U42.32 (D2), U43.32 (D2)
- net D3: now also U42.31 (D3), U43.31 (D3)
- net D4: now also U42.30 (D4), U43.30 (D4)
- net D5: now also U42.29 (D5), U43.29 (D5)
- net D6: now also U42.28 (D6), U43.28 (D6)
- net D7: now also U42.27 (D7), U43.27 (D7)
- net GND: now also U42.7 (GND)
- net IO~M: now also U22.12 (IO8); no longer U22.13 (IO7)
- net P0: now also J6.1 (Pin_1)
- net P1: now also J6.2 (Pin_2)
- net P10: now also J7.3 (Pin_3)
- net P11: now also J7.4 (Pin_4)
- net P12: now also J7.5 (Pin_5)
- net P13: now also J7.6 (Pin_6)
- net P14: now also J7.7 (Pin_7)
- net P15: now also J7.8 (Pin_8)
- net P16: now also J8.1 (Pin_1)
- net P17: now also J8.2 (Pin_2)
- net P18: now also J8.3 (Pin_3)
- net P19: now also J8.4 (Pin_4)
- net P2: now also J6.3 (Pin_3)
- net P20: now also J8.5 (Pin_5)
- net P21: now also J8.6 (Pin_6)
- net P22: now also J8.7 (Pin_7)
- net P23: now also J8.8 (Pin_8)
- net P24: now also J9.1 (Pin_1), U43.4 (PA0)
- net P3: now also J6.4 (Pin_4)
- net P4: now also J6.5 (Pin_5)
- net P5: now also J6.6 (Pin_6)
- net P6: now also J6.7 (Pin_7)
- net P7: now also J6.8 (Pin_8)
- net P8: now also J7.1 (Pin_1)
- net P9: now also J7.2 (Pin_2)
- net RESET: now also U42.35 (RESET), U43.35 (RESET)
- net VCC: now also U42.26 (VCC), U43.26 (VCC)
- net ~RD: now also U42.5 (~RD~), U43.5 (~RD~)
- net ~WR: now also U42.36 (~WR~), U43.36 (~WR~)
- net at U23.6 (~CS~): now also U22.19 (IO1); no longer U22.12 (IO8)
- net at U22.17 (I03): now also U42.6 (~CS~)
- net at U22.18 (IO2): now also U43.6 (~CS~)
- new net A2: U22.1 (I1)
- new net P25: J9.2 (Pin_2), U43.3 (PA1)
- new net P26: J9.3 (Pin_3), U43.2 (PA2)
- new net P27: J9.4 (Pin_4), U43.1 (PA3)
- new net P28: J9.5 (Pin_5), U43.40 (PA4)
- new net P29: J9.6 (Pin_6), U43.39 (PA5)
- new net P30: J9.7 (Pin_7), U43.38 (PA6)
- new net P31: J9.8 (Pin_8), U43.37 (PA7)
- new net P32: J10.1 (Pin_1), U43.18 (PB0)
- new net P33: J10.2 (Pin_2), U43.19 (PB1)
- new net P34: J10.3 (Pin_3), U43.20 (PB2)
- new net P35: J10.4 (Pin_4), U43.21 (PB3)
- new net P36: J10.5 (Pin_5), U43.22 (PB4)
- new net P37: J10.6 (Pin_6), U43.23 (PB5)
- new net P38: J10.7 (Pin_7), U43.24 (PB6)
- new net P39: J10.8 (Pin_8), U43.25 (PB7)
- new net P40: J11.1 (Pin_1), U43.14 (PC0)
- new net P41: J11.2 (Pin_2), U43.15 (PC1)
- new net P42: J11.3 (Pin_3), U43.16 (PC2)
- new net P43: J11.4 (Pin_4), U43.17 (PC3)
- new net P44: J11.5 (Pin_5), U43.13 (PC4)
- new net P45: J11.6 (Pin_6), U43.12 (PC5)
- new net P46: J11.7 (Pin_7), U43.11 (PC6)
- new net P47: J11.8 (Pin_8), U43.10 (PC7)
- new net P48: J1.1 (Pin_1), U42.4 (PA0)
- new net P49: J1.2 (Pin_2), U42.3 (PA1)
- new net P50: J1.3 (Pin_3), U42.2 (PA2)
- new net P51: J1.4 (Pin_4), U42.1 (PA3)
- new net P52: J1.5 (Pin_5), U42.40 (PA4)
- new net P53: J1.6 (Pin_6), U42.39 (PA5)
- new net P54: J1.7 (Pin_7), U42.38 (PA6)
- new net P55: J1.8 (Pin_8), U42.37 (PA7)
- new net P56: J4.1 (Pin_1), U42.18 (PB0)
- new net P57: J4.2 (Pin_2), U42.19 (PB1)
- new net P58: J4.3 (Pin_3), U42.20 (PB2)
- new net P59: J4.4 (Pin_4), U42.21 (PB3)
- new net P60: J4.5 (Pin_5), U42.22 (PB4)
- new net P61: J4.6 (Pin_6), U42.23 (PB5)
- new net P62: J4.7 (Pin_7), U42.24 (PB6)
- new net P63: J4.8 (Pin_8), U42.25 (PB7)
- new net P64: J5.1 (Pin_1), U42.14 (PC0)
- new net P65: J5.2 (Pin_2), U42.15 (PC1)
- new net P66: J5.3 (Pin_3), U42.16 (PC2)
- new net P67: J5.4 (Pin_4), U42.17 (PC3)
- new net P68: J5.5 (Pin_5), U42.13 (PC4)
- new net P69: J5.6 (Pin_6), U42.12 (PC5)
- new net P70: J5.7 (Pin_7), U42.11 (PC6)
- new net P71: J5.8 (Pin_8), U42.10 (PC7)
- no-connect marks 2 -> 0
Other:
- moved on the sheet: U22, U23

Commit message: Final?
Parts:
- renumbered U23 to PPI1, U43 to PPI2, U42 to PPI3, U22 to PPI_Decoder1, J6 to PPI_Header1, J7 to PPI_Header2, J8 to PPI_Header3, J9 to PPI_Header4, J10 to PPI_Header5, J11 to PPI_Header6, J1 to PPI_Header7, J4 to PPI_Header8, J5 to PPI_Header9
Connections:
- net GND: now also PPI2.7 (GND)

Commit message: Hopefully the board is here
Parts:
- PPI_Decoder1: footprint (none) -> Package_DIP:DIP-20_W7.62mm
- PPI_Header1, PPI_Header2, PPI_Header3, PPI_Header4, PPI_Header5, PPI_Header6, PPI_Header7, PPI_Header8, PPI_Header9: footprint (none) -> Connector_PinHeader_1.00mm:PinHeader_1x08_P1.00mm_Horizontal
Changed lines of the file:
@@
 F 0 "PPI_Decoder1" H 2000 3031 50  0000 C CNN
 F 1 "PAL16L8" H 2000 2940 50  0000 C CNN
-F 2 "" H 2000 2150 50  0001 C CNN
+F 2 "Package_DIP:DIP-20_W7.62mm" H 2000 2150 50  0001 C CNN
 F 3 "" H 2000 2150 50  0001 C CNN
 	1    2000 2150
@@
 F 0 "PPI_Header7" H 5028 4876 50  0000 L CNN
 F 1 "Conn_01x08_Female" H 5028 4785 50  0000 L CNN
-F 2 "" H 5000 4900 50  0001 C CNN
+F 2 "Connector_PinHeader_1.00mm:PinHeader_1x08_P1.00mm_Horizontal" H 5000 4900 50  0001 C CNN
 F 3 "~" H 5000 4900 50  0001 C CNN
 	1    5000 4900
@@
 F 0 "PPI_Header8" H 5028 5776 50  0000 L CNN
 F 1 "Conn_01x08_Female" H 5028 5685 50  0000 L CNN
-F 2 "" H 5000 5800 50  0001 C CNN
+F 2 "Connector_PinHeader_1.00mm:PinHeader_1x08_P1.00mm_Horizontal" H 5000 5800 50  0001 C CNN
 F 3 "~" H 5000 5800 50  0001 C CNN
 	1    5000 5800
@@
 F 0 "PPI_Header9" H 5028 6676 50  0000 L CNN
 F 1 "Conn_01x08_Female" H 5028 6585 50  0000 L CNN
-F 2 "" H 5000 6700 50  0001 C CNN
+F 2 "Connector_PinHeader_1.00mm:PinHeader_1x08_P1.00mm_Horizontal" H 5000 6700 50  0001 C CNN
 F 3 "~" H 5000 6700 50  0001 C CNN
 	1    5000 6700
@@
 F 0 "PPI_Header4" H 10378 1626 50  0000 L CNN
 F 1 "Conn_01x08_Female" H 10378 1535 50  0000 L CNN
-F 2 "" H 10350 1650 50  0001 C CNN
+F 2 "Connector_PinHeader_1.00mm:PinHeader_1x08_P1.00mm_Horizontal" H 10350 1650 50  0001 C CNN
 F 3 "~" H 10350 1650 50  0001 C CNN
 	1    10350 1650
@@
 F 0 "PPI_Header5" H 10378 2526 50  0000 L CNN
 F 1 "Conn_01x08_Female" H 10378 2435 50  0000 L CNN
-F 2 "" H 10350 2550 50  0001 C CNN
+F 2 "Connector_PinHeader_1.00mm:PinHeader_1x08_P1.00mm_Horizontal" H 10350 2550 50  0001 C CNN
 F 3 "~" H 10350 2550 50  0001 C CNN
 	1    10350 2550
@@
 F 0 "PPI_Header6" H 10378 3426 50  0000 L CNN
 F 1 "Conn_01x08_Female" H 10378 3335 50  0000 L CNN
-F 2 "" H 10350 3450 50  0001 C CNN
+F 2 "Connector_PinHeader_1.00mm:PinHeader_1x08_P1.00mm_Horizontal" H 10350 3450 50  0001 C CNN
 F 3 "~" H 10350 3450 50  0001 C CNN
 	1    10350 3450
@@
 F 0 "PPI_Header3" H 6778 3426 50  0000 L CNN
 F 1 "Conn_01x08_Female" H 6778 3335 50  0000 L CNN
-F 2 "" H 6750 3450 50  0001 C CNN
+F 2 "Connector_PinHeader_1.00mm:PinHeader_1x08_P1.00mm_Horizontal" H 6750 3450 50  0001 C CNN
 F 3 "~" H 6750 3450 50  0001 C CNN
 	1    6750 3450
@@
 F 0 "PPI_Header2" H 6778 2526 50  0000 L CNN
 F 1 "Conn_01x08_Female" H 6778 2435 50  0000 L CNN
-F 2 "" H 6750 2550 50  0001 C CNN
+F 2 "Connector_PinHeader_1.00mm:PinHeader_1x08_P1.00mm_Horizontal" H 6750 2550 50  0001 C CNN
 F 3 "~" H 6750 2550 50  0001 C CNN
 	1    6750 2550
@@
 F 0 "PPI_Header1" H 6778 1626 50  0000 L CNN
 F 1 "Conn_01x08_Female" H 6778 1535 50  0000 L CNN
-F 2 "" H 6750 1650 50  0001 C CNN
+F 2 "Connector_PinHeader_1.00mm:PinHeader_1x08_P1.00mm_Horizontal" H 6750 1650 50  0001 C CNN
 F 3 "~" H 6750 1650 50  0001 C CNN
 	1    6750 1650

Commit message: Added some final touches
Parts:
- PPI_Header1, PPI_Header2, PPI_Header3, PPI_Header4, PPI_Header5, PPI_Header6, PPI_Header7, PPI_Header8, PPI_Header9: footprint Connector_PinHeader_1.00mm:PinHeader_1x08_P1.00mm_Horizontal -> Connector_PinHeader_1.00mm:PinHeader_1x08_P1.00mm_Vertical
Changed lines of the file:
@@
 encoding utf-8
 Sheet 8 16
-Title ""
+Title "8255 and Decode"
 Date ""
 Rev ""
-Comp ""
-Comment1 ""
+Comp "UMBC 2021"
+Comment1 "Andrew Mathews"
 Comment2 ""
 Comment3 ""
@@
 F 0 "PPI_Header7" H 5028 4876 50  0000 L CNN
 F 1 "Conn_01x08_Female" H 5028 4785 50  0000 L CNN
-F 2 "Connector_PinHeader_1.00mm:PinHeader_1x08_P1.00mm_Horizontal" H 5000 4900 50  0001 C CNN
+F 2 "Connector_PinHeader_1.00mm:PinHeader_1x08_P1.00mm_Vertical" H 5000 4900 50  0001 C CNN
 F 3 "~" H 5000 4900 50  0001 C CNN
 	1    5000 4900
@@
 F 0 "PPI_Header8" H 5028 5776 50  0000 L CNN
 F 1 "Conn_01x08_Female" H 5028 5685 50  0000 L CNN
-F 2 "Connector_PinHeader_1.00mm:PinHeader_1x08_P1.00mm_Horizontal" H 5000 5800 50  0001 C CNN
+F 2 "Connector_PinHeader_1.00mm:PinHeader_1x08_P1.00mm_Vertical" H 5000 5800 50  0001 C CNN
 F 3 "~" H 5000 5800 50  0001 C CNN
 	1    5000 5800
@@
 F 0 "PPI_Header9" H 5028 6676 50  0000 L CNN
 F 1 "Conn_01x08_Female" H 5028 6585 50  0000 L CNN
-F 2 "Connector_PinHeader_1.00mm:PinHeader_1x08_P1.00mm_Horizontal" H 5000 6700 50  0001 C CNN
+F 2 "Connector_PinHeader_1.00mm:PinHeader_1x08_P1.00mm_Vertical" H 5000 6700 50  0001 C CNN
 F 3 "~" H 5000 6700 50  0001 C CNN
 	1    5000 6700
@@
 F 0 "PPI_Header4" H 10378 1626 50  0000 L CNN
 F 1 "Conn_01x08_Female" H 10378 1535 50  0000 L CNN
-F 2 "Connector_PinHeader_1.00mm:PinHeader_1x08_P1.00mm_Horizontal" H 10350 1650 50  0001 C CNN
+F 2 "Connector_PinHeader_1.00mm:PinHeader_1x08_P1.00mm_Vertical" H 10350 1650 50  0001 C CNN
 F 3 "~" H 10350 1650 50  0001 C CNN
 	1    10350 1650
@@
 F 0 "PPI_Header5" H 10378 2526 50  0000 L CNN
 F 1 "Conn_01x08_Female" H 10378 2435 50  0000 L CNN
-F 2 "Connector_PinHeader_1.00mm:PinHeader_1x08_P1.00mm_Horizontal" H 10350 2550 50  0001 C CNN
+F 2 "Connector_PinHeader_1.00mm:PinHeader_1x08_P1.00mm_Vertical" H 10350 2550 50  0001 C CNN
 F 3 "~" H 10350 2550 50  0001 C CNN
 	1    10350 2550
@@
 F 0 "PPI_Header6" H 10378 3426 50  0000 L CNN
 F 1 "Conn_01x08_Female" H 10378 3335 50  0000 L CNN
-F 2 "Connector_PinHeader_1.00mm:PinHeader_1x08_P1.00mm_Horizontal" H 10350 3450 50  0001 C CNN
+F 2 "Connector_PinHeader_1.00mm:PinHeader_1x08_P1.00mm_Vertical" H 10350 3450 50  0001 C CNN
 F 3 "~" H 10350 3450 50  0001 C CNN
 	1    10350 3450
@@
 F 0 "PPI_Header3" H 6778 3426 50  0000 L CNN
 F 1 "Conn_01x08_Female" H 6778 3335 50  0000 L CNN
-F 2 "Connector_PinHeader_1.00mm:PinHeader_1x08_P1.00mm_Horizontal" H 6750 3450 50  0001 C CNN
+F 2 "Connector_PinHeader_1.00mm:PinHeader_1x08_P1.00mm_Vertical" H 6750 3450 50  0001 C CNN
 F 3 "~" H 6750 3450 50  0001 C CNN
 	1    6750 3450
@@
 F 0 "PPI_Header2" H 6778 2526 50  0000 L CNN
 F 1 "Conn_01x08_Female" H 6778 2435 50  0000 L CNN
-F 2 "Connector_PinHeader_1.00mm:PinHeader_1x08_P1.00mm_Horizontal" H 6750 2550 50  0001 C CNN
+F 2 "Connector_PinHeader_1.00mm:PinHeader_1x08_P1.00mm_Vertical" H 6750 2550 50  0001 C CNN
 F 3 "~" H 6750 2550 50  0001 C CNN
 	1    6750 2550
@@
 F 0 "PPI_Header1" H 6778 1626 50  0000 L CNN
 F 1 "Conn_01x08_Female" H 6778 1535 50  0000 L CNN
-F 2 "Connector_PinHeader_1.00mm:PinHeader_1x08_P1.00mm_Horizontal" H 6750 1650 50  0001 C CNN
+F 2 "Connector_PinHeader_1.00mm:PinHeader_1x08_P1.00mm_Vertical" H 6750 1650 50  0001 C CNN
 F 3 "~" H 6750 1650 50  0001 C CNN
 	1    6750 1650
