File: Final/SRAM(FINAL).sch (KiCad schematic (older format))
At the start: 0 parts

Commit message: New stuff
Parts:
- added U10, U11, U13, U15: CY7C199, symbol Memory_RAM:CY7C199
- added U16: 74LS138, symbol 74xx:74LS138
- added U17, U18: 74LVC1GU04DRL, Package_TO_SOT_SMD:SOT-553, symbol 74xGxx:74LVC1GU04DRL
- added U19, U20, U21: 74AHC1G08, symbol 74xGxx:74AHC1G08
Connections:
- new net: U16.14 (O1), U18.2, U19.2, U21.2
- new net: U16.15 (O0), U17.2, U19.1, U20.1
- new net: U18.4, U20.2
- new net: U17.4, U21.1
- new net A0: U10.21 (A0), U11.21 (A0), U13.21 (A0), U15.21 (A0)
- new net A1: U10.23 (A1), U11.23 (A1), U13.23 (A1), U15.23 (A1)
- new net A10: U10.6 (A10), U11.6 (A10), U13.6 (A10), U15.6 (A10)
- new net A11: U10.7 (A11), U11.7 (A11), U13.7 (A11), U15.7 (A11)
- new net A12: U10.8 (A12), U11.8 (A12), U13.8 (A12), U15.8 (A12)
- new net A13: U10.9 (A13), U11.9 (A13), U13.9 (A13), U15.9 (A13)
- new net A14: U10.10 (A14), U11.10 (A14), U13.10 (A14), U15.10 (A14)
- new net A15: U16.1 (A0)
- new net A16: U16.2 (A1)
- new net A17: U16.3 (A2)
- new net A18: U16.5 (E2)
- new net A19: U16.4 (E1)
- new net A2: U10.24 (A2), U11.24 (A2), U13.24 (A2), U15.24 (A2)
- new net A3: U10.25 (A3), U11.25 (A3), U13.25 (A3), U15.25 (A3)
- new net A4: U10.26 (A4), U11.26 (A4), U13.26 (A4), U15.26 (A4)
- new net A5: U10.1 (A5), U11.1 (A5), U13.1 (A5), U15.1 (A5)
- new net A6: U10.2 (A6), U11.2 (A6), U13.2 (A6), U15.2 (A6)
- new net A7: U10.3 (A7), U11.3 (A7), U13.3 (A7), U15.3 (A7)
- new net A8: U10.4 (A8), U11.4 (A8), U13.4 (A8), U15.4 (A8)
- new net A9: U10.5 (A9), U11.5 (A9), U13.5 (A9), U15.5 (A9)
- new net CE00: U10.20 (~CE~)
- new net CE01: U11.20 (~CE~), U21.4
- new net CE10: U13.20 (~CE~), U20.4
- new net CE11: U15.20 (~CE~), U19.4
- new net D0: U10.11 (D0), U11.11 (D0), U13.11 (D0), U15.11 (D0)
- new net D1: U10.12 (D1), U11.12 (D1), U13.12 (D1), U15.12 (D1)
- new net D2: U10.13 (D2), U11.13 (D2), U13.13 (D2), U15.13 (D2)
- new net D3: U10.15 (D3), U11.15 (D3), U13.15 (D3), U15.15 (D3)
- new net D4: U10.16 (D4), U11.16 (D4), U13.16 (D4), U15.16 (D4)
- new net D5: U10.17 (D5), U11.17 (D5), U13.17 (D5), U15.17 (D5)
- new net D6: U10.18 (D6), U11.18 (D6), U13.18 (D6), U15.18 (D6)
- new net D7: U10.19 (D7), U11.19 (D7), U13.19 (D7), U15.19 (D7)
- new net GND: U10.14 (GND), U11.14 (GND), U13.14 (GND), U15.14 (GND), U16.6 (E3), U16.8 (GND), U19.3 (GND), U20.3 (GND), U21.3 (GND)
- new net VCC: U10.28 (VCC), U11.28 (VCC), U13.28 (VCC), U15.28 (VCC), U16.16 (VCC), U19.5 (VCC), U20.5 (VCC), U21.5 (VCC)
- new net ~RD: U10.22 (~OE~), U11.22 (~OE~), U13.22 (~OE~), U15.22 (~OE~)
- new net ~WR: U10.27 (~WE~), U11.27 (~WE~), U13.27 (~WE~), U15.27 (~WE~)
- no-connect marks 0 -> 6
Other:
- note added: "0\nH\n"
- note added: "0\nL\n"
- note added: "1\nH"
- note added: "1\nL\n"
- note added: "CE ; lsb ; msb\nChipEnable ; left = 0, right = 1; low = 0, high = 1"
