File: Final/SRAM(FINAL).sch (KiCad schematic (older format))
At the start: 10 parts, among them U10 CY7C199, U11 CY7C199, U13 CY7C199, U15 CY7C199, U16 74LS138, U17 74LVC1GU04DRL, U18 74LVC1GU04DRL, U19 74AHC1G08, U20 74AHC1G08, U21 74AHC1G08

Commit message: For Commenting
Parts:
- removed U17, U18: 74LVC1GU04DRL, Package_TO_SOT_SMD:SOT-553, symbol 74xGxx:74LVC1GU04DRL
- added U17, U18: 74LS04, symbol 74xx:74LS04
Connections:
- net D0: no longer U11.11 (D0), U15.11 (D0)
- net D1: no longer U11.12 (D1), U15.12 (D1)
- net D2: no longer U11.13 (D2), U15.13 (D2)
- net D3: no longer U11.15 (D3), U15.15 (D3)
- net D4: no longer U11.16 (D4), U15.16 (D4)
- net D5: no longer U11.17 (D5), U15.17 (D5)
- net D6: no longer U11.18 (D6), U15.18 (D6)
- net D7: no longer U11.19 (D7), U15.19 (D7)
- net at U16.14 (O1), U19.2, U21.2: now also U18.1
- net at U20.2: now also U18.2
- net at U21.1: now also U17.2
- new net D10: U11.13 (D2), U15.13 (D2)
- new net D11: U11.15 (D3), U15.15 (D3)
- new net D12: U11.16 (D4), U15.16 (D4)
- new net D13: U11.17 (D5), U15.17 (D5)
- new net D14: U11.18 (D6), U15.18 (D6)
- new net D15: U11.19 (D7), U15.19 (D7)
- new net D8: U11.11 (D0), U15.11 (D0)
- new net D9: U11.12 (D1), U15.12 (D1)
Changed lines of the file:
@@
 $Descr A4 11693 8268
 encoding utf-8
-Sheet 5 14
+Sheet 7 16
 Title ""
 Date ""
@@
 $EndDescr
 $Comp
-L 74xx:74LS138 U16
-U 1 1 608F8DF6
-P 8350 4750
-F 0 "U16" H 8350 5531 50  0000 C CNN
-F 1 "74LS138" H 8350 5440 50  0000 C CNN
-F 2 "" H 8350 4750 50  0001 C CNN
-F 3 "http://www.ti.com/lit/gpn/sn74LS138" H 8350 4750 50  0001 C CNN
-	1    8350 4750
-	1    0    0    -1
-$EndComp
-$Comp
 L Memory_RAM:CY7C199 U15
 U 1 1 60931DB6
@@
 Wire Wire Line
 	5900 4500 6000 4500
-Text Label 7550 4350 2    50   ~ 0
-A[15..19]
-Wire Bus Line
-	7550 4350 7650 4350
-Entry Wire Line
-	7650 4350 7750 4450
-Entry Wire Line
-	7650 4450 7750 4550
-Entry Wire Line
-	7650 4550 7750 4650
-Wire Wire Line
-	7750 4650 7850 4650
-Wire Wire Line
-	7750 4550 7850 4550
-Wire Wire Line
-	7750 4450 7850 4450
-Text Label 7750 4450 0    50   ~ 0
-A15
-Text Label 7750 4550 0    50   ~ 0
-A16
-Text Label 7750 4650 0    50   ~ 0
-A17
 $Comp
 L power:GND #PWR024
@@
 	1    0    0    -1
 $EndComp
-Entry Wire Line
-	7650 5050 7750 5150
-Entry Wire Line
-	7650 4950 7750 5050
-$Comp
-L power:GND #PWR029
-U 1 1 612AF1D8
-P 7850 4950
-F 0 "#PWR029" H 7850 4700 50  0001 C CNN
-F 1 "GND" H 7855 4777 50  0000 C CNN
-F 2 "" H 7850 4950 50  0001 C CNN
-F 3 "" H 7850 4950 50  0001 C CNN
-	1    7850 4950
-	-1   0    0    1
-$EndComp
-Wire Wire Line
-	7750 5050 7850 5050
-Wire Wire Line
-	7750 5150 7850 5150
-Text Label 7750 5050 0    50   ~ 0
-A18
-Text Label 7750 5150 0    50   ~ 0
-A19
 Text Notes 3100 6300 0    50   ~ 0
 0\nL\n
@@
 Wire Wire Line
 	10150 6000 10500 6000
-$Comp
-L 74xGxx:74LVC1GU04DRL U18
-U 1 1 6138973A
-P 9450 4750
-F 0 "U18" H 9206 4704 50  0000 R CNN
-F 1 "74LVC1GU04DRL" H 9206 4795 50  0000 R CNN
-F 2 "Package_TO_SOT_SMD:SOT-553" H 9450 4500 50  0001 C CNN
-F 3 "http://www.ti.com/lit/ds/symlink/sn74lvc1gu04.pdf" H 9375 4750 50  0001 C CNN
-	1    9450 4750
-	0    1    1    0
-$EndComp
-Connection ~ 9450 4550
-Wire Wire Line
-	9450 4550 9600 4550
 Wire Wire Line
 	9150 4450 9150 5200
-Wire Wire Line
-	9150 5200 9300 5200
 Connection ~ 9150 4450
 Wire Wire Line
 	9150 4450 9600 4450
 Wire Wire Line
-	9450 5050 9450 5300
-Wire Wire Line
-	9450 5300 9600 5300
-$Comp
-L 74xGxx:74LVC1GU04DRL U17
-U 1 1 613EE8C0
-P 9300 5400
-F 0 "U17" V 9304 5644 50  0000 L CNN
-F 1 "74LVC1GU04DRL" V 9395 5644 50  0000 L CNN
-F 2 "Package_TO_SOT_SMD:SOT-553" H 9300 5150 50  0001 C CNN
-F 3 "http://www.ti.com/lit/ds/symlink/sn74lvc1gu04.pdf" H 9225 5400 50  0001 C CNN
-	1    9300 5400
-	0    1    1    0
-$EndComp
-Connection ~ 9300 5200
-Wire Wire Line
-	9300 5200 9600 5200
-Wire Wire Line
-	8950 4550 8950 6050
+	9450 5050 9450 5150
 Wire Wire Line
 	8950 6050 9600 6050
 Connection ~ 8950 4550
-Wire Wire Line
-	8950 4550 9450 4550
-Wire Wire Line
-	9300 5700 9300 5950
 Wire Wire Line
 	9300 5950 9600 5950
@@
 D7
 Text HLabel 5600 1100 2    50   Input ~ 0
-D0
+D8
 Text HLabel 5600 1200 2    50   Input ~ 0
-D1
+D9
 Text HLabel 5600 1300 2    50   Input ~ 0
-D2
+D10
 Text HLabel 5600 1400 2    50   Input ~ 0
-D3
+D11
 Text HLabel 5600 1500 2    50   Input ~ 0
-D4
+D12
 Text HLabel 5600 1600 2    50   Input ~ 0
-D5
+D13
 Text HLabel 5600 1700 2    50   Input ~ 0
-D6
+D14
 Text HLabel 5600 1800 2    50   Input ~ 0
-D7
+D15
 Wire Wire Line
 	6500 1100 6600 1100
@@
 A14
 Text HLabel 7950 1100 2    50   Input ~ 0
-D0
+D8
 Text HLabel 7950 1200 2    50   Input ~ 0
-D1
+D9
 Text HLabel 7950 1300 2    50   Input ~ 0
-D2
+D10
 Text HLabel 7950 1400 2    50   Input ~ 0
-D3
+D11
 Text HLabel 7950 1500 2    50   Input ~ 0
-D4
+D12
 Text HLabel 7950 1600 2    50   Input ~ 0
-D5
+D13
 Text HLabel 7950 1700 2    50   Input ~ 0
-D6
+D14
 Text HLabel 7950 1800 2    50   Input ~ 0
-D7
+D15
 Wire Wire Line
 	7800 1100 7950 1100
@@
 Wire Wire Line
 	7800 1800 7950 1800
-Wire Bus Line
-	7650 4350 7650 5050
+$Comp
+L 74xx:74LS04 U18
+U 1 1 619E8FEB
+P 9450 4850
+F 0 "U18" V 9404 5030 50  0000 L CNN
+F 1 "74LS04" V 9495 5030 50  0000 L CNN
+F 2 "" H 9450 4850 50  0001 C CNN
+F 3 "http://www.ti.com/lit/gpn/sn74LS04" H 9450 4850 50  0001 C CNN
+	1    9450 4850
+	0    1    1    0
+$EndComp
+Wire Wire Line
+	8950 4550 9450 4550
+Connection ~ 9450 4550
+Wire Wire Line
+	9450 4550 9600 4550
+Wire Wire Line
+	9600 5300 9450 5300
+Wire Wire Line
+	9450 5300 9450 5150
+Connection ~ 9450 5150
+Wire Wire Line
+	9150 5200 9600 5200
+$Comp
+L 74xx:74LS04 U17
+U 1 1 619F3CB3
+P 9300 5500
+F 0 "U17" V 9254 5680 50  0000 L CNN
+F 1 "74LS04" V 9345 5680 50  0000 L CNN
+F 2 "" H 9300 5500 50  0001 C CNN
+F 3 "http://www.ti.com/lit/gpn/sn74LS04" H 9300 5500 50  0001 C CNN
+	1    9300 5500
+	0    1    1    0
+$EndComp
+Wire Wire Line
+	9300 5950 9300 5800
+Wire Wire Line
+	8950 4550 8950 6050
+$Comp
+L power:GND #PWR0132
+U 1 1 61A0948D
+P 7850 4950
+F 0 "#PWR0132" H 7850 4700 50  0001 C CNN
+F 1 "GND" V 7855 4822 50  0000 R CNN
+F 2 "" H 7850 4950 50  0001 C CNN
+F 3 "" H 7850 4950 50  0001 C CNN
+	1    7850 4950
+	0    1    1    0
+$EndComp
+Text HLabel 7850 5150 0    50   Input ~ 0
+A19
+Text HLabel 7850 5050 0    50   Input ~ 0
+A18
+Text HLabel 7850 4650 0    50   Input ~ 0
+A17
+Text HLabel 7850 4550 0    50   Input ~ 0
+A16
+Text HLabel 7850 4450 0    50   Input ~ 0
+A15
+$Comp
+L 74xx:74LS138 U16
+U 1 1 608F8DF6
+P 8350 4750
+F 0 "U16" H 8350 5531 50  0000 C CNN
+F 1 "74LS138" H 8350 5440 50  0000 C CNN
+F 2 "" H 8350 4750 50  0001 C CNN
+F 3 "http://www.ti.com/lit/gpn/sn74LS138" H 8350 4750 50  0001 C CNN
+	1    8350 4750
+	1    0    0    -1
+$EndComp
 $EndSCHEMATC

Commit message: Final?
Parts:
- removed U16: 74LS138, symbol 74xx:74LS138
- added SRAMSelector1: PAL16L8, symbol Logic_Programmable:PAL16L8
- added U1: 74AHC1G08, symbol 74xGxx:74AHC1G08
- renumbered U15 to HighHighSRAM1, U11 to HighLowSRAM1, U13 to LowHighSRAM1, U10 to LowLowSRAM1
Connections:
- net A0: now also SRAMSelector1.16 (IO4)
- net A1: now also SRAMSelector1.1 (I1)
- net A10: now also SRAMSelector1.17 (I03)
- net A2: now also SRAMSelector1.2 (I2)
- net A3: now also SRAMSelector1.3 (I3)
- net A4: now also SRAMSelector1.4 (I4)
- net A5: now also SRAMSelector1.5 (I5)
- net A6: now also SRAMSelector1.6 (I6)
- net A7: now also SRAMSelector1.7 (I7)
- net A8: now also SRAMSelector1.8 (I8)
- net A9: now also SRAMSelector1.9 (I9)
- net CE00: now also U1.4
- net GND: now also SRAMSelector1.10 (GND), U1.3 (GND)
- net VCC: now also SRAMSelector1.20 (VCC), U1.5 (VCC)
- net at U18.1, U19.2, U21.2: now also SRAMSelector1.18 (IO2)
- net at U19.1, U20.1: now also U17.1, SRAMSelector1.19 (IO1)
- net at U18.2, U20.2: now also U1.1
- net at U17.2, U21.1: now also U1.2
- new net ~BHE: SRAMSelector1.11 (I10)
- no-connect marks 6 -> 4
Other:
- moved on the sheet: U17A, U18A, U19, U20, U21

Commit message: Hopefully the board is here
Parts:
- HighHighSRAM1, HighLowSRAM1, LowHighSRAM1, LowLowSRAM1: footprint (none) -> Package_DIP:DIP-28_W7.62mm
- SRAMSelector1: footprint (none) -> Package_DIP:DIP-20_W7.62mm
- U1, U19, U20, U21: footprint (none) -> Package_DIP:DIP-5-6_W7.62mm
- U17, U18: footprint (none) -> Package_DIP:DIP-14_W7.62mm
Changed lines of the file:
@@
 F 0 "HighHighSRAM1" H 7200 3381 50  0000 C CNN
 F 1 "CY7C199" H 7200 3290 50  0000 C CNN
-F 2 "" H 7200 2000 50  0001 C CNN
+F 2 "Package_DIP:DIP-28_W7.62mm" H 7200 2000 50  0001 C CNN
 F 3 "" H 7200 2000 50  0001 C CNN
 	1    7200 2000
@@
 F 0 "LowLowSRAM1" H 3100 6081 50  0000 C CNN
 F 1 "CY7C199" H 3100 5990 50  0000 C CNN
-F 2 "" H 3100 4700 50  0001 C CNN
+F 2 "Package_DIP:DIP-28_W7.62mm" H 3100 4700 50  0001 C CNN
 F 3 "" H 3100 4700 50  0001 C CNN
 	1    3100 4700
@@
 F 0 "U19" H 9875 4117 50  0000 C CNN
 F 1 "74AHC1G08" H 9875 4026 50  0000 C CNN
-F 2 "" H 9900 3850 50  0001 C CNN
+F 2 "Package_DIP:DIP-5-6_W7.62mm" H 9900 3850 50  0001 C CNN
 F 3 "http://www.ti.com/lit/sg/scyt129e/scyt129e.pdf" H 9900 3850 50  0001 C CNN
 	1    9900 3850
@@
 F 0 "U20" H 9875 4867 50  0000 C CNN
 F 1 "74AHC1G08" H 9875 4776 50  0000 C CNN
-F 2 "" H 9900 4600 50  0001 C CNN
+F 2 "Package_DIP:DIP-5-6_W7.62mm" H 9900 4600 50  0001 C CNN
 F 3 "http://www.ti.com/lit/sg/scyt129e/scyt129e.pdf" H 9900 4600 50  0001 C CNN
 	1    9900 4600
@@
 F 0 "U21" H 9875 5617 50  0000 C CNN
 F 1 "74AHC1G08" H 9875 5526 50  0000 C CNN
-F 2 "" H 9900 5350 50  0001 C CNN
+F 2 "Package_DIP:DIP-5-6_W7.62mm" H 9900 5350 50  0001 C CNN
 F 3 "http://www.ti.com/lit/sg/scyt129e/scyt129e.pdf" H 9900 5350 50  0001 C CNN
 	1    9900 5350
@@
 F 0 "HighLowSRAM1" H 5000 3381 50  0000 C CNN
 F 1 "CY7C199" H 5000 3290 50  0000 C CNN
-F 2 "" H 5000 2000 50  0001 C CNN
+F 2 "Package_DIP:DIP-28_W7.62mm" H 5000 2000 50  0001 C CNN
 F 3 "" H 5000 2000 50  0001 C CNN
 	1    5000 2000
@@
 F 0 "LowHighSRAM1" H 5300 6081 50  0000 C CNN
 F 1 "CY7C199" H 5300 5990 50  0000 C CNN
-F 2 "" H 5300 4700 50  0001 C CNN
+F 2 "Package_DIP:DIP-28_W7.62mm" H 5300 4700 50  0001 C CNN
 F 3 "" H 5300 4700 50  0001 C CNN
 	1    5300 4700
@@
 F 0 "U18" V 9404 4380 50  0000 L CNN
 F 1 "74LS04" V 9495 4380 50  0000 L CNN
-F 2 "" H 9450 4200 50  0001 C CNN
+F 2 "Package_DIP:DIP-14_W7.62mm" H 9450 4200 50  0001 C CNN
 F 3 "http://www.ti.com/lit/gpn/sn74LS04" H 9450 4200 50  0001 C CNN
 	1    9450 4200
@@
 F 0 "U17" V 9254 5030 50  0000 L CNN
 F 1 "74LS04" V 9345 5030 50  0000 L CNN
-F 2 "" H 9300 4850 50  0001 C CNN
+F 2 "Package_DIP:DIP-14_W7.62mm" H 9300 4850 50  0001 C CNN
 F 3 "http://www.ti.com/lit/gpn/sn74LS04" H 9300 4850 50  0001 C CNN
 	1    9300 4850
@@
 F 0 "SRAMSelector1" H 7650 5481 50  0000 C CNN
 F 1 "PAL16L8" H 7650 5390 50  0000 C CNN
-F 2 "" H 7650 4600 50  0001 C CNN
+F 2 "Package_DIP:DIP-20_W7.62mm" H 7650 4600 50  0001 C CNN
 F 3 "" H 7650 4600 50  0001 C CNN
 	1    7650 4600
@@
 F 0 "U1" H 9875 6217 50  0000 C CNN
 F 1 "74AHC1G08" H 9875 6126 50  0000 C CNN
-F 2 "" H 9900 5950 50  0001 C CNN
+F 2 "Package_DIP:DIP-5-6_W7.62mm" H 9900 5950 50  0001 C CNN
 F 3 "http://www.ti.com/lit/sg/scyt129e/scyt129e.pdf" H 9900 5950 50  0001 C CNN
 	1    9900 5950
