File: Final/LCD(FINAL).sch (KiCad schematic (older format))
At the start: 2 parts, among them U14 PAL16L8

Commit message: Final?
Parts:
- renumbered U14 to LCD_16L8, DS1 to LCD_4x20
Connections:
- net VSS is gone; now on net GND: LCD_4x20.1 (VSS)
- net VDD renamed +3V3
Changed lines of the file:
@@
 $EndDescr
 $Comp
-L Logic_Programmable:PAL16L8 U14
+L Logic_Programmable:PAL16L8 LCD_16L8
 U 1 1 6158A041
 P 2800 2350
-F 0 "U14" H 2800 3231 50  0000 C CNN
+F 0 "LCD_16L8" H 2800 3231 50  0000 C CNN
 F 1 "PAL16L8" H 2800 3140 50  0000 C CNN
 F 2 "" H 2800 2350 50  0001 C CNN
@@
 $EndComp
 $Comp
-L LCD4x20:LCD4x20 DS1
+L LCD4x20:LCD4x20 LCD_4x20
 U 1 1 61587A20
 P 4500 1900
-F 0 "DS1" H 5050 2165 50  0000 C CNN
+F 0 "LCD_4x20" H 5050 2165 50  0000 C CNN
 F 1 "LCD4x20" H 5050 2074 50  0000 C CNN
 F 2 "LCD4x20" H 5450 2000 50  0001 L CNN
@@
 NoConn ~ 5600 2700
 NoConn ~ 5600 2800
-$Comp
-L power:VSS #PWR0123
-U 1 1 6162CD84
-P 4500 1900
-F 0 "#PWR0123" H 4500 1750 50  0001 C CNN
-F 1 "VSS" V 4515 2028 50  0000 L CNN
-F 2 "" H 4500 1900 50  0001 C CNN
-F 3 "" H 4500 1900 50  0001 C CNN
-	1    4500 1900
-	0    -1   -1   0
-$EndComp
-$Comp
-L power:VDD #PWR0124
-U 1 1 6162D4FF
-P 4500 2000
-F 0 "#PWR0124" H 4500 1850 50  0001 C CNN
-F 1 "VDD" V 4515 2127 50  0000 L CNN
-F 2 "" H 4500 2000 50  0001 C CNN
-F 3 "" H 4500 2000 50  0001 C CNN
-	1    4500 2000
-	0    -1   -1   0
-$EndComp
 Wire Wire Line
 	2800 1400 2800 1650
@@
 Text HLabel 4500 2200 0    50   Input ~ 0
 M~IO
+$Comp
+L power:GND #PWR0115
+U 1 1 6201B679
+P 4500 1900
+F 0 "#PWR0115" H 4500 1650 50  0001 C CNN
+F 1 "GND" V 4505 1772 50  0000 R CNN
+F 2 "" H 4500 1900 50  0001 C CNN
+F 3 "" H 4500 1900 50  0001 C CNN
+	1    4500 1900
+	0    1    1    0
+$EndComp
+$Comp
+L power:+3.3V #PWR0123
+U 1 1 6201BDAC
+P 4500 2000
+F 0 "#PWR0123" H 4500 1850 50  0001 C CNN
+F 1 "+3.3V" V 4515 2128 50  0000 L CNN
+F 2 "" H 4500 2000 50  0001 C CNN
+F 3 "" H 4500 2000 50  0001 C CNN
+	1    4500 2000
+	0    -1   -1   0
+$EndComp
 $EndSCHEMATC

Commit message: Final..I Hope
Parts:
- LCD_4x20: footprint LCD4x20 -> (none)
Changed lines of the file:
@@
 F 0 "LCD_4x20" H 5050 2165 50  0000 C CNN
 F 1 "LCD4x20" H 5050 2074 50  0000 C CNN
-F 2 "LCD4x20" H 5450 2000 50  0001 L CNN
+F 2 "" H 5450 2000 50  0001 L CNN
 F 3 "https://componentsearchengine.com/Datasheets/1/LCD4x20.pdf" H 5450 1900 50  0001 L CNN
 F 4 "LCD Character Display Modules & Accessories STN-Y/G Transfl 77.5 x 47.0" H 5450 1800 50  0001 L CNN "Description"

Commit message: Hopefully the board is here
Parts:
- LCD_16L8, LCD_4x20: footprint (none) -> Package_DIP:DIP-20_W7.62mm
Changed lines of the file:
@@
 F 0 "LCD_16L8" H 2800 3231 50  0000 C CNN
 F 1 "PAL16L8" H 2800 3140 50  0000 C CNN
-F 2 "" H 2800 2350 50  0001 C CNN
+F 2 "Package_DIP:DIP-20_W7.62mm" H 2800 2350 50  0001 C CNN
 F 3 "" H 2800 2350 50  0001 C CNN
 	1    2800 2350
@@
 F 0 "LCD_4x20" H 5050 2165 50  0000 C CNN
 F 1 "LCD4x20" H 5050 2074 50  0000 C CNN
-F 2 "" H 5450 2000 50  0001 L CNN
+F 2 "Package_DIP:DIP-20_W7.62mm" H 5450 2000 50  0001 L CNN
 F 3 "https://componentsearchengine.com/Datasheets/1/LCD4x20.pdf" H 5450 1900 50  0001 L CNN
 F 4 "LCD Character Display Modules & Accessories STN-Y/G Transfl 77.5 x 47.0" H 5450 1800 50  0001 L CNN "Description"
