File: Final/Final.kicad_pcb (KiCad board)
At the start: 2 copper layers, 12 parts, among them U1 8086_Min_Mode, U17 74LVC1GU04DRL, U18 74LVC1GU04DRL, U23 8255, U25 8259, U27 8254, U28 pkd8279, U30 16550, U36 MAN71A, U37 MAN71A, U8 8284

Commit message: Final..I Hope
Parts:
- removed DS1: LCD4x20, LCD4x20
- removed U23: 8255, Package_DIP:DIP-40_W15.24mm
- removed U25: 8259, Package_DIP:DIP-28_W15.24mm
- removed U27: 8254, Package_DIP:DIP-24_W15.24mm
- removed U28: pkd8279, pkd8279
- removed U30: 16550, Package_DIP:DIP-40_W15.24mm
- removed U36, U37: MAN71A, Display_7Segment:MAN71A
- removed U8: 8284, Package_DIP:DIP-18_W7.62mm
- added 8259INTR1: 8259, Package_DIP:DIP-28_W15.24mm, F.Cu at (201.6, 75.6)
- added 8259Selector1: PAL16L8, Package_DIP:DIP-20_W7.62mm, F.Cu at (201.6, 57.2)
- added 8279Keyboard1: pkd8279, Package_DIP:DIP-40_W15.24mm, F.Cu at (17.6, 18.1)
- added C10: CP1_Small, Capacitor_THT:CP_Axial_L10.0mm_D4.5mm_P15.00mm_Horizontal, F.Cu at (163.2, 117.8)
- added C11: CP1_Small, Capacitor_THT:CP_Axial_L10.0mm_D4.5mm_P15.00mm_Horizontal, F.Cu at (126.1, 143.9)
- added C12: CP1_Small, Capacitor_THT:CP_Axial_L10.0mm_D4.5mm_P15.00mm_Horizontal, F.Cu at (163.2, 124.3)
- added C13: CP1_Small, Capacitor_THT:CP_Axial_L10.0mm_D4.5mm_P15.00mm_Horizontal, F.Cu at (144.6, 137.4)
- added C14: CP1_Small, Capacitor_THT:CP_Axial_L10.0mm_D4.5mm_P15.00mm_Horizontal, F.Cu at (163.2, 130.9)
- added C15: CP1_Small, Capacitor_THT:CP_Axial_L10.0mm_D4.5mm_P15.00mm_Horizontal, F.Cu at (144.6, 143.9)
- added C16: CP1_Small, Capacitor_THT:CP_Axial_L10.0mm_D4.5mm_P15.00mm_Horizontal, F.Cu at (144.6, 124.3)
- added C17: CP1_Small, Capacitor_THT:CP_Axial_L10.0mm_D4.5mm_P15.00mm_Horizontal, F.Cu at (163.2, 137.4)
- added C18: CP1_Small, Capacitor_THT:CP_Axial_L10.0mm_D4.5mm_P15.00mm_Horizontal, F.Cu at (163.2, 111.3)
- added C19: CP1_Small, Capacitor_THT:CP_Axial_L10.0mm_D4.5mm_P15.00mm_Horizontal, F.Cu at (163.2, 104.8)
- added C20: CP1_Small, Capacitor_THT:CP_Axial_L10.0mm_D4.5mm_P15.00mm_Horizontal, F.Cu at (107.5, 143.9)
- added C21: CP1_Small, Capacitor_THT:CP_Axial_L10.0mm_D4.5mm_P15.00mm_Horizontal, F.Cu at (163.2, 143.9)
- added C22: CP1_Small, Capacitor_THT:CP_Axial_L10.0mm_D4.5mm_P15.00mm_Horizontal, F.Cu at (126.1, 130.9)
- added C23: CP1_Small, Capacitor_THT:CP_Axial_L10.0mm_D4.5mm_P15.00mm_Horizontal, F.Cu at (107.5, 137.4)
- added C24: CP1_Small, Capacitor_THT:CP_Axial_L10.0mm_D4.5mm_P15.00mm_Horizontal, F.Cu at (126.1, 124.3)
- added C25: CP1_Small, Capacitor_THT:CP_Axial_L10.0mm_D4.5mm_P15.00mm_Horizontal, F.Cu at (144.6, 111.3)
- added C26: CP1_Small, Capacitor_THT:CP_Axial_L10.0mm_D4.5mm_P15.00mm_Horizontal, F.Cu at (144.6, 117.8)
- added C27: CP1_Small, Capacitor_THT:CP_Axial_L10.0mm_D4.5mm_P15.00mm_Horizontal, F.Cu at (144.6, 104.8)
- added C28: CP1_Small, Capacitor_THT:CP_Axial_L10.0mm_D4.5mm_P15.00mm_Horizontal, F.Cu at (126.1, 137.4)
- added C3: CP1_Small, Capacitor_THT:CP_Axial_L10.0mm_D4.5mm_P15.00mm_Horizontal, F.Cu at (126.1, 117.8)
- added C4: CP1_Small, Capacitor_THT:CP_Axial_L10.0mm_D4.5mm_P15.00mm_Horizontal, F.Cu at (126.1, 111.3)
- added C5: CP1_Small, Capacitor_THT:CP_Axial_L10.0mm_D4.5mm_P15.00mm_Horizontal, F.Cu at (107.5, 130.9)
- added C6: CP1_Small, Capacitor_THT:CP_Axial_L10.0mm_D4.5mm_P15.00mm_Horizontal, F.Cu at (107.5, 124.3)
- added C7: CP1_Small, Capacitor_THT:CP_Axial_L10.0mm_D4.5mm_P15.00mm_Horizontal, F.Cu at (126.1, 104.8)
- added C8: CP1_Small, Capacitor_THT:CP_Axial_L10.0mm_D4.5mm_P15.00mm_Horizontal, F.Cu at (107.5, 117.8)
- added C9: CP1_Small, Capacitor_THT:CP_Axial_L10.0mm_D4.5mm_P15.00mm_Horizontal, F.Cu at (144.6, 130.9)
- added CLK1: 8284, Package_DIP:DIP-18_W7.62mm, F.Cu at (151.0, 149.6)
- added CLK_Capacitor1: 10uF, Capacitor_THT:CP_Axial_L10.0mm_D4.5mm_P15.00mm_Horizontal, F.Cu at (162.0, 151.0)
- added CLK_Resistor1: 10k, Resistor_THT:R_Axial_DIN0204_L3.6mm_D1.6mm_P1.90mm_Vertical, F.Cu at (161.8, 169.0)
- added CLK_Switch1: SW_DPST_x2, Button_Switch_THT:Push_E-Switch_KS01Q01, F.Cu at (164.6, 158.5)
- added CMOS1: 28F010, Package_DIP:DIP-32_W7.62mm, F.Cu at (141.0, 24.1)
- added CPU1: 8086_Min_Mode, Package_DIP:DIP-40_W15.24mm, F.Cu at (17.6, 93.4)
- added CPU_ADecode1: 74LS373, Package_DIP:DIP-20_W7.62mm, F.Cu at (36.0, 93.4)
- added CPU_ADecode2: 74LS373, Package_DIP:DIP-20_W7.62mm, F.Cu at (46.9, 120.4)
- added CPU_ADecode3: 74LS373, Package_DIP:DIP-20_W7.62mm, F.Cu at (36.0, 120.4)
- added CPU_Capacitor1: CP1_Small, Capacitor_THT:CP_Axial_L10.0mm_D4.5mm_P15.00mm_Horizontal, F.Cu at (57.9, 121.8)
- added CPU_DDecode1: 74LS245, Package_DIP:DIP-20_W7.62mm, F.Cu at (68.6, 93.4)
- added CPU_DDecode2: 74LS245, Package_DIP:DIP-20_W7.62mm, F.Cu at (57.7, 93.4)
- added CPU_IO/WR1: 74LS244, Package_DIP:DIP-20_W7.62mm, F.Cu at (46.9, 93.4)
- added CPU_Resistor1: R_US, Resistor_THT:R_Axial_DIN0204_L3.6mm_D1.6mm_P1.90mm_Vertical, F.Cu at (17.6, 145.3)
- added CPU_Switch1: SW_Push, Button_Switch_THT:SW_CW_GPTS203211B, F.Cu at (79.8, 95.4)
- added CRYSTAL1: Crystal, Crystal:Crystal_AT310_D3.0mm_L10.0mm_Vertical, F.Cu at (180.0, 150.1)
- added Counter1: 8254, Package_DIP:DIP-24_W15.24mm, F.Cu at (69.7, 195.6)
- added Counter_Decode1: PAL16L8, Package_DIP:DIP-20_W7.62mm, F.Cu at (69.7, 177.2)
- added Counter_Header1: Conn_01x06_Female, Connector_PinHeader_1.00mm:PinHeader_1x06_P1.00mm_Horizontal, F.Cu at (69.2, 166.4)
- added Counter_Resistor1: 10000, Resistor_THT:R_Axial_DIN0204_L3.6mm_D1.6mm_P1.90mm_Vertical, F.Cu at (96.2, 177.2)
- added D1: CPU_Diode, Diode_THT:D_5KPW_P7.62mm_Vertical_KathodeUp, F.Cu at (95.6, 96.1)
- added D2: LED, LED_THT:LED_D1.8mm_W1.8mm_H2.4mm_Horizontal_O1.27mm_Z4.9mm, F.Cu at (210.9, 149.1)
- added D3: LED, LED_THT:LED_D1.8mm_W1.8mm_H2.4mm_Horizontal_O1.27mm_Z4.9mm, F.Cu at (204.8, 149.1)
- added D4: LED, LED_THT:LED_D1.8mm_W1.8mm_H2.4mm_Horizontal_O1.27mm_Z4.9mm, F.Cu at (192.7, 149.1)
- added D5: LED, LED_THT:LED_D1.8mm_W1.8mm_H2.4mm_Horizontal_O1.27mm_Z4.9mm, F.Cu at (186.7, 149.1)
- added D6: LED, LED_THT:LED_D1.8mm_W1.8mm_H2.4mm_Horizontal_O1.27mm_Z4.9mm, F.Cu at (186.7, 156.0)
- added D7: LED, LED_THT:LED_D1.8mm_W1.8mm_H2.4mm_Horizontal_O1.27mm_Z4.9mm, F.Cu at (198.8, 149.1)
- added D8: LED, LED_THT:LED_D1.8mm_W1.8mm_H2.4mm_Horizontal_O1.27mm_Z4.9mm, F.Cu at (192.7, 156.0)
- added D9: LED, LED_THT:LED_D1.8mm_W1.8mm_H2.4mm_Horizontal_O1.27mm_Z4.9mm, F.Cu at (198.8, 156.0)
- added DIP_16LA1: PAL16L8, Package_DIP:DIP-20_W7.62mm, F.Cu at (104.0, 196.0)
- added DIP_LS244: 74LS244, Package_DIP:DIP-20_W7.62mm, F.Cu at (104.0, 185.2)
- added DIP_Switches1: SW_DIP_x08, Button_Switch_THT:SW_CW_GPTS203211B, F.Cu at (106.1, 174.0)
- added DSUB1: DSUB-9, Connector_Dsub:DSUB-9_Female_Horizontal_P2.77x2.54mm_EdgePinOffset9.40mm, F.Cu at (46.3, 184.2)
- added Display1: 74LS374, Package_DIP:DIP-20_W7.62mm, F.Cu at (186.5, 122.4)
- added Display2: 74LS374, Package_DIP:DIP-20_W7.62mm, F.Cu at (197.4, 122.4)
- added Display3: 74LS374, Package_DIP:DIP-20_W7.62mm, F.Cu at (208.2, 122.4)
- added Display_Decode1: PAL16L8, Package_DIP:DIP-20_W7.62mm, F.Cu at (229.9, 122.4)
- added Display_Decode2: PAL16L8, Package_DIP:DIP-20_W7.62mm, F.Cu at (219.1, 122.4)
- added HighHighSRAM1: CY7C199, Package_DIP:DIP-28_W7.62mm, F.Cu at (168.7, 82.7)
- added HighLowSRAM1: CY7C199, Package_DIP:DIP-28_W7.62mm, F.Cu at (179.6, 82.7)
- added KeyboardSelector1: PAL16L8, Package_DIP:DIP-20_W7.62mm, F.Cu at (36.0, 18.1)
- added LCD_16L8: PAL16L8, Package_DIP:DIP-20_W7.62mm, F.Cu at (122.4, 167.2)
- added LCD_4x20: LCD4x20, Package_DIP:DIP-20_W7.62mm, F.Cu at (122.4, 156.3)
- added LowHighSRAM1: CY7C199, Package_DIP:DIP-28_W7.62mm, F.Cu at (190.4, 82.7)
- added LowLowSRAM1: CY7C199, Package_DIP:DIP-28_W7.62mm, F.Cu at (201.3, 82.7)
- added MAX235: max235cpg, Package_DIP:DIP-24_W7.62mm, F.Cu at (69.0, 128.3)
- added PPI1: 8255, Package_DIP:DIP-40_W15.24mm, F.Cu at (196.3, 77.2)
- added PPI2: 8255, Package_DIP:DIP-40_W15.24mm, F.Cu at (177.9, 77.2)
- added PPI3: 8255, Package_DIP:DIP-40_W15.24mm, F.Cu at (159.5, 77.2)
- added PPI_Decoder1: PAL16L8, Package_DIP:DIP-20_W7.62mm, F.Cu at (141.1, 77.2)
- added PPI_Header1: Conn_01x08_Female, Connector_PinHeader_1.00mm:PinHeader_1x08_P1.00mm_Horizontal, F.Cu at (130.3, 57.6)
- added PPI_Header2: Conn_01x08_Female, Connector_PinHeader_1.00mm:PinHeader_1x08_P1.00mm_Horizontal, F.Cu at (130.3, 77.7)
- added PPI_Header3: Conn_01x08_Female, Connector_PinHeader_1.00mm:PinHeader_1x08_P1.00mm_Horizontal, F.Cu at (141.2, 50.7)
- added PPI_Header4: Conn_01x08_Female, Connector_PinHeader_1.00mm:PinHeader_1x08_P1.00mm_Horizontal, F.Cu at (118.7, 67.7)
- added PPI_Header5: Conn_01x08_Female, Connector_PinHeader_1.00mm:PinHeader_1x08_P1.00mm_Horizontal, F.Cu at (124.5, 67.7)
- added PPI_Header6: Conn_01x08_Female, Connector_PinHeader_1.00mm:PinHeader_1x08_P1.00mm_Horizontal, F.Cu at (130.3, 67.7)
- added PPI_Header7: Conn_01x08_Female, Connector_PinHeader_1.00mm:PinHeader_1x08_P1.00mm_Horizontal, F.Cu at (112.9, 77.7)
- added PPI_Header8: Conn_01x08_Female, Connector_PinHeader_1.00mm:PinHeader_1x08_P1.00mm_Horizontal, F.Cu at (118.7, 77.7)
- added PPI_Header9: Conn_01x08_Female, Connector_PinHeader_1.00mm:PinHeader_1x08_P1.00mm_Horizontal, F.Cu at (124.5, 77.7)
- added Power_1: Conn_01x02_Female, Connector_PinHeader_1.00mm:PinHeader_1x02_P1.00mm_Horizontal, F.Cu at (105.4, 110.5)
- added R1: 10000, Resistor_THT:R_Axial_DIN0204_L3.6mm_D1.6mm_P2.54mm_Vertical, F.Cu at (228.1, 57.2)
- added R10: 330, Resistor_THT:R_Axial_DIN0204_L3.6mm_D1.6mm_P2.54mm_Vertical, F.Cu at (210.2, 155.8)
- added R11: 330, Resistor_THT:R_Axial_DIN0204_L3.6mm_D1.6mm_P2.54mm_Vertical, F.Cu at (222.3, 148.9)
- added R12: 330, Resistor_THT:R_Axial_DIN0204_L3.6mm_D1.6mm_P2.54mm_Vertical, F.Cu at (216.7, 148.9)
- added R13: 330, Resistor_THT:R_Axial_DIN0204_L3.6mm_D1.6mm_P2.54mm_Vertical, F.Cu at (204.6, 159.0)
- added R14: R_Small_US, Resistor_THT:R_Axial_DIN0204_L3.6mm_D1.6mm_P2.54mm_Vertical, F.Cu at (109.8, 158.9)
- added R15: R_Small_US, Resistor_THT:R_Axial_DIN0204_L3.6mm_D1.6mm_P2.54mm_Vertical, F.Cu at (117.1, 168.8)
- added R16: R_Small_US, Resistor_THT:R_Axial_DIN0204_L3.6mm_D1.6mm_P2.54mm_Vertical, F.Cu at (123.4, 174.4)
- added R17: R_Small_US, Resistor_THT:R_Axial_DIN0204_L3.6mm_D1.6mm_P2.54mm_Vertical, F.Cu at (103.5, 153.3)
- added R18: R_Small_US, Resistor_THT:R_Axial_DIN0204_L3.6mm_D1.6mm_P2.54mm_Vertical, F.Cu at (120.2, 174.4)
- added R19: R_Small_US, Resistor_THT:R_Axial_DIN0204_L3.6mm_D1.6mm_P2.54mm_Vertical, F.Cu at (103.5, 158.9)
- added R20: R_Small_US, Resistor_THT:R_Axial_DIN0204_L3.6mm_D1.6mm_P2.54mm_Vertical, F.Cu at (106.7, 158.9)
- added R21: R_Small_US, Resistor_THT:R_Axial_DIN0204_L3.6mm_D1.6mm_P2.54mm_Vertical, F.Cu at (117.1, 174.4)
- added R4: R, Resistor_THT:R_Axial_DIN0204_L3.6mm_D1.6mm_P2.54mm_Vertical, F.Cu at (252.3, 121.9)
- added R5: R, Resistor_THT:R_Axial_DIN0204_L3.6mm_D1.6mm_P2.54mm_Vertical, F.Cu at (204.6, 155.8)
- added R6: 330, Resistor_THT:R_Axial_DIN0204_L3.6mm_D1.6mm_P2.54mm_Vertical, F.Cu at (222.3, 152.1)
- added R7: 330, Resistor_THT:R_Axial_DIN0204_L3.6mm_D1.6mm_P2.54mm_Vertical, F.Cu at (216.7, 152.1)
- added R8: 330, Resistor_THT:R_Axial_DIN0204_L3.6mm_D1.6mm_P2.54mm_Vertical, F.Cu at (233.5, 148.9)
- added R9: 330, Resistor_THT:R_Axial_DIN0204_L3.6mm_D1.6mm_P2.54mm_Vertical, F.Cu at (227.9, 148.9)
- added Resistor10K1: Resistor, Resistor_THT:R_Axial_DIN0204_L3.6mm_D1.6mm_P2.54mm_Vertical, F.Cu at (62.2, 157.5)
- added SIXTEENL8: PAL16L8, Package_DIP:DIP-20_W7.62mm, F.Cu at (58.4, 129.5)
- added SRAMSelector1: PAL16L8, Package_DIP:DIP-20_W7.62mm, F.Cu at (212.1, 82.7)
- added SW10: SW_Push, Button_Switch_THT:SW_PUSH-12mm, F.Cu at (69.5, 74.5)
- added SW11: SW_Push, Button_Switch_THT:SW_PUSH-12mm, F.Cu at (87.9, 60.9)
- added SW12: SW_Push, Button_Switch_THT:SW_PUSH-12mm, F.Cu at (105.0, 47.4)
- added SW13: SW_Push, Button_Switch_THT:SW_PUSH-12mm, F.Cu at (70.8, 47.4)
- added SW14: SW_Push, Button_Switch_THT:SW_PUSH-12mm, F.Cu at (98.8, 20.3)
- added SW15: SW_Push, Button_Switch_THT:SW_PUSH-12mm, F.Cu at (18.3, 72.7)
- added SW16: SW_Push, Button_Switch_THT:SW_PUSH-12mm, F.Cu at (47.6, 20.3)
- added SW17: SW_Push, Button_Switch_THT:SW_PUSH-12mm, F.Cu at (35.4, 74.4)
- added SW18: SW_Push, Button_Switch_THT:SW_PUSH-12mm, F.Cu at (53.8, 60.9)
- added SW19: SW_Push, Button_Switch_THT:SW_PUSH-12mm, F.Cu at (70.8, 33.8)
- added SW20: SW_Push, Button_Switch_THT:SW_PUSH-12mm, F.Cu at (81.7, 20.3)
- added SW21: SW_Push, Button_Switch_THT:SW_PUSH-12mm, F.Cu at (64.6, 20.3)
- added SW22: SW_Push, Button_Switch_THT:SW_PUSH-12mm, F.Cu at (36.7, 60.8)
- added SW23: SW_Push, Button_Switch_THT:SW_PUSH-12mm, F.Cu at (53.8, 47.4)
- added SW24: SW_Push, Button_Switch_THT:SW_PUSH-12mm, F.Cu at (53.8, 33.8)
- added SW25: SW_Push, Button_Switch_THT:SW_PUSH-12mm, F.Cu at (36.7, 47.3)
- added SW3: SW_Push, Button_Switch_THT:SW_PUSH-12mm, F.Cu at (203.8, 45.6)
- added SW4: SW_Push, Button_Switch_THT:SW_PUSH-12mm, F.Cu at (87.9, 33.8)
- added SW5: SW_Push, Button_Switch_THT:SW_PUSH-12mm, F.Cu at (52.4, 74.5)
- added SW6: SW_Push, Button_Switch_THT:SW_PUSH-12mm, F.Cu at (70.8, 60.9)
- added SW7: SW_Push, Button_Switch_THT:SW_PUSH-12mm, F.Cu at (87.9, 47.4)
- added SW8: SW_Push, Button_Switch_THT:SW_PUSH-12mm, F.Cu at (115.8, 20.3)
- added SW9: SW_Push, Button_Switch_THT:SW_PUSH-12mm, F.Cu at (105.0, 33.8)
- added Seven_Seg1: MAN71A, Display_7Segment:MAN71A, F.Cu at (241.3, 122.9)
- added Seven_Seg2: MAN71A, Display_7Segment:MAN71A, F.Cu at (241.3, 143.2)
- added U12: 74LS04, Package_DIP:DIP-14_W7.62mm, F.Cu at (161.8, 177.3)
- added U19: 74AHC1G08, Package_DIP:DIP-5-6_W7.62mm, F.Cu at (233.8, 102.1)
- added U20: 74AHC1G08, Package_DIP:DIP-5-6_W7.62mm, F.Cu at (223.0, 102.1)
- added U21: 74AHC1G08, Package_DIP:DIP-5-6_W7.62mm, F.Cu at (212.1, 109.7)
- added U41: 28F010, Package_DIP:DIP-32_W7.62mm, F.Cu at (80.0, 108.0)
- added U9: 74LS138, Package_DIP:DIP-16_W7.62mm, F.Cu at (151.0, 177.3)
- added UART1: 16550, Package_DIP:DIP-40_W15.24mm, F.Cu at (14.0, 176.5)
- U1: value 8086_Min_Mode -> 74AHC1G08; footprint Package_DIP:DIP-40_W15.24mm -> Package_DIP:DIP-5-6_W7.62mm
- U17, U18: value 74LVC1GU04DRL -> 74LS04; footprint Package_TO_SOT_SMD:SOT-553 -> Package_DIP:DIP-14_W7.62mm
- moved U1 125.0 mm to (223.0, 111.3)
- moved U17 98.1 mm to (233.8, 82.7)
- moved U18 83.9 mm to (223.0, 82.7)
Connections:
- U1 pad 1: GND -> Net-(U1-Pad1)
- U1 pad 2: /8086/AD14 -> Net-(U1-Pad2)
- U1 pad 3: /8086/AD13 -> GND
- U1 pad 4: /8086/AD12 -> /SRAM/CE00
- U1 pad 6: /8086/AD10 -> (no net)
- U17 pad 2: Net-(U16-Pad15) -> Net-(U1-Pad2)
- U17 pad 3: Net-(U17-Pad3) -> (no net)
- U17 pad 4: Net-(U17-Pad4) -> (no net)
- U17 pad 5: Net-(U17-Pad5) -> (no net)
- U18 pad 2: Net-(U16-Pad14) -> Net-(U1-Pad1)
- U18 pad 3: Net-(U18-Pad3) -> (no net)
- U18 pad 4: Net-(U18-Pad4) -> (no net)
- U18 pad 5: Net-(U18-Pad5) -> (no net)
