File: Final/Final.sch (KiCad schematic (older format))
At the start: 0 parts

Commit message: Stuffs
Changed lines of the file:
@@
 F28 "A10" I R 1950 4850 50
 F29 "A2" I R 1950 4050 50
+F30 "CLK" I L 900 4200 50
 $EndSheet
 $Sheet
@@
 Text Label 7300 5100 0    50   ~ 0
 ~WR
+Wire Wire Line
+	900  4200 800  4200
+Text Label 800  4200 2    50   ~ 0
+CLK
 $EndSCHEMATC
