File: Final/16550(FINAL).sch (KiCad schematic (older format))
At the start: 1 part

Commit message: New stuff
Parts:
- gave numbers to parts that had none: 1
Changed lines of the file:
@@
 $EndDescr
 $Comp
-L Interface_UART:16550 U?
+L Interface_UART:16550 U30
 U 1 1 6077B6BD
 P 5100 3650
-F 0 "U?" H 5100 5531 50  0000 C CNN
+F 0 "U30" H 5100 5531 50  0000 C CNN
 F 1 "16550" H 5100 5440 50  0000 C CNN
 F 2 "Package_DIP:DIP-40_W15.24mm" H 5100 3650 50  0001 C CIN
@@
 ~WR
 $Comp
-L power:GND1 #PWR?
+L power:GND1 #PWR052
 U 1 1 6077FCC2
 P 3850 5600
-F 0 "#PWR?" H 3850 5350 50  0001 C CNN
+F 0 "#PWR052" H 3850 5350 50  0001 C CNN
 F 1 "GND1" H 3855 5427 50  0000 C CNN
 F 2 "" H 3850 5600 50  0001 C CNN
@@
 Connection ~ 5100 1950
 $Comp
-L power:VCC #PWR?
+L power:VCC #PWR053
 U 1 1 608C1403
 P 5100 1900
-F 0 "#PWR?" H 5100 1750 50  0001 C CNN
+F 0 "#PWR053" H 5100 1750 50  0001 C CNN
 F 1 "VCC" H 5115 2073 50  0000 C CNN
 F 2 "" H 5100 1900 50  0001 C CNN

Commit message: For Commenting
Connections:
- net DDIS: no longer names the net of U30.23 (DDIS)
- net ~OUT1: no longer names the net of U30.34 (~OUT1~)
- net ~OUT2: no longer names the net of U30.31 (~OUT2~)
- net ~RXRDY: no longer names the net of U30.29 (~RXRDY~)
- net ~TXRDY: no longer names the net of U30.24 (~TXRDY~)
- no-connect marks 0 -> 5
Changed lines of the file:
@@
 $Descr A4 11693 8268
 encoding utf-8
-Sheet 10 14
+Sheet 11 16
 Title ""
 Date ""
@@
 Text HLabel 6100 2750 2    50   Input ~ 0
 ~CTS
-Text HLabel 6100 3050 2    50   Output ~ 0
-~OUT1
 Text HLabel 6100 3150 2    50   Output ~ 0
 ~DTR
 Text HLabel 6100 3250 2    50   Output ~ 0
 ~RTS
-Text HLabel 6100 3350 2    50   Output ~ 0
-~OUT2
 Text HLabel 6100 3850 2    50   Input ~ 0
 SIN
 Text HLabel 6100 3950 2    50   Output ~ 0
 SOUT
-Text HLabel 6100 4250 2    50   Output ~ 0
-~RXRDY
-Text HLabel 6100 4350 2    50   Output ~ 0
-~TXRDY
-Text HLabel 6100 4450 2    50   Output ~ 0
-DDIS
 Wire Wire Line
 	6100 4850 6150 4850
@@
 Wire Wire Line
 	5100 1900 5100 1950
+NoConn ~ 6100 4250
+NoConn ~ 6100 4350
+NoConn ~ 6100 4450
+NoConn ~ 6100 3050
+NoConn ~ 6100 3350
 $EndSCHEMATC

Commit message: Final?
Parts:
- added DSUB1: DSUB-9, DSUB-9, symbol DSUB-9:DSUB-9
- added MAX235: max235cpg, max235cpg, symbol max235cpg:max235cpg
- added Resistor10K1: Resistor, symbol Device:R
- added SIXTEENL8: PAL16L8, symbol Logic_Programmable:PAL16L8
- renumbered U30 to UART1
Connections:
- net A0: now also SIXTEENL8.1 (I1)
- net A1: now also SIXTEENL8.2 (I2)
- net A2: now also SIXTEENL8.3 (I3)
- net SIN: now also MAX235.6 (R2OUT)
- net SOUT: now also MAX235.8 (T1IN)
- net VCC: now also MAX235.12 (VCC), Resistor10K1.1, SIXTEENL8.20 (VCC); no longer UART1.13 (CS1), UART1.39 (~RI~)
- net ~CTS: now also MAX235.17 (R4OUT)
- net CLK renamed PCLK
- net GND1 renamed GND
- net GND: now also DSUB1.5 (GND), MAX235.11 (GND), MAX235.20 (*EN), MAX235.21 (SHDN), SIXTEENL8.10 (GND); no longer UART1.14 (~CS2~)
- net IO~M: no longer names the net of UART1.12 (CS0)
- net IO~M: now also UART1.13 (CS1), Resistor10K1.2
- net XOUT: no longer names the net of UART1.17 (XOUT)
- net ~DCD renamed DCD
- net DCD: now also MAX235.9 (R1OUT)
- net ~DSR renamed DSR
- net DSR: now also MAX235.23 (R3OUT)
- net ~DTR renamed DTR
- net DTR: now also MAX235.7 (T2IN)
- net ~RTS renamed RTS
- net RTS: now also MAX235.15 (T3IN)
- new net: SIXTEENL8.19 (IO1), UART1.14 (~CS2~)
- new net A11: SIXTEENL8.18 (IO2)
- new net A12: SIXTEENL8.17 (I03)
- new net A13: SIXTEENL8.16 (IO4)
- new net A14: SIXTEENL8.15 (IO5)
- new net A15: SIXTEENL8.14 (IO6)
- new net A3: SIXTEENL8.4 (I4)
- new net A4: SIXTEENL8.5 (I5)
- new net A5: SIXTEENL8.6 (I6)
- new net A6: SIXTEENL8.7 (I7)
- new net A7: SIXTEENL8.8 (I8)
- new net A8: SIXTEENL8.9 (I9)
- new net A9: SIXTEENL8.11 (I10)
- new net CTS: DSUB1.8 (CTS), MAX235.18 (R4IN)
- new net DCD9: DSUB1.1 (DCD), MAX235.10 (R1IN)
- new net DSR9: DSUB1.6 (DSR), MAX235.24 (R3IN)
- new net DTR9: DSUB1.4 (DTR), MAX235.4 (T2OUT)
- new net RI: MAX235.14 (R5OUT), UART1.39 (~RI~)
- new net RI9: DSUB1.9 (RI), MAX235.13 (R5IN)
- new net RTS9: DSUB1.7 (RTS), MAX235.2 (T3OUT)
- new net RXD: DSUB1.2 (RDX), MAX235.5 (R2IN)
- new net TXD: DSUB1.3 (TDX), MAX235.3 (T1OUT)
- no-connect marks 5 -> 12

Commit message: Final..I Hope
Parts:
- DSUB1: footprint DSUB-9 -> (none)
- MAX235: footprint max235cpg -> (none)
Changed lines of the file:
@@
 F 0 "MAX235" H 9000 4437 60  0000 C CNN
 F 1 "max235cpg" H 9000 4331 60  0000 C CNN
-F 2 "max235cpg" H 9000 4290 60  0001 C CNN
+F 2 "" H 9000 4290 60  0001 C CNN
 F 3 "" H 7700 4050 60  0000 C CNN
 	1    7700 4050
@@
 F 0 "DSUB1" H 5778 5553 60  0000 L CNN
 F 1 "DSUB-9" H 5778 5447 60  0000 L CNN
-F 2 "DSUB-9" H 5550 5540 60  0001 C CNN
+F 2 "" H 5550 5540 60  0001 C CNN
 F 3 "" H 4950 5900 60  0000 C CNN
 	1    4950 5900

Commit message: Hopefully the board is here
Parts:
- DSUB1: footprint (none) -> Connector_Dsub:DSUB-9_Female_Horizontal_P2.77x2.54mm_EdgePinOffset9.40mm
- MAX235: footprint (none) -> Package_DIP:DIP-24_W7.62mm
- Resistor10K1: footprint (none) -> Resistor_THT:R_Axial_DIN0204_L3.6mm_D1.6mm_P2.54mm_Vertical
- SIXTEENL8: footprint (none) -> Package_DIP:DIP-20_W7.62mm
Changed lines of the file:
@@
 F 0 "SIXTEENL8" H 2250 6981 50  0000 C CNN
 F 1 "PAL16L8" H 2250 6890 50  0000 C CNN
-F 2 "" H 2250 6100 50  0001 C CNN
+F 2 "Package_DIP:DIP-20_W7.62mm" H 2250 6100 50  0001 C CNN
 F 3 "" H 2250 6100 50  0001 C CNN
 	1    2250 6100
@@
 F 0 "MAX235" H 9000 4437 60  0000 C CNN
 F 1 "max235cpg" H 9000 4331 60  0000 C CNN
-F 2 "" H 9000 4290 60  0001 C CNN
+F 2 "Package_DIP:DIP-24_W7.62mm" H 9000 4290 60  0001 C CNN
 F 3 "" H 7700 4050 60  0000 C CNN
 	1    7700 4050
@@
 F 0 "Resistor10K1" H 3370 3346 50  0000 L CNN
 F 1 "Resistor" H 3370 3255 50  0000 L CNN
-F 2 "" V 3230 3300 50  0001 C CNN
+F 2 "Resistor_THT:R_Axial_DIN0204_L3.6mm_D1.6mm_P2.54mm_Vertical" V 3230 3300 50  0001 C CNN
 F 3 "~" H 3300 3300 50  0001 C CNN
 	1    3300 3300
@@
 F 0 "DSUB1" H 5778 5553 60  0000 L CNN
 F 1 "DSUB-9" H 5778 5447 60  0000 L CNN
-F 2 "" H 5550 5540 60  0001 C CNN
+F 2 "Connector_Dsub:DSUB-9_Female_Horizontal_P2.77x2.54mm_EdgePinOffset9.40mm" H 5550 5540 60  0001 C CNN
 F 3 "" H 4950 5900 60  0000 C CNN
 	1    4950 5900
