File: Final/8086(FINAL).sch (KiCad schematic (older format))
At the start: 11 parts, among them SW1 SW_Push, U1 8086_Min_Mode, U2 74LS373, U3 74LS373, U4 74LS373, U5 74LS244, U6 74LS245, U7 74LS245

Commit message: New stuff
Connections:
- net GNDREF is gone; now on net GND: C1.2, SW1.1
- net M~IO: no longer U1.28 (M/~IO~), U5.2 (I0a)
- net ~RD: no longer U1.32 (~RD~), U5.6 (I2a)
- net ~WR: no longer U1.29 (~WR~), U5.4 (I1a)
- new net IO: U1.28 (M/~IO~), U5.2 (I0a)
- new net Read: U1.32 (~RD~), U5.6 (I2a)
- new net Write: U1.29 (~WR~), U5.4 (I1a)
Changed lines of the file:
@@
 	3900 1000 4700 1000
 $Comp
-L power:VCC #PWR0101
+L power:VCC #PWR05
 U 1 1 60762F72
 P 4700 1000
-F 0 "#PWR0101" H 4700 850 50  0001 C CNN
+F 0 "#PWR05" H 4700 850 50  0001 C CNN
 F 1 "VCC" H 4715 1173 50  0000 C CNN
 F 2 "" H 4700 1000 50  0001 C CNN
@@
 AD0
 Text Label 4850 2000 0    50   ~ 0
-AD[0:19]
+AD[0..19]
 Text Label 4600 2250 0    50   ~ 0
 AD1
@@
 	2200 2000 2250 2000
 $Comp
-L power:VCC #PWR0102
+L power:VCC #PWR01
 U 1 1 60778894
 P 1600 2350
-F 0 "#PWR0102" H 1600 2200 50  0001 C CNN
+F 0 "#PWR01" H 1600 2200 50  0001 C CNN
 F 1 "VCC" H 1615 2523 50  0000 C CNN
 F 2 "" H 1600 2350 50  0001 C CNN
@@
 	1    0    0    -1
 $EndComp
-$Comp
-L power:GNDREF #PWR0103
-U 1 1 60779236
-P 2200 1350
-F 0 "#PWR0103" H 2200 1100 50  0001 C CNN
-F 1 "GNDREF" H 2205 1177 50  0000 C CNN
-F 2 "" H 2200 1350 50  0001 C CNN
-F 3 "" H 2200 1350 50  0001 C CNN
-	1    2200 1350
-	-1   0    0    1
-$EndComp
-Connection ~ 2200 1350
 Wire Wire Line
 	1800 1800 1800 2350
@@
 	6850 1650 6950 1750
 Text Label 6850 850  0    50   ~ 0
-AD[0:19]
+AD[0..19]
 Text HLabel 8250 1750 2    50   Output ~ 0
 A7
@@
 AD6
 $Comp
-L power:VCC #PWR0104
+L power:VCC #PWR09
 U 1 1 607B535A
 P 8650 700
-F 0 "#PWR0104" H 8650 550 50  0001 C CNN
+F 0 "#PWR09" H 8650 550 50  0001 C CNN
 F 1 "VCC" H 8665 873 50  0000 C CNN
 F 2 "" H 8650 700 50  0001 C CNN
@@
 ALE
 $Comp
-L power:GND #PWR0105
+L power:GND #PWR07
 U 1 1 607CF9AE
 P 7450 4300
-F 0 "#PWR0105" H 7450 4050 50  0001 C CNN
+F 0 "#PWR07" H 7450 4050 50  0001 C CNN
 F 1 "GND" H 7455 4127 50  0000 C CNN
 F 2 "" H 7450 4300 50  0001 C CNN
@@
 	7250 2350 7250 2050
 $Comp
-L power:GND #PWR0106
+L power:GND #PWR06
 U 1 1 607D6379
 P 7450 2350
-F 0 "#PWR0106" H 7450 2100 50  0001 C CNN
+F 0 "#PWR06" H 7450 2100 50  0001 C CNN
 F 1 "GND" H 7455 2177 50  0000 C CNN
 F 2 "" H 7450 2350 50  0001 C CNN
@@
 	7250 6200 7250 5900
 $Comp
-L power:GND #PWR0107
+L power:GND #PWR08
 U 1 1 607DB402
 P 7450 6200
-F 0 "#PWR0107" H 7450 5950 50  0001 C CNN
+F 0 "#PWR08" H 7450 5950 50  0001 C CNN
 F 1 "GND" H 7455 6027 50  0000 C CNN
 F 2 "" H 7450 6200 50  0001 C CNN
@@
 Connection ~ 9650 2050
 $Comp
-L power:GND #PWR0108
+L power:GND #PWR010
 U 1 1 60803BF6
 P 9900 2350
-F 0 "#PWR0108" H 9900 2100 50  0001 C CNN
+F 0 "#PWR010" H 9900 2100 50  0001 C CNN
 F 1 "GND" H 9905 2177 50  0000 C CNN
 F 2 "" H 9900 2350 50  0001 C CNN
@@
 	4600 4550 4750 4550
 Text Label 4750 4350 0    50   ~ 0
-M~IO
-Text Label 4750 4450 0    50   ~ 0
-~WR
+IO
 Text Label 4750 4550 0    50   ~ 0
-~RD
+Read
 Text Label 9650 1050 2    50   ~ 0
-M~IO
+IO
 Text Label 9650 1150 2    50   ~ 0
-~WR
+Write
 Text Label 9650 1250 2    50   ~ 0
-~RD
+Read
 Text HLabel 10650 1050 2    50   Output ~ 0
 M~IO
@@
 	9650 5600 9350 5600
 Text Label 9250 2850 0    50   ~ 0
-AD[0:15]
+AD[0..15]
 Text Label 4750 1750 0    50   ~ 0
 ~DEN
@@
 	10150 4350 10400 4350
 $Comp
-L power:GND #PWR0109
+L power:GND #PWR011
 U 1 1 6083EB10
 P 10150 6200
-F 0 "#PWR0109" H 10150 5950 50  0001 C CNN
+F 0 "#PWR011" H 10150 5950 50  0001 C CNN
 F 1 "GND" H 10155 6027 50  0000 C CNN
 F 2 "" H 10150 6200 50  0001 C CNN
@@
 $EndComp
 $Comp
-L power:GND #PWR0110
+L power:GND #PWR012
 U 1 1 6083F138
 P 10400 4350
-F 0 "#PWR0110" H 10400 4100 50  0001 C CNN
+F 0 "#PWR012" H 10400 4100 50  0001 C CNN
 F 1 "GND" H 10405 4177 50  0000 C CNN
 F 2 "" H 10400 4350 50  0001 C CNN
@@
 Text HLabel 10650 5000 2    50   Output ~ 0
 D9
-Text HLabel 10650 4900 2    50   Output ~ 0
+Text HLabel 10750 4900 2    50   Output ~ 0
 D8
 Text Label 3050 2050 2    50   ~ 0
@@
 READY
 $Comp
-L power:GND #PWR0111
+L power:GND #PWR03
 U 1 1 6085F789
 P 3800 4950
-F 0 "#PWR0111" H 3800 4700 50  0001 C CNN
+F 0 "#PWR03" H 3800 4700 50  0001 C CNN
 F 1 "GND" H 3805 4777 50  0000 C CNN
 F 2 "" H 3800 4950 50  0001 C CNN
@@
 $EndComp
 $Comp
-L power:GND #PWR0112
+L power:GND #PWR04
 U 1 1 60860099
 P 4000 4950
-F 0 "#PWR0112" H 4000 4700 50  0001 C CNN
+F 0 "#PWR04" H 4000 4700 50  0001 C CNN
 F 1 "GND" H 4005 4777 50  0000 C CNN
 F 2 "" H 4000 4950 50  0001 C CNN
@@
 F5 "PCLK" O R 1750 5600 50
 $EndSheet
-Wire Wire Line
-	1750 5150 1850 5150
-Wire Wire Line
-	1750 5300 1850 5300
 Text Label 1850 5150 0    50   ~ 0
 CLK
 Text Label 1850 5300 0    50   ~ 0
 RESET
-Wire Wire Line
-	1750 5450 1850 5450
 Text Label 1850 5450 0    50   ~ 0
 READY
 Wire Wire Line
 	1750 5600 1850 5600
+Text HLabel 1850 5600 2    50   Output ~ 0
+PCLK
+Wire Wire Line
+	1750 5450 1850 5450
+Wire Wire Line
+	1750 5300 2200 5300
+Text HLabel 2200 5300 2    50   Output ~ 0
+RESET
+Wire Wire Line
+	1750 5150 2200 5150
+Text HLabel 2200 5150 2    50   Output ~ 0
+CLK
+Text Label 4750 4450 0    50   ~ 0
+Write
+$Comp
+L power:GND #PWR0101
+U 1 1 60B7CA3A
+P 2200 1350
+F 0 "#PWR0101" H 2200 1100 50  0001 C CNN
+F 1 "GND" H 2205 1177 50  0000 C CNN
+F 2 "" H 2200 1350 50  0001 C CNN
+F 3 "" H 2200 1350 50  0001 C CNN
+	1    2200 1350
+	-1   0    0    1
+$EndComp
+Connection ~ 2200 1350
+Wire Wire Line
+	10650 4900 10750 4900
 Wire Bus Line
 	9250 2850 9250 5500
@@
 Wire Bus Line
 	4850 2000 4850 4050
-Text HLabel 1850 5600 2    50   Output ~ 0
-PCLK
 $EndSCHEMATC

Commit message: For Commenting
Parts:
- D1: value DIODE -> CPU_Diode
- renumbered U1 to CPU, C1 to CPU_Capacitor, R1 to CPU_Resistor, SW1 to CPU_Switch
Connections:
- net A16: no longer CPU.38 (A16/S3), U4.3 (D0)
- net A17: no longer CPU.37 (A17/S4), U4.4 (D1)
- net A18: no longer CPU.36 (A18/S5), U4.7 (D2)
- net A19: no longer CPU.35 (A19/S6), U4.8 (D3)
- net VCC: now also CPU.33 (MN/~MX~)
- new net S3: CPU.38 (A16/S3), U4.3 (D0)
- new net S4: CPU.37 (A17/S4), U4.4 (D1)
- new net S5: CPU.36 (A18/S5), U4.7 (D2)
- new net S6: CPU.35 (A19/S6), U4.8 (D3)
- no-connect marks 22 -> 21
Changed lines of the file:
@@
 $Descr A4 11693 8268
 encoding utf-8
-Sheet 2 14
+Sheet 2 16
 Title ""
 Date ""
@@
 $EndDescr
 $Comp
-L Switch:SW_Push SW1
+L Switch:SW_Push CPU_Switch
 U 1 1 607622DA
 P 2200 1700
-F 0 "SW1" V 2154 1848 50  0000 L CNN
+F 0 "CPU_Switch" V 2154 1848 50  0000 L CNN
 F 1 "SW_Push" V 2245 1848 50  0000 L CNN
 F 2 "" H 2200 1900 50  0001 C CNN
@@
 AD15
 Text Label 4600 3850 0    50   ~ 0
-A16
+S3
 Text Label 4600 3950 0    50   ~ 0
-A17
+S4
 Text Label 4600 4050 0    50   ~ 0
-A18
+S5
 Text Label 4600 4150 0    50   ~ 0
-A19
+S6
 Wire Wire Line
 	2200 1500 2200 1350
@@
 	1800 1800 1800 2350
 $Comp
-L Device:CP1_Small C1
+L Device:CP1_Small CPU_Capacitor
 U 1 1 6077E7C3
 P 1800 1700
-F 0 "C1" H 1891 1654 50  0000 L CNN
+F 0 "CPU_Capacitor" H 1891 1654 50  0000 L CNN
 F 1 "CP1_Small" H 1891 1745 50  0000 L CNN
 F 2 "" H 1800 1700 50  0001 C CNN
@@
 P 2400 2350
 F 0 "D1" H 2400 2085 50  0000 C CNN
-F 1 "DIODE" H 2400 2176 50  0000 C CNN
+F 1 "CPU_Diode" H 2400 2176 50  0000 C CNN
 F 2 "" H 2400 2350 50  0001 C CNN
 F 3 "~" H 2400 2350 50  0001 C CNN
@@
 Connection ~ 1800 2350
 $Comp
-L Device:R_US R1
+L Device:R_US CPU_Resistor
 U 1 1 607846D6
 P 2400 2000
-F 0 "R1" V 2195 2000 50  0000 C CNN
+F 0 "CPU_Resistor" V 2195 2000 50  0000 C CNN
 F 1 "R_US" V 2286 2000 50  0000 C CNN
 F 2 "" V 2440 1990 50  0001 C CNN
@@
 	6850 4800 6950 4900
 Text Label 7000 4900 0    50   ~ 0
-A16
+S3
 Entry Wire Line
 	6850 4900 6950 5000
 Text Label 7000 5000 0    50   ~ 0
-A17
+S4
 Entry Wire Line
 	6850 5000 6950 5100
 Text Label 7000 5100 0    50   ~ 0
-A18
+S5
 Entry Wire Line
 	6850 5100 6950 5200
 Text Label 7000 5200 0    50   ~ 0
-A19
+S6
 NoConn ~ 7250 5300
 NoConn ~ 7250 5400
@@
 Text HLabel 10650 5000 2    50   Output ~ 0
 D9
-Text HLabel 10750 4900 2    50   Output ~ 0
+Text HLabel 10650 4900 2    50   Output ~ 0
 D8
 Text Label 3050 2050 2    50   ~ 0
@@
 NoConn ~ 3200 3350
 NoConn ~ 3200 3550
-NoConn ~ 3200 4650
-Text HLabel 4600 1950 2    50   Output ~ 0
+Text HLabel 4600 1950 2    50   3State ~ 0
 ~BHE~S7
 Text Label 3050 1850 2    50   ~ 0
@@
 	3200 1650 3050 1650
 $Comp
-L MCU_Intel:8086_Min_Mode U1
+L MCU_Intel:8086_Min_Mode CPU
 U 1 1 60761E58
 P 3900 3150
-F 0 "U1" H 3900 5131 50  0000 C CNN
+F 0 "CPU" H 3900 5131 50  0000 C CNN
 F 1 "8086_Min_Mode" H 3900 5040 50  0000 C CNN
 F 2 "Package_DIP:DIP-40_W15.24mm" H 3950 3250 50  0001 C CIN
@@
 $EndComp
 Connection ~ 2200 1350
-Wire Wire Line
-	10650 4900 10750 4900
 Wire Bus Line
 	9250 2850 9250 5500
@@
 Wire Bus Line
 	4850 2000 4850 4050
+$Comp
+L power:VCC #PWR0120
+U 1 1 61629C6A
+P 3200 4650
+F 0 "#PWR0120" H 3200 4500 50  0001 C CNN
+F 1 "VCC" V 3215 4777 50  0000 L CNN
+F 2 "" H 3200 4650 50  0001 C CNN
+F 3 "" H 3200 4650 50  0001 C CNN
+	1    3200 4650
+	0    -1   -1   0
+$EndComp
 $EndSCHEMATC

Commit message: Stuffs
Parts:
- renumbered U2 to CPU_ADecode1, U3 to CPU_ADecode2, U4 to CPU_ADecode3, U6 to CPU_DDecode1, U7 to CPU_DDecode2, U5 to CPU_IO/WR
Changed lines of the file:
@@
 A1
 $Comp
-L 74xx:74LS373 U2
+L 74xx:74LS373 CPU_ADecode1
 U 1 1 607721F2
 P 7750 1550
-F 0 "U2" H 7750 2531 50  0000 C CNN
+F 0 "CPU_ADecode1" H 7750 2531 50  0000 C CNN
 F 1 "74LS373" H 7750 2440 50  0000 C CNN
 F 2 "" H 7750 1550 50  0001 C CNN
@@
 A0
 $Comp
-L 74xx:74LS373 U3
+L 74xx:74LS373 CPU_ADecode2
 U 1 1 607A162B
 P 7750 3500
-F 0 "U3" H 7750 4481 50  0000 C CNN
+F 0 "CPU_ADecode2" H 7750 4481 50  0000 C CNN
 F 1 "74LS373" H 7750 4390 50  0000 C CNN
 F 2 "" H 7750 3500 50  0001 C CNN
@@
 	6950 5000 7250 5000
 $Comp
-L 74xx:74LS373 U4
+L 74xx:74LS373 CPU_ADecode3
 U 1 1 607A2E66
 P 7750 5400
-F 0 "U4" H 7750 6381 50  0000 C CNN
+F 0 "CPU_ADecode3" H 7750 6381 50  0000 C CNN
 F 1 "74LS373" H 7750 6290 50  0000 C CNN
 F 2 "" H 7750 5400 50  0001 C CNN
@@
 A16
 $Comp
-L 74xx:74LS244 U5
+L 74xx:74LS244 CPU_IO/WR
 U 1 1 607EFA33
 P 10150 1550
-F 0 "U5" H 10150 2531 50  0000 C CNN
+F 0 "CPU_IO/WR" H 10150 2531 50  0000 C CNN
 F 1 "74LS244" H 10150 2440 50  0000 C CNN
 F 2 "" H 10150 1550 50  0001 C CNN
@@
 ~RD
 $Comp
-L 74xx:74LS245 U6
+L 74xx:74LS245 CPU_DDecode1
 U 1 1 60814065
 P 10150 3550
-F 0 "U6" H 10150 4531 50  0000 C CNN
+F 0 "CPU_DDecode1" H 10150 4531 50  0000 C CNN
 F 1 "74LS245" H 10150 4440 50  0000 C CNN
 F 2 "" H 10150 3550 50  0001 C CNN
@@
 $EndComp
 $Comp
-L 74xx:74LS245 U7
+L 74xx:74LS245 CPU_DDecode2
 U 1 1 608151DF
 P 10150 5400
-F 0 "U7" H 10150 6381 50  0000 C CNN
+F 0 "CPU_DDecode2" H 10150 6381 50  0000 C CNN
 F 1 "74LS245" H 10150 6290 50  0000 C CNN
 F 2 "" H 10150 5400 50  0001 C CNN

Commit message: Final?
Parts:
- renumbered CPU to CPU1, CPU_Capacitor to CPU_Capacitor1, CPU_IO/WR to CPU_IO/WR1, CPU_Resistor to CPU_Resistor1, CPU_Switch to CPU_Switch1
Changed lines of the file:
@@
 $EndDescr
 $Comp
-L Switch:SW_Push CPU_Switch
+L Switch:SW_Push CPU_Switch1
 U 1 1 607622DA
 P 2200 1700
-F 0 "CPU_Switch" V 2154 1848 50  0000 L CNN
+F 0 "CPU_Switch1" V 2154 1848 50  0000 L CNN
 F 1 "SW_Push" V 2245 1848 50  0000 L CNN
 F 2 "" H 2200 1900 50  0001 C CNN
@@
 Wire Wire Line
 	3900 1350 3900 1000
-Wire Wire Line
-	3900 1000 4700 1000
 $Comp
 L power:VCC #PWR05
@@
 	2200 1500 2200 1350
 Wire Wire Line
-	2200 1350 1800 1350
-Wire Wire Line
 	1800 1350 1800 1600
-Wire Wire Line
-	1600 2350 1800 2350
 Wire Wire Line
 	2200 2000 2250 2000
@@
 	1800 1800 1800 2350
 $Comp
-L Device:CP1_Small CPU_Capacitor
+L Device:CP1_Small CPU_Capacitor1
 U 1 1 6077E7C3
 P 1800 1700
-F 0 "CPU_Capacitor" H 1891 1654 50  0000 L CNN
+F 0 "CPU_Capacitor1" H 1891 1654 50  0000 L CNN
 F 1 "CP1_Small" H 1891 1745 50  0000 L CNN
 F 2 "" H 1800 1700 50  0001 C CNN
@@
 Connection ~ 1800 2350
 $Comp
-L Device:R_US CPU_Resistor
+L Device:R_US CPU_Resistor1
 U 1 1 607846D6
 P 2400 2000
-F 0 "CPU_Resistor" V 2195 2000 50  0000 C CNN
+F 0 "CPU_Resistor1" V 2195 2000 50  0000 C CNN
 F 1 "R_US" V 2286 2000 50  0000 C CNN
 F 2 "" V 2440 1990 50  0001 C CNN
@@
 	7450 4300 7250 4300
 Wire Wire Line
-	7250 4300 7250 4000
-Wire Wire Line
 	7750 2350 7450 2350
 Wire Wire Line
-	7250 2350 7250 2050
+	7250 2350 7250 2200
 $Comp
 L power:GND #PWR06
@@
 Text Label 7250 5800 2    50   ~ 0
 ALE
-Wire Wire Line
-	7750 6200 7450 6200
-Wire Wire Line
-	7250 6200 7250 5900
 $Comp
 L power:GND #PWR08
@@
 	1    0    0    -1
 $EndComp
-Connection ~ 7450 6200
 Wire Wire Line
 	7450 6200 7250 6200
@@
 A16
 $Comp
-L 74xx:74LS244 CPU_IO/WR
+L 74xx:74LS244 CPU_IO/WR1
 U 1 1 607EFA33
 P 10150 1550
-F 0 "CPU_IO/WR" H 10150 2531 50  0000 C CNN
+F 0 "CPU_IO/WR1" H 10150 2531 50  0000 C CNN
 F 1 "74LS244" H 10150 2440 50  0000 C CNN
 F 2 "" H 10150 1550 50  0001 C CNN
@@
 	9650 1950 9650 2050
 Wire Wire Line
-	9650 2050 9650 2350
+	9650 2050 9650 2200
 Wire Wire Line
 	9650 2350 9900 2350
@@
 ~RD
 $Comp
-L 74xx:74LS245 CPU_DDecode1
-U 1 1 60814065
-P 10150 3550
-F 0 "CPU_DDecode1" H 10150 4531 50  0000 C CNN
-F 1 "74LS245" H 10150 4440 50  0000 C CNN
-F 2 "" H 10150 3550 50  0001 C CNN
-F 3 "http://www.ti.com/lit/gpn/sn74LS245" H 10150 3550 50  0001 C CNN
-	1    10150 3550
-	1    0    0    -1
-$EndComp
-$Comp
 L 74xx:74LS245 CPU_DDecode2
 U 1 1 608151DF
@@
 L power:GND #PWR011
 U 1 1 6083EB10
-P 10150 6200
-F 0 "#PWR011" H 10150 5950 50  0001 C CNN
-F 1 "GND" H 10155 6027 50  0000 C CNN
-F 2 "" H 10150 6200 50  0001 C CNN
-F 3 "" H 10150 6200 50  0001 C CNN
-	1    10150 6200
+P 10150 6300
+F 0 "#PWR011" H 10150 6050 50  0001 C CNN
+F 1 "GND" H 10155 6127 50  0000 C CNN
+F 2 "" H 10150 6300 50  0001 C CNN
+F 3 "" H 10150 6300 50  0001 C CNN
+	1    10150 6300
 	1    0    0    -1
 $EndComp
@@
 NoConn ~ 3200 3350
 NoConn ~ 3200 3550
-Text HLabel 4600 1950 2    50   3State ~ 0
+Text HLabel 4600 1950 2    50   Output ~ 0
 ~BHE~S7
 Text Label 3050 1850 2    50   ~ 0
@@
 L power:GND #PWR03
 U 1 1 6085F789
-P 3800 4950
-F 0 "#PWR03" H 3800 4700 50  0001 C CNN
-F 1 "GND" H 3805 4777 50  0000 C CNN
-F 2 "" H 3800 4950 50  0001 C CNN
-F 3 "" H 3800 4950 50  0001 C CNN
-	1    3800 4950
-	1    0    0    -1
-$EndComp
-$Comp
-L power:GND #PWR04
-U 1 1 60860099
-P 4000 4950
-F 0 "#PWR04" H 4000 4700 50  0001 C CNN
-F 1 "GND" H 4005 4777 50  0000 C CNN
-F 2 "" H 4000 4950 50  0001 C CNN
-F 3 "" H 4000 4950 50  0001 C CNN
-	1    4000 4950
+P 3850 5150
+F 0 "#PWR03" H 3850 4900 50  0001 C CNN
+F 1 "GND" H 3855 4977 50  0000 C CNN
+F 2 "" H 3850 5150 50  0001 C CNN
+F 3 "" H 3850 5150 50  0001 C CNN
+	1    3850 5150
 	1    0    0    -1
 $EndComp
@@
 	3200 1650 3050 1650
 $Comp
-L MCU_Intel:8086_Min_Mode CPU
+L MCU_Intel:8086_Min_Mode CPU1
 U 1 1 60761E58
 P 3900 3150
-F 0 "CPU" H 3900 5131 50  0000 C CNN
+F 0 "CPU1" H 3900 5131 50  0000 C CNN
 F 1 "8086_Min_Mode" H 3900 5040 50  0000 C CNN
 F 2 "Package_DIP:DIP-40_W15.24mm" H 3950 3250 50  0001 C CIN
@@
 Connection ~ 8650 2700
 Wire Wire Line
-	8650 2700 8650 750
-Wire Wire Line
 	10150 750  8650 750
-Wire Wire Line
-	10150 2750 8650 2750
 Connection ~ 8650 2750
 Wire Wire Line
@@
 Wire Wire Line
 	10900 4600 10900 2750
-Wire Wire Line
-	10900 2750 10150 2750
-Connection ~ 10150 2750
 $Sheet
 S 800  5050 950  1150
@@
 	-1   0    0    1
 $EndComp
-Connection ~ 2200 1350
-Wire Bus Line
-	9250 2850 9250 5500
-Wire Bus Line
-	6850 850  6850 5100
-Wire Bus Line
-	4850 2000 4850 4050
 $Comp
 L power:VCC #PWR0120
@@
 	0    -1   -1   0
 $EndComp
+Wire Wire Line
+	7750 6200 7450 6200
+Connection ~ 7450 6200
+$Comp
+L power:PWR_FLAG #FLG0101
+U 1 1 61A61862
+P 4200 1000
+F 0 "#FLG0101" H 4200 1075 50  0001 C CNN
+F 1 "PWR_FLAG" H 4200 1173 50  0000 C CNN
+F 2 "" H 4200 1000 50  0001 C CNN
+F 3 "~" H 4200 1000 50  0001 C CNN
+	1    4200 1000
+	1    0    0    -1
+$EndComp
+Wire Wire Line
+	1800 1350 2200 1350
+Connection ~ 2200 1350
+Wire Wire Line
+	3800 4950 3800 5150
+Wire Wire Line
+	3800 5150 3850 5150
+Wire Wire Line
+	4000 4950 4000 5150
+$Comp
+L power:PWR_FLAG #FLG0104
+U 1 1 61A86F05
+P 4000 5150
+F 0 "#FLG0104" H 4000 5225 50  0001 C CNN
+F 1 "PWR_FLAG" H 4000 5323 50  0000 C CNN
+F 2 "" H 4000 5150 50  0001 C CNN
+F 3 "~" H 4000 5150 50  0001 C CNN
+	1    4000 5150
+	0    1    1    0
+$EndComp
+Wire Wire Line
+	4000 5150 3850 5150
+Connection ~ 4000 5150
+Connection ~ 3850 5150
+Wire Wire Line
+	7200 2200 7250 2200
+Connection ~ 7250 2200
+Wire Wire Line
+	7250 2200 7250 2050
+Wire Wire Line
+	9600 2200 9650 2200
+Connection ~ 9650 2200
+Wire Wire Line
+	9650 2200 9650 2350
+Wire Bus Line
+	9250 2850 9250 5500
+Wire Bus Line
+	6850 850  6850 5100
+Wire Bus Line
+	4850 2000 4850 4050
+Wire Wire Line
+	3900 1000 4200 1000
+Connection ~ 4200 1000
+Wire Wire Line
+	4200 1000 4700 1000
+Wire Wire Line
+	8650 750  8650 2700
+Wire Wire Line
+	7250 4000 7250 4300
+Wire Wire Line
+	10150 2750 8650 2750
+Wire Wire Line
+	10900 2750 10150 2750
+Connection ~ 10150 2750
+$Comp
+L 74xx:74LS245 CPU_DDecode1
+U 1 1 60814065
+P 10150 3550
+F 0 "CPU_DDecode1" H 10150 4531 50  0000 C CNN
+F 1 "74LS245" H 10150 4440 50  0000 C CNN
+F 2 "" H 10150 3550 50  0001 C CNN
+F 3 "http://www.ti.com/lit/gpn/sn74LS245" H 10150 3550 50  0001 C CNN
+	1    10150 3550
+	1    0    0    -1
+$EndComp
+Wire Wire Line
+	7250 5900 7250 6200
+Wire Wire Line
+	10150 6200 10150 6300
+Wire Wire Line
+	1600 2350 1800 2350
 $EndSCHEMATC

Commit message: Hopefully the board is here
Parts:
- CPU_ADecode1, CPU_ADecode2, CPU_ADecode3, CPU_DDecode1, CPU_DDecode2, CPU_IO/WR1: footprint (none) -> Package_DIP:DIP-20_W7.62mm
- CPU_Capacitor1: footprint (none) -> Capacitor_THT:CP_Axial_L10.0mm_D4.5mm_P15.00mm_Horizontal
- CPU_Resistor1: footprint (none) -> Resistor_THT:R_Axial_DIN0204_L3.6mm_D1.6mm_P1.90mm_Vertical
- CPU_Switch1: footprint (none) -> Button_Switch_THT:SW_CW_GPTS203211B
- D1: footprint (none) -> Diode_THT:D_5KPW_P7.62mm_Vertical_KathodeUp
Changed lines of the file:
@@
 F 0 "CPU_Switch1" V 2154 1848 50  0000 L CNN
 F 1 "SW_Push" V 2245 1848 50  0000 L CNN
-F 2 "" H 2200 1900 50  0001 C CNN
+F 2 "Button_Switch_THT:SW_CW_GPTS203211B" H 2200 1900 50  0001 C CNN
 F 3 "~" H 2200 1900 50  0001 C CNN
 	1    2200 1700
@@
 F 0 "CPU_Capacitor1" H 1891 1654 50  0000 L CNN
 F 1 "CP1_Small" H 1891 1745 50  0000 L CNN
-F 2 "" H 1800 1700 50  0001 C CNN
+F 2 "Capacitor_THT:CP_Axial_L10.0mm_D4.5mm_P15.00mm_Horizontal" H 1800 1700 50  0001 C CNN
 F 3 "~" H 1800 1700 50  0001 C CNN
 	1    1800 1700
@@
 F 0 "D1" H 2400 2085 50  0000 C CNN
 F 1 "CPU_Diode" H 2400 2176 50  0000 C CNN
-F 2 "" H 2400 2350 50  0001 C CNN
+F 2 "Diode_THT:D_5KPW_P7.62mm_Vertical_KathodeUp" H 2400 2350 50  0001 C CNN
 F 3 "~" H 2400 2350 50  0001 C CNN
 	1    2400 2350
@@
 F 0 "CPU_Resistor1" V 2195 2000 50  0000 C CNN
 F 1 "R_US" V 2286 2000 50  0000 C CNN
-F 2 "" V 2440 1990 50  0001 C CNN
+F 2 "Resistor_THT:R_Axial_DIN0204_L3.6mm_D1.6mm_P1.90mm_Vertical" V 2440 1990 50  0001 C CNN
 F 3 "~" H 2400 2000 50  0001 C CNN
 	1    2400 2000
@@
 F 0 "CPU_ADecode1" H 7750 2531 50  0000 C CNN
 F 1 "74LS373" H 7750 2440 50  0000 C CNN
-F 2 "" H 7750 1550 50  0001 C CNN
+F 2 "Package_DIP:DIP-20_W7.62mm" H 7750 1550 50  0001 C CNN
 F 3 "http://www.ti.com/lit/gpn/sn74LS373" H 7750 1550 50  0001 C CNN
 	1    7750 1550
@@
 F 0 "CPU_ADecode2" H 7750 4481 50  0000 C CNN
 F 1 "74LS373" H 7750 4390 50  0000 C CNN
-F 2 "" H 7750 3500 50  0001 C CNN
+F 2 "Package_DIP:DIP-20_W7.62mm" H 7750 3500 50  0001 C CNN
 F 3 "http://www.ti.com/lit/gpn/sn74LS373" H 7750 3500 50  0001 C CNN
 	1    7750 3500
@@
 F 0 "CPU_ADecode3" H 7750 6381 50  0000 C CNN
 F 1 "74LS373" H 7750 6290 50  0000 C CNN
-F 2 "" H 7750 5400 50  0001 C CNN
+F 2 "Package_DIP:DIP-20_W7.62mm" H 7750 5400 50  0001 C CNN
 F 3 "http://www.ti.com/lit/gpn/sn74LS373" H 7750 5400 50  0001 C CNN
 	1    7750 5400
@@
 F 0 "CPU_IO/WR1" H 10150 2531 50  0000 C CNN
 F 1 "74LS244" H 10150 2440 50  0000 C CNN
-F 2 "" H 10150 1550 50  0001 C CNN
+F 2 "Package_DIP:DIP-20_W7.62mm" H 10150 1550 50  0001 C CNN
 F 3 "http://www.ti.com/lit/ds/symlink/sn74ls244.pdf" H 10150 1550 50  0001 C CNN
 	1    10150 1550
@@
 F 0 "CPU_DDecode2" H 10150 6381 50  0000 C CNN
 F 1 "74LS245" H 10150 6290 50  0000 C CNN
-F 2 "" H 10150 5400 50  0001 C CNN
+F 2 "Package_DIP:DIP-20_W7.62mm" H 10150 5400 50  0001 C CNN
 F 3 "http://www.ti.com/lit/gpn/sn74LS245" H 10150 5400 50  0001 C CNN
 	1    10150 5400
@@
 Wire Wire Line
 	9650 2200 9650 2350
+Wire Wire Line
+	3900 1000 4200 1000
+Connection ~ 4200 1000
+Wire Wire Line
+	4200 1000 4700 1000
+Wire Wire Line
+	8650 750  8650 2700
+Wire Wire Line
+	7250 4000 7250 4300
+Wire Wire Line
+	10150 2750 8650 2750
+Wire Wire Line
+	10900 2750 10150 2750
+Connection ~ 10150 2750
+$Comp
+L 74xx:74LS245 CPU_DDecode1
+U 1 1 60814065
+P 10150 3550
+F 0 "CPU_DDecode1" H 10150 4531 50  0000 C CNN
+F 1 "74LS245" H 10150 4440 50  0000 C CNN
+F 2 "Package_DIP:DIP-20_W7.62mm" H 10150 3550 50  0001 C CNN
+F 3 "http://www.ti.com/lit/gpn/sn74LS245" H 10150 3550 50  0001 C CNN
+	1    10150 3550
+	1    0    0    -1
+$EndComp
+Wire Wire Line
+	7250 5900 7250 6200
+Wire Wire Line
+	10150 6200 10150 6300
+Wire Wire Line
+	1600 2350 1800 2350
 Wire Bus Line
 	9250 2850 9250 5500
@@
 Wire Bus Line
 	4850 2000 4850 4050
-Wire Wire Line
-	3900 1000 4200 1000
-Connection ~ 4200 1000
-Wire Wire Line
-	4200 1000 4700 1000
-Wire Wire Line
-	8650 750  8650 2700
-Wire Wire Line
-	7250 4000 7250 4300
-Wire Wire Line
-	10150 2750 8650 2750
-Wire Wire Line
-	10900 2750 10150 2750
-Connection ~ 10150 2750
-$Comp
-L 74xx:74LS245 CPU_DDecode1
-U 1 1 60814065
-P 10150 3550
-F 0 "CPU_DDecode1" H 10150 4531 50  0000 C CNN
-F 1 "74LS245" H 10150 4440 50  0000 C CNN
-F 2 "" H 10150 3550 50  0001 C CNN
-F 3 "http://www.ti.com/lit/gpn/sn74LS245" H 10150 3550 50  0001 C CNN
-	1    10150 3550
-	1    0    0    -1
-$EndComp
-Wire Wire Line
-	7250 5900 7250 6200
-Wire Wire Line
-	10150 6200 10150 6300
-Wire Wire Line
-	1600 2350 1800 2350
 $EndSCHEMATC
