File: Final/8254(FINAL).sch (KiCad schematic (older format))
At the start: 2 parts, among them U1 PAL16L8, U2 8254

Commit message: New stuff
Parts:
- added J2: Conn_01x08_Female, symbol Connector:Conn_01x08_Female
- renumbered U1 to U26, U2 to U27
Connections:
- net A0: now also U26.2 (I2)
- net D7: now reaches U27.1 (D7)
- net D6: now reaches U27.2 (D6)
- net A1: now reaches U27.20 (A1)
- net D5: now reaches U27.3 (D5)
- net D4: now reaches U27.4 (D4)
- net D3: now reaches U27.5 (D3)
- net D2: now reaches U27.6 (D2)
- net D1: now reaches U27.7 (D1)
- net D0: now reaches U27.8 (D0)
- net A10: now reaches U26.11 (I10)
- net A11: now reaches U26.13 (IO7)
- net A12: now reaches U26.14 (IO6)
- net A13: now reaches U26.15 (IO5)
- net A14: now reaches U26.16 (IO4)
- net A15: now reaches U26.17 (I03)
- net A3: now reaches U26.3 (I3)
- net A4: now reaches U26.4 (I4)
- net A5: now reaches U26.5 (I5)
- net A6: now reaches U26.6 (I6)
- net A7: now reaches U26.7 (I7)
- net A8: now reaches U26.8 (I8)
- net A9: now reaches U26.9 (I9)
- net CLK0: no longer names the net of U27.9 (CLK0)
- net CLK0: now also J2.1 (Pin_1)
- net CLK1: no longer names the net of U27.15 (CLK1)
- net CLK1: now also J2.4 (Pin_4)
- net CLK2: no longer names the net of U27.18 (CLK2)
- net CLK2: now also J2.6 (Pin_6)
- net G0: no longer names the net of U27.11 (G0)
- net G0: now also J2.2 (Pin_2)
- net G1: no longer names the net of U27.14 (G1)
- net G1: now also J2.5 (Pin_5)
- net G2: no longer names the net of U27.16 (G2)
- net G2: now also J2.7 (Pin_7)
- net IR1 renamed COUNTER2
- net OUT0: no longer names the net of U27.10 (OUT0)
- net OUT0: now also J2.3 (Pin_3)
- net OUT2: no longer names the net of U27.17 (OUT2)
- net OUT2: now also J2.8 (Pin_8)
- net ~WAIT2: no longer names the net of U26.18 (IO2), U26.19 (IO1), U27.21 (~CS~)
Changed lines of the file:
@@
 $EndDescr
 $Comp
-L Timer:8254 U2
+L Timer:8254 U27
 U 1 1 60845EE8
 P 5650 3250
-F 0 "U2" H 5650 4431 50  0000 C CNN
+F 0 "U27" H 5650 4431 50  0000 C CNN
 F 1 "8254" H 5650 4340 50  0000 C CNN
 F 2 "Package_DIP:DIP-24_W15.24mm" H 5700 3500 50  0001 C CNN
@@
 $EndComp
 $Comp
-L power:GND #PWR04
+L power:GND #PWR045
 U 1 1 60848002
 P 5650 4250
-F 0 "#PWR04" H 5650 4000 50  0001 C CNN
+F 0 "#PWR045" H 5650 4000 50  0001 C CNN
 F 1 "GND" H 5655 4077 50  0000 C CNN
 F 2 "" H 5650 4250 50  0001 C CNN
@@
 $EndComp
 $Comp
-L power:VCC #PWR03
+L power:VCC #PWR044
 U 1 1 6084836A
 P 5650 1950
-F 0 "#PWR03" H 5650 1800 50  0001 C CNN
+F 0 "#PWR044" H 5650 1800 50  0001 C CNN
 F 1 "VCC" H 5665 2123 50  0000 C CNN
 F 2 "" H 5650 1950 50  0001 C CNN
@@
 	4250 2650 4350 2550
 Text HLabel 4250 2650 0    50   Input ~ 0
-D[0:7]
+D[0..7]
 Text HLabel 4350 3450 0    50   Input ~ 0
 ~RD
@@
 M~IO
 $Comp
-L power:GND #PWR02
+L power:GND #PWR043
 U 1 1 6085575F
 P 2200 5900
-F 0 "#PWR02" H 2200 5650 50  0001 C CNN
+F 0 "#PWR043" H 2200 5650 50  0001 C CNN
 F 1 "GND" H 2205 5727 50  0000 C CNN
 F 2 "" H 2200 5900 50  0001 C CNN
@@
 $EndComp
 $Comp
-L power:VCC #PWR01
+L power:VCC #PWR042
 U 1 1 60855DD6
 P 2200 4200
-F 0 "#PWR01" H 2200 4050 50  0001 C CNN
+F 0 "#PWR042" H 2200 4050 50  0001 C CNN
 F 1 "VCC" H 2215 4373 50  0000 C CNN
 F 2 "" H 2200 4200 50  0001 C CNN
@@
 Wire Wire Line
 	2200 4600 2200 4200
-Text HLabel 3850 3950 0    50   Input ~ 0
-~WAIT2
 Wire Wire Line
 	5050 3950 4700 3950
@@
 Wire Wire Line
 	4700 4900 4700 4800
-Connection ~ 4700 3950
-Wire Wire Line
-	4700 3950 3850 3950
 Wire Wire Line
 	2700 4800 4700 4800
@@
 Wire Wire Line
 	3750 6950 1050 6950
-Wire Wire Line
-	1050 3650 5050 3650
-Wire Wire Line
-	1050 3750 5050 3750
-Entry Wire Line
-	950  3750 1050 3650
-Entry Wire Line
-	950  3850 1050 3750
 Entry Wire Line
 	950  5000 1050 4900
@@
 Wire Wire Line
 	1700 4800 1200 4800
-Wire Wire Line
-	6250 2850 6550 2850
-Text HLabel 6550 2850 2    50   Output ~ 0
-OUT0
-Text HLabel 6550 3850 2    50   Output ~ 0
-OUT2
-Text HLabel 6550 3350 2    50   Output ~ 0
-IR1
-Wire Wire Line
-	6250 2650 6550 2650
-Wire Wire Line
-	6250 2750 6550 2750
-Wire Wire Line
-	6250 3150 6550 3150
-Wire Wire Line
-	6250 3250 6550 3250
-Wire Wire Line
-	6250 3650 6550 3650
-Wire Wire Line
-	6250 3750 6550 3750
-Wire Wire Line
-	6250 3850 6550 3850
-Wire Wire Line
-	6250 3350 6550 3350
-Text HLabel 6550 2650 2    50   Output ~ 0
-CLK0
-Text HLabel 6550 3150 2    50   Output ~ 0
-CLK1
-Text HLabel 6550 3650 2    50   Output ~ 0
-CLK2
-Text HLabel 6550 2750 2    50   Output ~ 0
-G0
-Text HLabel 6550 3250 2    50   Output ~ 0
-G1
-Text HLabel 6550 3750 2    50   Output ~ 0
-G2
-Text HLabel 950  4150 0    50   Input ~ 0
-A[0:15]
-$Comp
-L Logic_Programmable:PAL16L8 U1
+Text HLabel 950  5050 0    50   Input ~ 0
+A[0..15]
+$Comp
+L Logic_Programmable:PAL16L8 U26
 U 1 1 6084E134
 P 2200 5300
-F 0 "U1" H 2200 6181 50  0000 C CNN
+F 0 "U26" H 2200 6181 50  0000 C CNN
 F 1 "PAL16L8" H 2200 6090 50  0000 C CNN
 F 2 "" H 2200 5300 50  0001 C CNN
@@
 $EndComp
 NoConn ~ 2700 5500
+Text HLabel 5050 3650 0    50   Input ~ 0
+A0
+Text HLabel 5050 3750 0    50   Input ~ 0
+A1
+Text HLabel 6250 3350 2    50   Output ~ 0
+COUNTER2
+Text Label 1350 4900 2    50   ~ 0
+A0
+Text Label 1350 5000 2    50   ~ 0
+A3
+Text Label 1350 5100 2    50   ~ 0
+A4
+Text Label 1350 5200 2    50   ~ 0
+A5
+Text Label 1350 5300 2    50   ~ 0
+A6
+Text Label 1350 5400 2    50   ~ 0
+A7
+Text Label 1350 5500 2    50   ~ 0
+A8
+Text Label 1350 5600 2    50   ~ 0
+A9
+Text Label 1350 5700 2    50   ~ 0
+A10
+Text Label 2750 5400 0    50   ~ 0
+A11
+Text Label 2750 5300 0    50   ~ 0
+A12
+Text Label 2750 5200 0    50   ~ 0
+A13
+Text Label 2750 5100 0    50   ~ 0
+A14
+Text Label 2750 5000 0    50   ~ 0
+A15
+Text Label 4750 2550 0    50   ~ 0
+D0
+Text Label 4750 2650 0    50   ~ 0
+D1
+Text Label 4750 2750 0    50   ~ 0
+D2
+Text Label 4750 2850 0    50   ~ 0
+D3
+Text Label 4750 2950 0    50   ~ 0
+D4
+Text Label 4750 3050 0    50   ~ 0
+D5
+Text Label 4750 3150 0    50   ~ 0
+D6
+Text Label 4750 3250 0    50   ~ 0
+D7
+$Comp
+L Connector:Conn_01x08_Female J2
+U 1 1 60B4C76F
+P 7850 3150
+F 0 "J2" H 7878 3126 50  0000 L CNN
+F 1 "Conn_01x08_Female" H 7878 3035 50  0000 L CNN
+F 2 "" H 7850 3150 50  0001 C CNN
+F 3 "~" H 7850 3150 50  0001 C CNN
+	1    7850 3150
+	1    0    0    -1
+$EndComp
+Wire Wire Line
+	6250 2650 7550 2650
+Wire Wire Line
+	7550 2650 7550 2850
+Wire Wire Line
+	7550 2850 7650 2850
+Wire Wire Line
+	6250 2750 7500 2750
+Wire Wire Line
+	7500 2750 7500 2950
+Wire Wire Line
+	7500 2950 7650 2950
+Wire Wire Line
+	6250 2850 7450 2850
+Wire Wire Line
+	7450 2850 7450 3050
+Wire Wire Line
+	7450 3050 7650 3050
+Wire Wire Line
+	6250 3150 7650 3150
+Wire Wire Line
+	6250 3250 7650 3250
+Wire Wire Line
+	6250 3850 7550 3850
+Wire Wire Line
+	7550 3850 7550 3550
+Wire Wire Line
+	7550 3550 7650 3550
+Wire Wire Line
+	6250 3750 7500 3750
+Wire Wire Line
+	7500 3750 7500 3450
+Wire Wire Line
+	7500 3450 7650 3450
+Wire Wire Line
+	6250 3650 7450 3650
+Wire Wire Line
+	7450 3650 7450 3350
+Wire Wire Line
+	7450 3350 7650 3350
 Wire Bus Line
 	4250 2650 4250 3350
 Wire Bus Line
-	950  3750 950  7050
-Text Label 2450 3650 2    50   ~ 0
-A0
+	950  5000 950  7050
 $EndSCHEMATC

Commit message: For Commenting
Connections:
- net A0: no longer U26.2 (I2)
- new net A2: U26.2 (I2)
Changed lines of the file:
@@
 $Descr A4 11693 8268
 encoding utf-8
-Sheet 8 14
+Sheet 10 16
 Title ""
 Date ""
@@
 Wire Wire Line
 	5050 3550 4350 3550
-Entry Wire Line
-	4250 2750 4350 2650
-Entry Wire Line
-	4250 2850 4350 2750
-Entry Wire Line
-	4250 2950 4350 2850
-Entry Wire Line
-	4250 3050 4350 2950
-Entry Wire Line
-	4250 3250 4350 3150
-Entry Wire Line
-	4250 3350 4350 3250
-Entry Wire Line
-	4250 3150 4350 3050
-Entry Wire Line
-	4250 2650 4350 2550
-Text HLabel 4250 2650 0    50   Input ~ 0
-D[0..7]
 Text HLabel 4350 3450 0    50   Input ~ 0
 ~RD
 Text HLabel 4350 3550 0    50   Input ~ 0
 ~WR
-Text HLabel 1200 4800 0    50   Input ~ 0
-M~IO
 $Comp
 L power:GND #PWR043
@@
 	4700 4800 4700 3950
 Wire Wire Line
-	2700 5400 3000 5400
-Wire Wire Line
-	3000 5400 3000 6200
-Wire Wire Line
-	3000 6200 1050 6200
-Wire Wire Line
-	3150 5300 3150 6350
-Wire Wire Line
-	3150 6350 1050 6350
-Wire Wire Line
-	2700 5300 3150 5300
-Wire Wire Line
-	3350 5200 3350 6550
-Wire Wire Line
-	3350 6550 1050 6550
-Wire Wire Line
-	2700 5200 3350 5200
-Wire Wire Line
-	3550 5100 3550 6750
-Wire Wire Line
-	3550 6750 1050 6750
-Wire Wire Line
-	2700 5100 3550 5100
-Wire Wire Line
-	2700 5000 3750 5000
-Wire Wire Line
-	3750 5000 3750 6950
-Wire Wire Line
-	3750 6950 1050 6950
-Entry Wire Line
-	950  5000 1050 4900
-Entry Wire Line
-	950  5100 1050 5000
-Entry Wire Line
-	950  5200 1050 5100
-Entry Wire Line
-	950  5300 1050 5200
-Entry Wire Line
-	950  5400 1050 5300
-Entry Wire Line
-	950  5500 1050 5400
-Entry Wire Line
-	950  5600 1050 5500
-Entry Wire Line
-	950  5700 1050 5600
-Entry Wire Line
-	950  5800 1050 5700
-Entry Wire Line
-	950  6300 1050 6200
-Entry Wire Line
-	950  6450 1050 6350
-Entry Wire Line
-	950  6650 1050 6550
-Entry Wire Line
-	950  6850 1050 6750
-Entry Wire Line
-	950  7050 1050 6950
-Wire Wire Line
 	1050 4900 1700 4900
 Wire Wire Line
@@
 Wire Wire Line
 	1700 4800 1200 4800
-Text HLabel 950  5050 0    50   Input ~ 0
-A[0..15]
 $Comp
 L Logic_Programmable:PAL16L8 U26
@@
 Text HLabel 6250 3350 2    50   Output ~ 0
 COUNTER2
-Text Label 1350 4900 2    50   ~ 0
-A0
-Text Label 1350 5000 2    50   ~ 0
-A3
-Text Label 1350 5100 2    50   ~ 0
-A4
-Text Label 1350 5200 2    50   ~ 0
-A5
-Text Label 1350 5300 2    50   ~ 0
-A6
-Text Label 1350 5400 2    50   ~ 0
-A7
-Text Label 1350 5500 2    50   ~ 0
-A8
-Text Label 1350 5600 2    50   ~ 0
-A9
-Text Label 1350 5700 2    50   ~ 0
-A10
-Text Label 2750 5400 0    50   ~ 0
-A11
-Text Label 2750 5300 0    50   ~ 0
-A12
-Text Label 2750 5200 0    50   ~ 0
-A13
-Text Label 2750 5100 0    50   ~ 0
-A14
-Text Label 2750 5000 0    50   ~ 0
-A15
-Text Label 4750 2550 0    50   ~ 0
-D0
-Text Label 4750 2650 0    50   ~ 0
-D1
-Text Label 4750 2750 0    50   ~ 0
-D2
-Text Label 4750 2850 0    50   ~ 0
-D3
-Text Label 4750 2950 0    50   ~ 0
-D4
-Text Label 4750 3050 0    50   ~ 0
-D5
-Text Label 4750 3150 0    50   ~ 0
-D6
-Text Label 4750 3250 0    50   ~ 0
-D7
 $Comp
 L Connector:Conn_01x08_Female J2
@@
 Wire Wire Line
 	7450 3350 7650 3350
-Wire Bus Line
-	4250 2650 4250 3350
-Wire Bus Line
-	950  5000 950  7050
+Text HLabel 4350 2550 0    50   Input ~ 0
+D0
+Text HLabel 4350 2650 0    50   Input ~ 0
+D1
+Text HLabel 4350 2750 0    50   Input ~ 0
+D2
+Text HLabel 4350 2850 0    50   Input ~ 0
+D3
+Text HLabel 4350 2950 0    50   Input ~ 0
+D4
+Text HLabel 4350 3050 0    50   Input ~ 0
+D5
+Text HLabel 4350 3150 0    50   Input ~ 0
+D6
+Text HLabel 4350 3250 0    50   Input ~ 0
+D7
+Text HLabel 1200 4800 0    50   Input ~ 0
+M~IO
+Text HLabel 1050 4900 0    50   Input ~ 0
+A2
+Wire Wire Line
+	2700 5000 3000 5000
+Wire Wire Line
+	2700 5100 3000 5100
+Wire Wire Line
+	2700 5200 3000 5200
+Wire Wire Line
+	2700 5300 3000 5300
+Wire Wire Line
+	2700 5400 3000 5400
+Text HLabel 3000 5000 2    50   Input ~ 0
+A15
+Text HLabel 3000 5100 2    50   Input ~ 0
+A14
+Text HLabel 3000 5200 2    50   Input ~ 0
+A13
+Text HLabel 3000 5300 2    50   Input ~ 0
+A12
+Text HLabel 3000 5400 2    50   Input ~ 0
+A11
+Text HLabel 1050 5000 0    50   Input ~ 0
+A3
+Text HLabel 1050 5100 0    50   Input ~ 0
+A4
+Text HLabel 1050 5200 0    50   Input ~ 0
+A5
+Text HLabel 1050 5300 0    50   Input ~ 0
+A6
+Text HLabel 1050 5400 0    50   Input ~ 0
+A7
+Text HLabel 1050 5500 0    50   Input ~ 0
+A8
+Text HLabel 1050 5600 0    50   Input ~ 0
+A9
+Text HLabel 1050 5700 0    50   Input ~ 0
+A10
 $EndSCHEMATC

Commit message: Stuffs
Parts:
- added R?: 10000, symbol Device:R_Small_US
Connections:
- net at U27.14 (G1): now also R?.2; no longer J2.5 (Pin_5)
- net at J2.4 (Pin_4): no longer U27.15 (CLK1)
- new net +5V: R?.1
- new net CLK: U27.15 (CLK1)
Changed lines of the file:
@@
 	7450 3050 7650 3050
-Wire Wire Line
-	6250 3150 7650 3150
-Wire Wire Line
-	6250 3250 7650 3250
 Wire Wire Line
 	6250 3850 7550 3850
@@
 Text HLabel 1050 5700 0    50   Input ~ 0
 A10
+$Comp
+L power:+5V #PWR0133
+U 1 1 61A121ED
+P 6900 3250
+F 0 "#PWR0133" H 6900 3100 50  0001 C CNN
+F 1 "+5V" V 6915 3378 50  0000 L CNN
+F 2 "" H 6900 3250 50  0001 C CNN
+F 3 "" H 6900 3250 50  0001 C CNN
+	1    6900 3250
+	0    1    1    0
+$EndComp
+$Comp
+L Device:R_Small_US R?
+U 1 1 61A1330B
+P 6650 3250
+F 0 "R?" V 6445 3250 50  0000 C CNN
+F 1 "10000" V 6536 3250 50  0000 C CNN
+F 2 "" H 6650 3250 50  0001 C CNN
+F 3 "~" H 6650 3250 50  0001 C CNN
+	1    6650 3250
+	0    1    1    0
+$EndComp
+Wire Wire Line
+	6900 3250 6750 3250
+Wire Wire Line
+	6550 3250 6250 3250
+Text HLabel 6250 3150 2    50   Input ~ 0
+CLK
 $EndSCHEMATC

Commit message: Final?
Parts:
- removed J2: Conn_01x08_Female, symbol Connector:Conn_01x08_Female
- added Counter_Header1: Conn_01x06_Female, symbol Connector:Conn_01x06_Female
- gave numbers to parts that had none: 1
- renumbered U27 to Counter1, U26 to Counter_Decode1
Connections:
- net at Counter1.10 (OUT0): now also Counter_Header1.3 (Pin_3)
- net at Counter1.11 (G0): now also Counter_Header1.2 (Pin_2)
- net at Counter1.16 (G2): now also Counter_Header1.5 (Pin_5)
- net at Counter1.17 (OUT2): now also Counter_Header1.6 (Pin_6)
- net at Counter1.18 (CLK2): now also Counter_Header1.4 (Pin_4)
- net at Counter1.9 (CLK0): now also Counter_Header1.1 (Pin_1)
Changed lines of the file:
@@
 $EndDescr
 $Comp
-L Timer:8254 U27
+L Timer:8254 Counter1
 U 1 1 60845EE8
 P 5650 3250
-F 0 "U27" H 5650 4431 50  0000 C CNN
+F 0 "Counter1" H 5650 4431 50  0000 C CNN
 F 1 "8254" H 5650 4340 50  0000 C CNN
 F 2 "Package_DIP:DIP-24_W15.24mm" H 5700 3500 50  0001 C CNN
@@
 $EndComp
 $Comp
-L power:GND #PWR045
-U 1 1 60848002
-P 5650 4250
-F 0 "#PWR045" H 5650 4000 50  0001 C CNN
-F 1 "GND" H 5655 4077 50  0000 C CNN
-F 2 "" H 5650 4250 50  0001 C CNN
-F 3 "" H 5650 4250 50  0001 C CNN
-	1    5650 4250
-	1    0    0    -1
-$EndComp
-$Comp
 L power:VCC #PWR044
 U 1 1 6084836A
-P 5650 1950
-F 0 "#PWR044" H 5650 1800 50  0001 C CNN
-F 1 "VCC" H 5665 2123 50  0000 C CNN
-F 2 "" H 5650 1950 50  0001 C CNN
-F 3 "" H 5650 1950 50  0001 C CNN
-	1    5650 1950
-	1    0    0    -1
-$EndComp
-Wire Wire Line
-	5650 2250 5650 1950
+P 5650 1600
+F 0 "#PWR044" H 5650 1450 50  0001 C CNN
+F 1 "VCC" H 5665 1773 50  0000 C CNN
+F 2 "" H 5650 1600 50  0001 C CNN
+F 3 "" H 5650 1600 50  0001 C CNN
+	1    5650 1600
+	1    0    0    -1
+$EndComp
 Wire Wire Line
 	5050 2550 4350 2550
@@
 L power:GND #PWR043
 U 1 1 6085575F
-P 2200 5900
-F 0 "#PWR043" H 2200 5650 50  0001 C CNN
-F 1 "GND" H 2205 5727 50  0000 C CNN
-F 2 "" H 2200 5900 50  0001 C CNN
-F 3 "" H 2200 5900 50  0001 C CNN
-	1    2200 5900
-	1    0    0    -1
-$EndComp
-$Comp
-L power:VCC #PWR042
-U 1 1 60855DD6
-P 2200 4200
-F 0 "#PWR042" H 2200 4050 50  0001 C CNN
-F 1 "VCC" H 2215 4373 50  0000 C CNN
-F 2 "" H 2200 4200 50  0001 C CNN
-F 3 "" H 2200 4200 50  0001 C CNN
-	1    2200 4200
-	1    0    0    -1
-$EndComp
-Wire Wire Line
-	2200 4600 2200 4200
+P 2200 6200
+F 0 "#PWR043" H 2200 5950 50  0001 C CNN
+F 1 "GND" H 2205 6027 50  0000 C CNN
+F 2 "" H 2200 6200 50  0001 C CNN
+F 3 "" H 2200 6200 50  0001 C CNN
+	1    2200 6200
+	1    0    0    -1
+$EndComp
 Wire Wire Line
 	5050 3950 4700 3950
@@
 	1700 4800 1200 4800
 $Comp
-L Logic_Programmable:PAL16L8 U26
+L Logic_Programmable:PAL16L8 Counter_Decode1
 U 1 1 6084E134
 P 2200 5300
-F 0 "U26" H 2200 6181 50  0000 C CNN
+F 0 "Counter_Decode1" H 2200 6181 50  0000 C CNN
 F 1 "PAL16L8" H 2200 6090 50  0000 C CNN
 F 2 "" H 2200 5300 50  0001 C CNN
@@
 Text HLabel 6250 3350 2    50   Output ~ 0
 COUNTER2
-$Comp
-L Connector:Conn_01x08_Female J2
-U 1 1 60B4C76F
-P 7850 3150
-F 0 "J2" H 7878 3126 50  0000 L CNN
-F 1 "Conn_01x08_Female" H 7878 3035 50  0000 L CNN
-F 2 "" H 7850 3150 50  0001 C CNN
-F 3 "~" H 7850 3150 50  0001 C CNN
-	1    7850 3150
-	1    0    0    -1
-$EndComp
 Wire Wire Line
 	6250 2650 7550 2650
 Wire Wire Line
-	7550 2650 7550 2850
-Wire Wire Line
-	7550 2850 7650 2850
+	7550 2650 7550 2950
 Wire Wire Line
 	6250 2750 7500 2750
 Wire Wire Line
-	7500 2750 7500 2950
-Wire Wire Line
-	7500 2950 7650 2950
+	7500 2750 7500 3050
 Wire Wire Line
 	6250 2850 7450 2850
 Wire Wire Line
-	7450 2850 7450 3050
-Wire Wire Line
-	7450 3050 7650 3050
+	7450 2850 7450 3150
 Wire Wire Line
 	6250 3850 7550 3850
 Wire Wire Line
-	7550 3850 7550 3550
-Wire Wire Line
-	7550 3550 7650 3550
+	7550 3850 7550 3450
 Wire Wire Line
 	6250 3750 7500 3750
 Wire Wire Line
-	7500 3750 7500 3450
-Wire Wire Line
-	7500 3450 7650 3450
+	7500 3750 7500 3350
 Wire Wire Line
 	6250 3650 7450 3650
-Wire Wire Line
-	7450 3650 7450 3350
-Wire Wire Line
-	7450 3350 7650 3350
 Text HLabel 4350 2550 0    50   Input ~ 0
 D0
@@
 $EndComp
 $Comp
-L Device:R_Small_US R?
+L Device:R_Small_US Counter_Resistor1
 U 1 1 61A1330B
 P 6650 3250
-F 0 "R?" V 6445 3250 50  0000 C CNN
+F 0 "Counter_Resistor1" V 6445 3250 50  0000 C CNN
 F 1 "10000" V 6536 3250 50  0000 C CNN
 F 2 "" H 6650 3250 50  0001 C CNN
@@
 Text HLabel 6250 3150 2    50   Input ~ 0
 CLK
+Wire Wire Line
+	2200 5900 2200 6050
+Wire Wire Line
+	5650 4250 5650 6050
+Wire Wire Line
+	5650 6050 2200 6050
+Connection ~ 2200 6050
+Wire Wire Line
+	2200 1900 5650 1900
+Wire Wire Line
+	2200 1900 2200 4600
+Connection ~ 5650 1900
+Wire Wire Line
+	5650 1900 5650 2250
+Wire Wire Line
+	2200 6050 2200 6200
+Wire Wire Line
+	5650 1600 5650 1900
+Wire Wire Line
+	7450 3650 7450 3250
+$Comp
+L Connector:Conn_01x06_Female Counter_Header1
+U 1 1 61FB5B66
+P 7950 3150
+F 0 "Counter_Header1" H 7978 3126 50  0000 L CNN
+F 1 "Conn_01x06_Female" H 7978 3035 50  0000 L CNN
+F 2 "" H 7950 3150 50  0001 C CNN
+F 3 "~" H 7950 3150 50  0001 C CNN
+	1    7950 3150
+	1    0    0    -1
+$EndComp
+Wire Wire Line
+	7450 3250 7750 3250
+Wire Wire Line
+	7500 3350 7750 3350
+Wire Wire Line
+	7550 3450 7750 3450
+Wire Wire Line
+	7450 3150 7750 3150
+Wire Wire Line
+	7500 3050 7750 3050
+Wire Wire Line
+	7550 2950 7750 2950
 $EndSCHEMATC

Commit message: Hopefully the board is here
Parts:
- Counter_Decode1: footprint (none) -> Package_DIP:DIP-20_W7.62mm
- Counter_Header1: footprint (none) -> Connector_PinHeader_1.00mm:PinHeader_1x06_P1.00mm_Horizontal
- Counter_Resistor1: footprint (none) -> Resistor_THT:R_Axial_DIN0204_L3.6mm_D1.6mm_P1.90mm_Vertical
Changed lines of the file:
@@
 F 0 "Counter_Decode1" H 2200 6181 50  0000 C CNN
 F 1 "PAL16L8" H 2200 6090 50  0000 C CNN
-F 2 "" H 2200 5300 50  0001 C CNN
+F 2 "Package_DIP:DIP-20_W7.62mm" H 2200 5300 50  0001 C CNN
 F 3 "" H 2200 5300 50  0001 C CNN
 	1    2200 5300
@@
 F 0 "Counter_Resistor1" V 6445 3250 50  0000 C CNN
 F 1 "10000" V 6536 3250 50  0000 C CNN
-F 2 "" H 6650 3250 50  0001 C CNN
+F 2 "Resistor_THT:R_Axial_DIN0204_L3.6mm_D1.6mm_P1.90mm_Vertical" H 6650 3250 50  0001 C CNN
 F 3 "~" H 6650 3250 50  0001 C CNN
 	1    6650 3250
@@
 F 0 "Counter_Header1" H 7978 3126 50  0000 L CNN
 F 1 "Conn_01x06_Female" H 7978 3035 50  0000 L CNN
-F 2 "" H 7950 3150 50  0001 C CNN
+F 2 "Connector_PinHeader_1.00mm:PinHeader_1x06_P1.00mm_Horizontal" H 7950 3150 50  0001 C CNN
 F 3 "~" H 7950 3150 50  0001 C CNN
 	1    7950 3150
