File: Final/8259(FINAL).sch (KiCad schematic (older format))
At the start: 4 parts

Commit message: New stuff
Parts:
- gave numbers to parts that had none: 4
Changed lines of the file:
@@
 $EndDescr
 $Comp
-L Interface:8259 U?
+L Interface:8259 U25
 U 1 1 6078126B
 P 7650 3050
-F 0 "U?" H 7650 4331 50  0000 C CNN
+F 0 "U25" H 7650 4331 50  0000 C CNN
 F 1 "8259" H 7650 4240 50  0000 C CNN
 F 2 "Package_DIP:DIP-28_W15.24mm" H 7650 3050 50  0001 C CIN
@@
 $EndComp
 $Comp
-L Switch:SW_Push SW?
+L Switch:SW_Push SW3
 U 1 1 60783CAD
 P 9500 2950
-F 0 "SW?" H 9500 3235 50  0000 C CNN
+F 0 "SW3" H 9500 3235 50  0000 C CNN
 F 1 "SW_Push" H 9500 3144 50  0000 C CNN
 F 2 "" H 9500 3150 50  0001 C CNN
@@
 $EndComp
 $Comp
-L power:GND #PWR?
+L power:GND #PWR041
 U 1 1 607858DC
 P 9700 3100
-F 0 "#PWR?" H 9700 2850 50  0001 C CNN
+F 0 "#PWR041" H 9700 2850 50  0001 C CNN
 F 1 "GND" H 9705 2927 50  0000 C CNN
 F 2 "" H 9700 3100 50  0001 C CNN
@@
 NoConn ~ 8250 2250
 $Comp
-L power:+5V #PWR?
+L power:+5V #PWR040
 U 1 1 6078B521
 P 8800 3550
-F 0 "#PWR?" H 8800 3400 50  0001 C CNN
+F 0 "#PWR040" H 8800 3400 50  0001 C CNN
 F 1 "+5V" V 8815 3678 50  0000 L CNN
 F 2 "" H 8800 3550 50  0001 C CNN
@@
 $EndComp
 $Comp
-L Device:R R?
+L Device:R R3
 U 1 1 6078C718
 P 8500 3550
-F 0 "R?" V 8293 3550 50  0000 C CNN
+F 0 "R3" V 8293 3550 50  0000 C CNN
 F 1 "R" V 8384 3550 50  0000 C CNN
 F 2 "" V 8430 3550 50  0001 C CNN
@@
 	6650 3750 7050 3750
 $Comp
-L power:+5V #PWR?
+L power:+5V #PWR039
 U 1 1 60791E23
 P 7850 1950
-F 0 "#PWR?" H 7850 1800 50  0001 C CNN
+F 0 "#PWR039" H 7850 1800 50  0001 C CNN
 F 1 "+5V" V 7865 2078 50  0000 L CNN
 F 2 "" H 7850 1950 50  0001 C CNN
@@
 	7850 1950 7650 1950
 $Comp
-L power:GND #PWR?
+L power:GND #PWR038
 U 1 1 607931C2
 P 7650 4150
-F 0 "#PWR?" H 7650 3900 50  0001 C CNN
+F 0 "#PWR038" H 7650 3900 50  0001 C CNN
 F 1 "GND" H 7655 3977 50  0000 C CNN
 F 2 "" H 7650 4150 50  0001 C CNN
@@
 8259INT_Out
 Text HLabel 6300 3000 0    50   BiDi ~ 0
-D[0:7]
+D[0..7]
 Wire Wire Line
 	7050 3150 6850 3150
@@
 	6850 3850 7050 3850
 $Comp
-L Logic_Programmable:PAL16L8 U?
+L Logic_Programmable:PAL16L8 U24
 U 1 1 60799BF8
 P 4350 3500
-F 0 "U?" H 4350 4381 50  0000 C CNN
+F 0 "U24" H 4350 4381 50  0000 C CNN
 F 1 "PAL16L8" H 4350 4290 50  0000 C CNN
 F 2 "" H 4350 3500 50  0001 C CNN
@@
 $EndComp
 $Comp
-L power:GND #PWR?
+L power:GND #PWR037
 U 1 1 6079CFEB
 P 4350 4100
-F 0 "#PWR?" H 4350 3850 50  0001 C CNN
+F 0 "#PWR037" H 4350 3850 50  0001 C CNN
 F 1 "GND" H 4355 3927 50  0000 C CNN
 F 2 "" H 4350 4100 50  0001 C CNN
@@
 $EndComp
 $Comp
-L power:+5V #PWR?
+L power:+5V #PWR036
 U 1 1 6079D620
 P 4350 2800
-F 0 "#PWR?" H 4350 2650 50  0001 C CNN
+F 0 "#PWR036" H 4350 2650 50  0001 C CNN
 F 1 "+5V" V 4365 2928 50  0000 L CNN
 F 2 "" H 4350 2800 50  0001 C CNN
@@
 	3050 4050 2850 4050
 Text HLabel 2850 4050 0    50   Input ~ 0
-A[2:11]
+A[0..15]
 Entry Wire Line
 	5200 3500 5300 3600
@@
 	5200 3200 5300 3300
 NoConn ~ 4850 3700
-Text HLabel 5300 3850 2    50   Input ~ 0
-A[12:15]
 Wire Wire Line
 	5200 3500 4850 3500
@@
 	5200 3200 4850 3200
 NoConn ~ 4850 3100
-Wire Bus Line
-	5300 3200 5300 3850
-Wire Bus Line
-	6600 2150 6600 3000
-Wire Bus Line
-	3050 2700 3050 4050
 Text HLabel 4850 3600 2    50   Input ~ 0
 IO\~M
@@
 Text Label 3400 3950 0    50   ~ 0
 A11
+Wire Bus Line
+	3050 4050 3050 4500
+Wire Bus Line
+	3050 4500 5300 4500
+Connection ~ 3050 4050
+Wire Bus Line
+	5300 3300 5300 4500
+Wire Bus Line
+	6600 2150 6600 3000
+Wire Bus Line
+	3050 2700 3050 4050
 $EndSCHEMATC

Commit message: Add files via upload
Changed lines of the file:
@@
 $Descr A4 11693 8268
 encoding utf-8
-Sheet 7 14
+Sheet 1 1
 Title ""
 Date ""
@@
 NoConn ~ 8250 3250
 NoConn ~ 8250 3350
-Entry Wire Line
-	6600 2850 6700 2950
-Entry Wire Line
-	6600 2750 6700 2850
-Entry Wire Line
-	6600 2650 6700 2750
-Entry Wire Line
-	6600 2550 6700 2650
-Entry Wire Line
-	6600 2450 6700 2550
-Entry Wire Line
-	6600 2350 6700 2450
-Entry Wire Line
-	6600 2250 6700 2350
-Entry Wire Line
-	6600 2150 6700 2250
-Wire Wire Line
-	6700 2250 7050 2250
-Wire Wire Line
-	6700 2350 7050 2350
-Wire Wire Line
-	6700 2450 7050 2450
-Wire Wire Line
-	6700 2550 7050 2550
-Wire Wire Line
-	6700 2650 7050 2650
-Wire Wire Line
-	6700 2750 7050 2750
-Wire Wire Line
-	6700 2850 7050 2850
-Wire Wire Line
-	6700 2950 7050 2950
 Wire Wire Line
 	8250 2850 8450 2850
@@
 	1    0    0    -1
 $EndComp
-Wire Bus Line
-	6300 3000 6600 3000
-Text Label 6850 2250 0    50   ~ 0
-D0
-Text Label 6850 2350 0    50   ~ 0
-D1
-Text Label 6850 2450 0    50   ~ 0
-D2
-Text Label 6850 2550 0    50   ~ 0
-D3
-Text Label 6850 2650 0    50   ~ 0
-D4
-Text Label 6850 2750 0    50   ~ 0
-D5
-Text Label 6850 2850 0    50   ~ 0
-D6
-Text Label 6850 2950 0    50   ~ 0
-D7
 Text HLabel 8450 2850 2    50   Input ~ 0
 8254_counter2
@@
 Text HLabel 6650 3750 0    50   Output ~ 0
 8259INT_Out
-Text HLabel 6300 3000 0    50   BiDi ~ 0
-D[0..7]
 Wire Wire Line
 	7050 3150 6850 3150
@@
 Wire Wire Line
 	5650 3350 7050 3350
-Entry Wire Line
-	3150 3800 3050 3900
-Entry Wire Line
-	3150 3650 3050 3750
-Entry Wire Line
-	3150 3800 3050 3900
-Entry Wire Line
-	3150 3650 3050 3750
-Entry Wire Line
-	3150 3500 3050 3600
-Entry Wire Line
-	3150 3350 3050 3450
-Entry Wire Line
-	3150 3200 3050 3300
-Entry Wire Line
-	3150 3500 3050 3600
-Entry Wire Line
-	3150 3350 3050 3450
-Entry Wire Line
-	3150 3200 3050 3300
-Entry Wire Line
-	3150 3050 3050 3150
-Entry Wire Line
-	3150 3200 3050 3300
-Entry Wire Line
-	3150 3050 3050 3150
-Entry Wire Line
-	3150 3800 3050 3900
-Entry Wire Line
-	3150 3650 3050 3750
-Entry Wire Line
-	3150 3500 3050 3600
-Entry Wire Line
-	3150 3350 3050 3450
-Entry Wire Line
-	3150 3200 3050 3300
-Entry Wire Line
-	3150 3500 3050 3600
-Entry Wire Line
-	3150 3350 3050 3450
-Entry Wire Line
-	3150 3200 3050 3300
-Entry Wire Line
-	3150 3050 3050 3150
-Entry Wire Line
-	3150 3200 3050 3300
-Entry Wire Line
-	3150 3050 3050 3150
-Entry Wire Line
-	3150 2900 3050 3000
-Entry Wire Line
-	3150 2750 3050 2850
-Entry Wire Line
-	3150 3050 3050 3150
-Entry Wire Line
-	3150 2900 3050 3000
-Entry Wire Line
-	3150 2750 3050 2850
-Entry Wire Line
-	3150 2600 3050 2700
-Entry Wire Line
-	3150 2600 3050 2700
-Entry Wire Line
-	3150 2900 3050 3000
-Entry Wire Line
-	3150 2750 3050 2850
-Entry Wire Line
-	3150 2600 3050 2700
-Entry Wire Line
-	3150 2600 3050 2700
-Wire Wire Line
-	3150 2600 3850 2600
 Wire Wire Line
 	3850 2600 3850 3000
 Wire Wire Line
-	3150 2750 3800 2750
-Wire Wire Line
 	3800 2750 3800 3100
 Wire Wire Line
 	3800 3100 3850 3100
 Wire Wire Line
-	3150 2900 3750 2900
-Wire Wire Line
 	3750 2900 3750 3200
 Wire Wire Line
 	3750 3200 3850 3200
 Wire Wire Line
-	3150 3050 3700 3050
-Wire Wire Line
 	3700 3050 3700 3300
 Wire Wire Line
 	3700 3300 3850 3300
 Wire Wire Line
-	3150 3200 3650 3200
-Wire Wire Line
 	3650 3200 3650 3400
 Wire Wire Line
 	3650 3400 3850 3400
 Wire Wire Line
-	3150 3350 3600 3350
-Wire Wire Line
 	3600 3350 3600 3500
 Wire Wire Line
 	3600 3500 3850 3500
 Wire Wire Line
-	3150 3500 3550 3500
-Wire Wire Line
 	3550 3500 3550 3600
 Wire Wire Line
 	3550 3600 3850 3600
 Wire Wire Line
-	3150 3650 3500 3650
-Wire Wire Line
 	3500 3650 3500 3700
 Wire Wire Line
 	3500 3700 3850 3700
 Wire Wire Line
-	3150 3800 3850 3800
-Wire Wire Line
-	3150 3950 3850 3950
-Wire Wire Line
 	3850 3950 3850 3900
-Entry Wire Line
-	3050 4050 3150 3950
-Wire Bus Line
-	3050 4050 2850 4050
-Text HLabel 2850 4050 0    50   Input ~ 0
-A[0..15]
-Entry Wire Line
-	5200 3500 5300 3600
-Entry Wire Line
-	5200 3400 5300 3500
-Entry Wire Line
-	5200 3300 5300 3400
-Entry Wire Line
-	5200 3200 5300 3300
 NoConn ~ 4850 3700
-Wire Wire Line
-	5200 3500 4850 3500
-Wire Wire Line
-	5200 3400 4850 3400
-Wire Wire Line
-	5200 3300 4850 3300
-Wire Wire Line
-	5200 3200 4850 3200
 NoConn ~ 4850 3100
 Text HLabel 4850 3600 2    50   Input ~ 0
 IO\~M
-Text Label 4850 3500 0    50   ~ 0
+Text HLabel 4850 3200 2    50   Input ~ 0
+A15
+Text HLabel 4850 3300 2    50   Input ~ 0
+A14
+Text HLabel 4850 3400 2    50   Input ~ 0
+A13
+Text HLabel 4850 3500 2    50   Input ~ 0
 A12
-Text Label 4850 3400 0    50   ~ 0
-A13
-Text Label 4850 3300 0    50   ~ 0
-A14
-Text Label 4850 3200 0    50   ~ 0
-A15
-Text Label 3650 2600 0    50   ~ 0
+Text HLabel 3850 3950 0    50   Input ~ 0
+A11
+Text HLabel 3850 3800 0    50   Input ~ 0
+A10
+Text HLabel 3500 3650 0    50   Input ~ 0
+A9
+Text HLabel 3550 3500 0    50   Input ~ 0
+A8
+Text HLabel 3600 3350 0    50   Input ~ 0
+A7
+Text HLabel 3650 3200 0    50   Input ~ 0
+A6
+Text HLabel 3700 3050 0    50   Input ~ 0
+A5
+Text HLabel 3750 2900 0    50   Input ~ 0
+A4
+Text HLabel 3800 2750 0    50   Input ~ 0
+A3
+Text HLabel 3850 2600 0    50   Input ~ 0
 A2
-Text Label 3650 2750 0    50   ~ 0
-A3
-Text Label 3650 2900 0    50   ~ 0
-A4
-Text Label 3650 3050 0    50   ~ 0
-A5
-Text Label 3600 3200 0    50   ~ 0
-A6
-Text Label 3550 3350 0    50   ~ 0
-A7
-Text Label 3500 3500 0    50   ~ 0
-A8
-Text Label 3450 3650 0    50   ~ 0
-A9
-Text Label 3400 3800 0    50   ~ 0
-A10
-Text Label 3400 3950 0    50   ~ 0
-A11
-Wire Bus Line
-	3050 4050 3050 4500
-Wire Bus Line
-	3050 4500 5300 4500
-Connection ~ 3050 4050
-Wire Bus Line
-	5300 3300 5300 4500
-Wire Bus Line
-	6600 2150 6600 3000
-Wire Bus Line
-	3050 2700 3050 4050
+Text HLabel 7050 2250 0    50   Input ~ 0
+D0
+Text HLabel 7050 2350 0    50   Input ~ 0
+D1
+Text HLabel 7050 2450 0    50   Input ~ 0
+D2
+Text HLabel 7050 2550 0    50   Input ~ 0
+D3
+Text HLabel 7050 2650 0    50   Input ~ 0
+D4
+Text HLabel 7050 2750 0    50   Input ~ 0
+D5
+Text HLabel 7050 2850 0    50   Input ~ 0
+D6
+Text HLabel 7050 2950 0    50   Input ~ 0
+D7
 $EndSCHEMATC

Commit message: Final?
Parts:
- removed R3: R, symbol Device:R
- added R1: 10000, symbol Device:R_Small_US
- renumbered U25 to 8259INTR1, U24 to 8259Selector1
Connections:
- net +5V: now also R1.1; no longer 8259INTR1.28 (VCC), 8259Selector1.20 (VCC)
- net at 8259INTR1.16 (~SP~/~EN~): now also R1.2
- new net VCC: 8259INTR1.28 (VCC), 8259Selector1.20 (VCC)
Changed lines of the file:
@@
 $EndDescr
 $Comp
-L Interface:8259 U25
+L Interface:8259 8259INTR1
 U 1 1 6078126B
 P 7650 3050
-F 0 "U25" H 7650 4331 50  0000 C CNN
+F 0 "8259INTR1" H 7650 4331 50  0000 C CNN
 F 1 "8259" H 7650 4240 50  0000 C CNN
 F 2 "Package_DIP:DIP-28_W15.24mm" H 7650 3050 50  0001 C CIN
@@
 NoConn ~ 8250 2350
 NoConn ~ 8250 2250
-$Comp
-L power:+5V #PWR040
-U 1 1 6078B521
-P 8800 3550
-F 0 "#PWR040" H 8800 3400 50  0001 C CNN
-F 1 "+5V" V 8815 3678 50  0000 L CNN
-F 2 "" H 8800 3550 50  0001 C CNN
-F 3 "" H 8800 3550 50  0001 C CNN
-	1    8800 3550
-	0    1    1    0
-$EndComp
-$Comp
-L Device:R R3
-U 1 1 6078C718
-P 8500 3550
-F 0 "R3" V 8293 3550 50  0000 C CNN
-F 1 "R" V 8384 3550 50  0000 C CNN
-F 2 "" V 8430 3550 50  0001 C CNN
-F 3 "~" H 8500 3550 50  0001 C CNN
-	1    8500 3550
-	0    1    1    0
-$EndComp
-Wire Wire Line
-	8250 3550 8350 3550
-Wire Wire Line
-	8650 3550 8800 3550
 NoConn ~ 8250 3150
 NoConn ~ 8250 3250
@@
 Wire Wire Line
 	6650 3750 7050 3750
-$Comp
-L power:+5V #PWR039
-U 1 1 60791E23
-P 7850 1950
-F 0 "#PWR039" H 7850 1800 50  0001 C CNN
-F 1 "+5V" V 7865 2078 50  0000 L CNN
-F 2 "" H 7850 1950 50  0001 C CNN
-F 3 "" H 7850 1950 50  0001 C CNN
-	1    7850 1950
-	0    1    1    0
-$EndComp
 Wire Wire Line
 	7850 1950 7650 1950
@@
 	6850 3850 7050 3850
 $Comp
-L Logic_Programmable:PAL16L8 U24
+L Logic_Programmable:PAL16L8 8259Selector1
 U 1 1 60799BF8
 P 4350 3500
-F 0 "U24" H 4350 4381 50  0000 C CNN
+F 0 "8259Selector1" H 4350 4381 50  0000 C CNN
 F 1 "PAL16L8" H 4350 4290 50  0000 C CNN
 F 2 "" H 4350 3500 50  0001 C CNN
@@
 	1    4350 4100
 	1    0    0    -1
-$EndComp
-$Comp
-L power:+5V #PWR036
-U 1 1 6079D620
-P 4350 2800
-F 0 "#PWR036" H 4350 2650 50  0001 C CNN
-F 1 "+5V" V 4365 2928 50  0000 L CNN
-F 2 "" H 4350 2800 50  0001 C CNN
-F 3 "" H 4350 2800 50  0001 C CNN
-	1    4350 2800
-	0    1    1    0
 $EndComp
 Text HLabel 7050 3450 0    50   Input ~ 0
@@
 Text HLabel 7050 2950 0    50   Input ~ 0
 D7
+$Comp
+L power:VCC #PWR0104
+U 1 1 620136AF
+P 7850 1950
+F 0 "#PWR0104" H 7850 1800 50  0001 C CNN
+F 1 "VCC" V 7865 2078 50  0000 L CNN
+F 2 "" H 7850 1950 50  0001 C CNN
+F 3 "" H 7850 1950 50  0001 C CNN
+	1    7850 1950
+	0    1    1    0
+$EndComp
+$Comp
+L power:VCC #PWR0105
+U 1 1 62013B54
+P 4350 2800
+F 0 "#PWR0105" H 4350 2650 50  0001 C CNN
+F 1 "VCC" V 4365 2928 50  0000 L CNN
+F 2 "" H 4350 2800 50  0001 C CNN
+F 3 "" H 4350 2800 50  0001 C CNN
+	1    4350 2800
+	0    1    1    0
+$EndComp
+$Comp
+L Device:R_Small_US R1
+U 1 1 62016C05
+P 8700 3550
+F 0 "R1" V 8495 3550 50  0000 C CNN
+F 1 "10000" V 8586 3550 50  0000 C CNN
+F 2 "" H 8700 3550 50  0001 C CNN
+F 3 "~" H 8700 3550 50  0001 C CNN
+	1    8700 3550
+	0    1    1    0
+$EndComp
+$Comp
+L power:+5V #PWR02
+U 1 1 6201736A
+P 9100 3550
+F 0 "#PWR02" H 9100 3400 50  0001 C CNN
+F 1 "+5V" V 9115 3678 50  0000 L CNN
+F 2 "" H 9100 3550 50  0001 C CNN
+F 3 "" H 9100 3550 50  0001 C CNN
+	1    9100 3550
+	0    1    1    0
+$EndComp
+Wire Wire Line
+	9100 3550 8800 3550
+Wire Wire Line
+	8250 3550 8600 3550
 $EndSCHEMATC

Commit message: Final..I Hope
Parts:
- 8259Selector1: footprint (none) -> Package_DIP:DIP-20_W7.62mm
Changed lines of the file:
@@
 F 0 "8259Selector1" H 4350 4381 50  0000 C CNN
 F 1 "PAL16L8" H 4350 4290 50  0000 C CNN
-F 2 "" H 4350 3500 50  0001 C CNN
+F 2 "Package_DIP:DIP-20_W7.62mm" H 4350 3500 50  0001 C CNN
 F 3 "" H 4350 3500 50  0001 C CNN
 	1    4350 3500

Commit message: Hopefully the board is here
Parts:
- R1: footprint (none) -> Resistor_THT:R_Axial_DIN0204_L3.6mm_D1.6mm_P2.54mm_Vertical
- SW3: footprint (none) -> Button_Switch_THT:SW_PUSH-12mm
Changed lines of the file:
@@
 F 0 "SW3" H 9500 3235 50  0000 C CNN
 F 1 "SW_Push" H 9500 3144 50  0000 C CNN
-F 2 "" H 9500 3150 50  0001 C CNN
+F 2 "Button_Switch_THT:SW_PUSH-12mm" H 9500 3150 50  0001 C CNN
 F 3 "~" H 9500 3150 50  0001 C CNN
 	1    9500 2950
@@
 F 0 "R1" V 8495 3550 50  0000 C CNN
 F 1 "10000" V 8586 3550 50  0000 C CNN
-F 2 "" H 8700 3550 50  0001 C CNN
+F 2 "Resistor_THT:R_Axial_DIN0204_L3.6mm_D1.6mm_P2.54mm_Vertical" H 8700 3550 50  0001 C CNN
 F 3 "~" H 8700 3550 50  0001 C CNN
 	1    8700 3550
