File: Final/8279(FINAL).sch (KiCad schematic (older format))
At the start: 24 parts, among them SW00 SW_Push, SW01 SW_Push, SW02 SW_Push, SW03 SW_Push, SW10 SW_Push, SW11 SW_Push, SW12 SW_Push, SW13 SW_Push, SW20 SW_Push, SW21 SW_Push, SW22 SW_Push, SW23 SW_Push, SW30 SW_Push, SW31 SW_Push, SW32 SW_Push, SW33 SW_Push

Commit message: New stuff
Parts:
- gave numbers to parts that had none: 8
- renumbered SW21 to SW10, SW31 to SW11, SW02 to SW12, SW12 to SW13, SW22 to SW14, SW32 to SW15, SW03 to SW16, SW13 to SW17, SW23 to SW18, SW33 to SW19, SW00 to SW4, SW10 to SW5, SW20 to SW6, SW30 to SW7, SW01 to SW8, SW11 to SW9
Changed lines of the file:
@@
 $EndDescr
 $Comp
-L pkd8279:pkd8279 U?
+L pkd8279:pkd8279 U28
 U 1 1 60761D14
 P 1850 3300
-F 0 "U?" H 2875 3687 60  0000 C CNN
+F 0 "U28" H 2875 3687 60  0000 C CNN
 F 1 "pkd8279" H 2875 3581 60  0000 C CNN
 F 2 "pkd8279" H 2850 3690 60  0001 C CNN
@@
 $EndComp
 $Comp
-L Switch:SW_Push SW00
+L Switch:SW_Push SW4
 U 1 1 6076E12A
 P 5800 2550
-F 0 "SW00" H 5800 2835 50  0000 C CNN
+F 0 "SW4" H 5800 2835 50  0000 C CNN
 F 1 "SW_Push" H 5800 2744 50  0000 C CNN
 F 2 "" H 5800 2750 50  0001 C CNN
@@
 Row0
 $Comp
-L Switch:SW_Push SW01
+L Switch:SW_Push SW8
 U 1 1 607E3FBB
 P 6650 2550
-F 0 "SW01" H 6650 2835 50  0000 C CNN
+F 0 "SW8" H 6650 2835 50  0000 C CNN
 F 1 "SW_Push" H 6650 2744 50  0000 C CNN
 F 2 "" H 6650 2750 50  0001 C CNN
@@
 	6450 2550 6450 2750
 $Comp
-L Switch:SW_Push SW02
+L Switch:SW_Push SW12
 U 1 1 607E4505
 P 7500 2550
-F 0 "SW02" H 7500 2835 50  0000 C CNN
+F 0 "SW12" H 7500 2835 50  0000 C CNN
 F 1 "SW_Push" H 7500 2744 50  0000 C CNN
 F 2 "" H 7500 2750 50  0001 C CNN
@@
 	7300 2550 7300 2750
 $Comp
-L Switch:SW_Push SW03
+L Switch:SW_Push SW16
 U 1 1 607E4DCD
 P 8350 2550
-F 0 "SW03" H 8350 2835 50  0000 C CNN
+F 0 "SW16" H 8350 2835 50  0000 C CNN
 F 1 "SW_Push" H 8350 2744 50  0000 C CNN
 F 2 "" H 8350 2750 50  0001 C CNN
@@
 	8150 2550 8150 2750
 $Comp
-L Switch:SW_Push SW10
+L Switch:SW_Push SW5
 U 1 1 607F069D
 P 5800 3150
-F 0 "SW10" H 5800 3435 50  0000 C CNN
+F 0 "SW5" H 5800 3435 50  0000 C CNN
 F 1 "SW_Push" H 5800 3344 50  0000 C CNN
 F 2 "" H 5800 3350 50  0001 C CNN
@@
 Row1
 $Comp
-L Switch:SW_Push SW11
+L Switch:SW_Push SW9
 U 1 1 607F06AC
 P 6650 3150
-F 0 "SW11" H 6650 3435 50  0000 C CNN
+F 0 "SW9" H 6650 3435 50  0000 C CNN
 F 1 "SW_Push" H 6650 3344 50  0000 C CNN
 F 2 "" H 6650 3350 50  0001 C CNN
@@
 Connection ~ 7000 3150
 $Comp
-L Switch:SW_Push SW12
+L Switch:SW_Push SW13
 U 1 1 607F06B7
 P 7500 3150
-F 0 "SW12" H 7500 3435 50  0000 C CNN
+F 0 "SW13" H 7500 3435 50  0000 C CNN
 F 1 "SW_Push" H 7500 3344 50  0000 C CNN
 F 2 "" H 7500 3350 50  0001 C CNN
@@
 Connection ~ 7850 3150
 $Comp
-L Switch:SW_Push SW13
+L Switch:SW_Push SW17
 U 1 1 607F06C2
 P 8350 3150
-F 0 "SW13" H 8350 3435 50  0000 C CNN
+F 0 "SW17" H 8350 3435 50  0000 C CNN
 F 1 "SW_Push" H 8350 3344 50  0000 C CNN
 F 2 "" H 8350 3350 50  0001 C CNN
@@
 	8700 2550 8700 3150
 $Comp
-L Switch:SW_Push SW20
+L Switch:SW_Push SW6
 U 1 1 607F452D
 P 5800 3750
-F 0 "SW20" H 5800 4035 50  0000 C CNN
+F 0 "SW6" H 5800 4035 50  0000 C CNN
 F 1 "SW_Push" H 5800 3944 50  0000 C CNN
 F 2 "" H 5800 3950 50  0001 C CNN
@@
 Row2
 $Comp
-L Switch:SW_Push SW21
+L Switch:SW_Push SW10
 U 1 1 607F453C
 P 6650 3750
-F 0 "SW21" H 6650 4035 50  0000 C CNN
+F 0 "SW10" H 6650 4035 50  0000 C CNN
 F 1 "SW_Push" H 6650 3944 50  0000 C CNN
 F 2 "" H 6650 3950 50  0001 C CNN
@@
 Connection ~ 7000 3750
 $Comp
-L Switch:SW_Push SW22
+L Switch:SW_Push SW14
 U 1 1 607F4547
 P 7500 3750
-F 0 "SW22" H 7500 4035 50  0000 C CNN
+F 0 "SW14" H 7500 4035 50  0000 C CNN
 F 1 "SW_Push" H 7500 3944 50  0000 C CNN
 F 2 "" H 7500 3950 50  0001 C CNN
@@
 Connection ~ 7850 3750
 $Comp
-L Switch:SW_Push SW23
+L Switch:SW_Push SW18
 U 1 1 607F4552
 P 8350 3750
-F 0 "SW23" H 8350 4035 50  0000 C CNN
+F 0 "SW18" H 8350 4035 50  0000 C CNN
 F 1 "SW_Push" H 8350 3944 50  0000 C CNN
 F 2 "" H 8350 3950 50  0001 C CNN
@@
 	8700 3150 8700 3750
 $Comp
-L Switch:SW_Push SW30
+L Switch:SW_Push SW7
 U 1 1 607FB339
 P 5800 4350
-F 0 "SW30" H 5800 4635 50  0000 C CNN
+F 0 "SW7" H 5800 4635 50  0000 C CNN
 F 1 "SW_Push" H 5800 4544 50  0000 C CNN
 F 2 "" H 5800 4550 50  0001 C CNN
@@
 Row3
 $Comp
-L Switch:SW_Push SW31
+L Switch:SW_Push SW11
 U 1 1 607FB348
 P 6650 4350
-F 0 "SW31" H 6650 4635 50  0000 C CNN
+F 0 "SW11" H 6650 4635 50  0000 C CNN
 F 1 "SW_Push" H 6650 4544 50  0000 C CNN
 F 2 "" H 6650 4550 50  0001 C CNN
@@
 	6450 4350 6450 4550
 $Comp
-L Switch:SW_Push SW32
+L Switch:SW_Push SW15
 U 1 1 607FB353
 P 7500 4350
-F 0 "SW32" H 7500 4635 50  0000 C CNN
+F 0 "SW15" H 7500 4635 50  0000 C CNN
 F 1 "SW_Push" H 7500 4544 50  0000 C CNN
 F 2 "" H 7500 4550 50  0001 C CNN
@@
 	7300 4350 7300 4550
 $Comp
-L Switch:SW_Push SW33
+L Switch:SW_Push SW19
 U 1 1 607FB35E
 P 8350 4350
-F 0 "SW33" H 8350 4635 50  0000 C CNN
+F 0 "SW19" H 8350 4635 50  0000 C CNN
 F 1 "SW_Push" H 8350 4544 50  0000 C CNN
 F 2 "" H 8350 4550 50  0001 C CNN
@@
 Row3
 $Comp
-L Switch:SW_Push SW?
+L Switch:SW_Push SW24
 U 1 1 608318B0
 P 10000 2750
-F 0 "SW?" H 10000 3035 50  0000 C CNN
+F 0 "SW24" H 10000 3035 50  0000 C CNN
 F 1 "SW_Push" H 10000 2944 50  0000 C CNN
 F 2 "" H 10000 2950 50  0001 C CNN
@@
 	9800 2750 9800 2950
 $Comp
-L Switch:SW_Push SW?
+L Switch:SW_Push SW25
 U 1 1 60833F86
 P 10050 3900
-F 0 "SW?" H 10050 4185 50  0000 C CNN
+F 0 "SW25" H 10050 4185 50  0000 C CNN
 F 1 "SW_Push" H 10050 4094 50  0000 C CNN
 F 2 "" H 10050 4100 50  0001 C CNN
@@
 	9850 3900 9850 4100
 $Comp
-L power:GND #PWR?
+L power:GND #PWR051
 U 1 1 60836773
 P 10400 4100
-F 0 "#PWR?" H 10400 3850 50  0001 C CNN
+F 0 "#PWR051" H 10400 3850 50  0001 C CNN
 F 1 "GND" H 10405 3927 50  0000 C CNN
 F 2 "" H 10400 4100 50  0001 C CNN
@@
 $EndComp
 $Comp
-L power:GND #PWR?
+L power:GND #PWR050
 U 1 1 60837AE5
 P 10350 2950
-F 0 "#PWR?" H 10350 2700 50  0001 C CNN
+F 0 "#PWR050" H 10350 2700 50  0001 C CNN
 F 1 "GND" H 10355 2777 50  0000 C CNN
 F 2 "" H 10350 2950 50  0001 C CNN
@@
 NoConn ~ 3900 4900
 $Comp
-L Switch:SW_Push SW?
+L Switch:SW_Push SW20
 U 1 1 608CF75F
 P 9200 2550
-F 0 "SW?" H 9200 2835 50  0000 C CNN
+F 0 "SW20" H 9200 2835 50  0000 C CNN
 F 1 "SW_Push" H 9200 2744 50  0000 C CNN
 F 2 "" H 9200 2750 50  0001 C CNN
@@
 	9000 2550 9000 2750
 $Comp
-L Switch:SW_Push SW?
+L Switch:SW_Push SW21
 U 1 1 608CF767
 P 9200 3150
-F 0 "SW?" H 9200 3435 50  0000 C CNN
+F 0 "SW21" H 9200 3435 50  0000 C CNN
 F 1 "SW_Push" H 9200 3344 50  0000 C CNN
 F 2 "" H 9200 3350 50  0001 C CNN
@@
 	9000 3150 9000 3350
 $Comp
-L Switch:SW_Push SW?
+L Switch:SW_Push SW22
 U 1 1 608CF76F
 P 9200 3750
-F 0 "SW?" H 9200 4035 50  0000 C CNN
+F 0 "SW22" H 9200 4035 50  0000 C CNN
 F 1 "SW_Push" H 9200 3944 50  0000 C CNN
 F 2 "" H 9200 3950 50  0001 C CNN
@@
 	9000 3750 9000 3950
 $Comp
-L Switch:SW_Push SW?
+L Switch:SW_Push SW23
 U 1 1 608CF777
 P 9200 4350
-F 0 "SW?" H 9200 4635 50  0000 C CNN
+F 0 "SW23" H 9200 4635 50  0000 C CNN
 F 1 "SW_Push" H 9200 4544 50  0000 C CNN
 F 2 "" H 9200 4550 50  0001 C CNN
@@
 	1600 3600 1850 3600
 Text HLabel 1100 5150 0    50   BiDi ~ 0
-D[0:7]
+D[0..7]
 Wire Bus Line
 	1300 5150 1100 5150
 $Comp
-L power:+5V #PWR?
+L power:+5V #PWR047
 U 1 1 607EFF38
 P 3900 3300
-F 0 "#PWR?" H 3900 3150 50  0001 C CNN
+F 0 "#PWR047" H 3900 3150 50  0001 C CNN
 F 1 "+5V" H 3915 3473 50  0000 C CNN
 F 2 "" H 3900 3300 50  0001 C CNN
@@
 PCLK
 $Comp
-L power:GND #PWR?
+L power:GND #PWR046
 U 1 1 607F178F
 P 1850 5200
-F 0 "#PWR?" H 1850 4950 50  0001 C CNN
+F 0 "#PWR046" H 1850 4950 50  0001 C CNN
 F 1 "GND" H 1855 5027 50  0000 C CNN
 F 2 "" H 1850 5200 50  0001 C CNN
@@
 8086_A1
 $Comp
-L Logic_Programmable:PAL16L8 U?
+L Logic_Programmable:PAL16L8 U29
 U 1 1 607FB29D
 P 4900 6200
-F 0 "U?" H 4900 7081 50  0000 C CNN
+F 0 "U29" H 4900 7081 50  0000 C CNN
 F 1 "PAL16L8" H 4900 6990 50  0000 C CNN
 F 2 "" H 4900 6200 50  0001 C CNN
@@
 $EndComp
 $Comp
-L power:GND #PWR?
+L power:GND #PWR049
 U 1 1 607FE8E4
 P 4900 6800
-F 0 "#PWR?" H 4900 6550 50  0001 C CNN
+F 0 "#PWR049" H 4900 6550 50  0001 C CNN
 F 1 "GND" H 4905 6627 50  0000 C CNN
 F 2 "" H 4900 6800 50  0001 C CNN
@@
 $EndComp
 $Comp
-L power:+5V #PWR?
+L power:+5V #PWR048
 U 1 1 607FF81B
 P 4900 5500
-F 0 "#PWR?" H 4900 5350 50  0001 C CNN
+F 0 "#PWR048" H 4900 5350 50  0001 C CNN
 F 1 "+5V" V 4915 5628 50  0000 L CNN
 F 2 "" H 4900 5500 50  0001 C CNN
@@
 	5800 6300 5900 6300
 Text HLabel 5900 6300 2    50   Input ~ 0
-A[12:15]
+A[12..15]
 Text HLabel 5400 6300 2    50   Input ~ 0
 IO\~M
 NoConn ~ 5400 6400
 NoConn ~ 5400 5800
-Wire Bus Line
-	5800 6000 5800 6300
-Wire Bus Line
-	3900 5600 3900 6650
-Wire Bus Line
-	1300 4300 1300 5150
 Text Label 5500 5900 0    50   ~ 0
 A15
@@
 A11
 Text HLabel 3900 6650 0    50   Input ~ 0
-A[2:11]
+A[2..11]
+Wire Bus Line
+	5800 6000 5800 6300
+Wire Bus Line
+	3900 5600 3900 6650
+Wire Bus Line
+	1300 4300 1300 5150
 $EndSCHEMATC

Commit message: Add files via upload
Connections:
- net D0: now reaches U28.12 (DB0)
- net D1: now reaches U28.13 (DB1)
- net D2: now reaches U28.14 (DB2)
- net D3: now reaches U28.15 (DB3)
- net D4: now reaches U28.16 (DB4)
- net D5: now reaches U28.17 (DB5)
- net D6: now reaches U28.18 (DB6)
- net D7: now reaches U28.19 (DB7)
Changed lines of the file:
@@
 $Descr A4 11693 8268
 encoding utf-8
-Sheet 9 14
+Sheet 1 1
 Title ""
 Date ""
@@
 Text Label 1700 3700 0    50   ~ 0
 Col4
-Wire Wire Line
-	1850 4500 1400 4500
-Wire Wire Line
-	1850 4600 1400 4600
-Wire Wire Line
-	1850 4700 1400 4700
-Wire Wire Line
-	1850 4800 1400 4800
-Wire Wire Line
-	1850 4900 1400 4900
-Wire Wire Line
-	1850 5000 1400 5000
-Wire Wire Line
-	1850 5100 1400 5100
-Wire Wire Line
-	1850 4400 1400 4400
-Entry Wire Line
-	1300 4300 1400 4400
-Entry Wire Line
-	1300 4300 1400 4400
-Entry Wire Line
-	1300 4400 1400 4500
-Entry Wire Line
-	1300 4500 1400 4600
-Entry Wire Line
-	1300 4600 1400 4700
-Entry Wire Line
-	1300 4700 1400 4800
-Entry Wire Line
-	1300 4800 1400 4900
-Entry Wire Line
-	1300 4900 1400 5000
-Entry Wire Line
-	1300 5000 1400 5100
 NoConn ~ 1850 3800
 NoConn ~ 1850 3900
@@
 Wire Wire Line
 	1600 3600 1850 3600
-Text HLabel 1100 5150 0    50   BiDi ~ 0
-D[0..7]
-Wire Bus Line
-	1300 5150 1100 5150
 $Comp
 L power:+5V #PWR047
@@
 	0    1    1    0
 $EndComp
-Entry Wire Line
-	3900 6300 4000 6400
-Entry Wire Line
-	3900 6200 4000 6300
-Entry Wire Line
-	3900 6100 4000 6200
-Entry Wire Line
-	3900 6000 4000 6100
-Entry Wire Line
-	3900 5900 4000 6000
-Entry Wire Line
-	3900 5800 4000 5900
-Entry Wire Line
-	3900 5700 4000 5800
-Entry Wire Line
-	3900 5600 4000 5700
-Wire Wire Line
-	4000 5700 4400 5700
-Wire Wire Line
-	4000 5800 4400 5800
-Wire Wire Line
-	4000 5900 4400 5900
-Wire Wire Line
-	4000 6000 4400 6000
-Wire Wire Line
-	4000 6100 4400 6100
-Wire Wire Line
-	4000 6200 4400 6200
-Wire Wire Line
-	4000 6300 4400 6300
-Wire Wire Line
-	4000 6400 4400 6400
-Wire Wire Line
-	4400 6500 4000 6500
-Wire Wire Line
-	4400 6600 4000 6600
-Entry Wire Line
-	3900 6500 4000 6600
-Entry Wire Line
-	3900 6400 4000 6500
-Entry Wire Line
-	5700 5900 5800 6000
-Entry Wire Line
-	5700 6000 5800 6100
-Entry Wire Line
-	5700 6100 5800 6200
-Entry Wire Line
-	5700 6200 5800 6300
-Wire Wire Line
-	5400 5900 5700 5900
-Wire Wire Line
-	5400 6000 5700 6000
-Wire Wire Line
-	5400 6100 5700 6100
 Wire Wire Line
 	3900 5100 5650 5100
@@
 Text Label 5450 5700 0    50   ~ 0
 CS
-Wire Wire Line
-	5400 6200 5700 6200
-Wire Bus Line
-	5800 6300 5900 6300
-Text HLabel 5900 6300 2    50   Input ~ 0
-A[12..15]
 Text HLabel 5400 6300 2    50   Input ~ 0
 IO\~M
 NoConn ~ 5400 6400
 NoConn ~ 5400 5800
-Text Label 5500 5900 0    50   ~ 0
+Text HLabel 1850 4400 0    50   Input ~ 0
+D0
+Text HLabel 1850 4500 0    50   Input ~ 0
+D1
+Text HLabel 1850 4600 0    50   Input ~ 0
+D2
+Text HLabel 1850 4700 0    50   Input ~ 0
+D3
+Text HLabel 1850 4800 0    50   Input ~ 0
+D4
+Text HLabel 1850 4900 0    50   Input ~ 0
+D5
+Text HLabel 1850 5000 0    50   Input ~ 0
+D6
+Text HLabel 1850 5100 0    50   Input ~ 0
+D7
+Text HLabel 4400 5700 0    50   Input ~ 0
+A2
+Text HLabel 4400 6600 0    50   Input ~ 0
+A11
+Text HLabel 4400 6500 0    50   Input ~ 0
+A10
+Text HLabel 4400 6400 0    50   Input ~ 0
+A9
+Text HLabel 4400 6300 0    50   Input ~ 0
+A8
+Text HLabel 4400 6200 0    50   Input ~ 0
+A7
+Text HLabel 4400 6100 0    50   Input ~ 0
+A6
+Text HLabel 4400 6000 0    50   Input ~ 0
+A5
+Text HLabel 4400 5900 0    50   Input ~ 0
+A4
+Text HLabel 4400 5800 0    50   Input ~ 0
+A3
+Text HLabel 5400 5900 2    50   Input ~ 0
 A15
-Text Label 5500 6000 0    50   ~ 0
+Text HLabel 5400 6000 2    50   Input ~ 0
 A14
-Text Label 5500 6100 0    50   ~ 0
+Text HLabel 5400 6100 2    50   Input ~ 0
 A13
-Text Label 5500 6200 0    50   ~ 0
+Text HLabel 5400 6200 2    50   Input ~ 0
 A12
-Text Label 4300 5700 0    50   ~ 0
-A2
-Text Label 4300 5800 0    50   ~ 0
-A3
-Text Label 4300 5900 0    50   ~ 0
-A4
-Text Label 4300 6000 0    50   ~ 0
-A5
-Text Label 4300 6100 0    50   ~ 0
-A6
-Text Label 4300 6200 0    50   ~ 0
-A7
-Text Label 4300 6300 0    50   ~ 0
-A8
-Text Label 4300 6400 0    50   ~ 0
-A9
-Text Label 4300 6500 0    50   ~ 0
-A10
-Text Label 4300 6600 0    50   ~ 0
-A11
-Text HLabel 3900 6650 0    50   Input ~ 0
-A[2..11]
-Wire Bus Line
-	5800 6000 5800 6300
-Wire Bus Line
-	3900 5600 3900 6650
-Wire Bus Line
-	1300 4300 1300 5150
 $EndSCHEMATC

Commit message: Final?
Parts:
- renumbered U28 to 8279Keyboard1, U29 to KeyboardSelector1
Changed lines of the file:
@@
 $EndDescr
 $Comp
-L pkd8279:pkd8279 U28
+L pkd8279:pkd8279 8279Keyboard1
 U 1 1 60761D14
 P 1850 3300
-F 0 "U28" H 2875 3687 60  0000 C CNN
+F 0 "8279Keyboard1" H 2875 3687 60  0000 C CNN
 F 1 "pkd8279" H 2875 3581 60  0000 C CNN
 F 2 "pkd8279" H 2850 3690 60  0001 C CNN
@@
 8086_A1
 $Comp
-L Logic_Programmable:PAL16L8 U29
+L Logic_Programmable:PAL16L8 KeyboardSelector1
 U 1 1 607FB29D
 P 4900 6200
-F 0 "U29" H 4900 7081 50  0000 C CNN
+F 0 "KeyboardSelector1" H 4900 7081 50  0000 C CNN
 F 1 "PAL16L8" H 4900 6990 50  0000 C CNN
 F 2 "" H 4900 6200 50  0001 C CNN

Commit message: Final..I Hope
Parts:
- 8279Keyboard1: footprint pkd8279 -> (none)
Changed lines of the file:
@@
 F 0 "8279Keyboard1" H 2875 3687 60  0000 C CNN
 F 1 "pkd8279" H 2875 3581 60  0000 C CNN
-F 2 "pkd8279" H 2850 3690 60  0001 C CNN
+F 2 "" H 2850 3690 60  0001 C CNN
 F 3 "" H 1850 3300 60  0000 C CNN
 	1    1850 3300

Commit message: Hopefully the board is here
Parts:
- 8279Keyboard1: footprint (none) -> Package_DIP:DIP-40_W15.24mm
- KeyboardSelector1: footprint (none) -> Package_DIP:DIP-20_W7.62mm
- SW10, SW11, SW12, SW13, SW14, SW15, SW16, SW17, SW18, SW19, SW20, SW21, SW22, SW23, SW24, SW25, SW4, SW5, SW6, SW7, SW8, SW9: footprint (none) -> Button_Switch_THT:SW_PUSH-12mm
Changed lines of the file:
@@
 F 0 "8279Keyboard1" H 2875 3687 60  0000 C CNN
 F 1 "pkd8279" H 2875 3581 60  0000 C CNN
-F 2 "" H 2850 3690 60  0001 C CNN
+F 2 "Package_DIP:DIP-40_W15.24mm" H 2850 3690 60  0001 C CNN
 F 3 "" H 1850 3300 60  0000 C CNN
 	1    1850 3300
@@
 F 0 "SW4" H 5800 2835 50  0000 C CNN
 F 1 "SW_Push" H 5800 2744 50  0000 C CNN
-F 2 "" H 5800 2750 50  0001 C CNN
+F 2 "Button_Switch_THT:SW_PUSH-12mm" H 5800 2750 50  0001 C CNN
 F 3 "~" H 5800 2750 50  0001 C CNN
 	1    5800 2550
@@
 F 0 "SW8" H 6650 2835 50  0000 C CNN
 F 1 "SW_Push" H 6650 2744 50  0000 C CNN
-F 2 "" H 6650 2750 50  0001 C CNN
+F 2 "Button_Switch_THT:SW_PUSH-12mm" H 6650 2750 50  0001 C CNN
 F 3 "~" H 6650 2750 50  0001 C CNN
 	1    6650 2550
@@
 F 0 "SW12" H 7500 2835 50  0000 C CNN
 F 1 "SW_Push" H 7500 2744 50  0000 C CNN
-F 2 "" H 7500 2750 50  0001 C CNN
+F 2 "Button_Switch_THT:SW_PUSH-12mm" H 7500 2750 50  0001 C CNN
 F 3 "~" H 7500 2750 50  0001 C CNN
 	1    7500 2550
@@
 F 0 "SW16" H 8350 2835 50  0000 C CNN
 F 1 "SW_Push" H 8350 2744 50  0000 C CNN
-F 2 "" H 8350 2750 50  0001 C CNN
+F 2 "Button_Switch_THT:SW_PUSH-12mm" H 8350 2750 50  0001 C CNN
 F 3 "~" H 8350 2750 50  0001 C CNN
 	1    8350 2550
@@
 F 0 "SW5" H 5800 3435 50  0000 C CNN
 F 1 "SW_Push" H 5800 3344 50  0000 C CNN
-F 2 "" H 5800 3350 50  0001 C CNN
+F 2 "Button_Switch_THT:SW_PUSH-12mm" H 5800 3350 50  0001 C CNN
 F 3 "~" H 5800 3350 50  0001 C CNN
 	1    5800 3150
@@
 F 0 "SW9" H 6650 3435 50  0000 C CNN
 F 1 "SW_Push" H 6650 3344 50  0000 C CNN
-F 2 "" H 6650 3350 50  0001 C CNN
+F 2 "Button_Switch_THT:SW_PUSH-12mm" H 6650 3350 50  0001 C CNN
 F 3 "~" H 6650 3350 50  0001 C CNN
 	1    6650 3150
@@
 F 0 "SW13" H 7500 3435 50  0000 C CNN
 F 1 "SW_Push" H 7500 3344 50  0000 C CNN
-F 2 "" H 7500 3350 50  0001 C CNN
+F 2 "Button_Switch_THT:SW_PUSH-12mm" H 7500 3350 50  0001 C CNN
 F 3 "~" H 7500 3350 50  0001 C CNN
 	1    7500 3150
@@
 F 0 "SW17" H 8350 3435 50  0000 C CNN
 F 1 "SW_Push" H 8350 3344 50  0000 C CNN
-F 2 "" H 8350 3350 50  0001 C CNN
+F 2 "Button_Switch_THT:SW_PUSH-12mm" H 8350 3350 50  0001 C CNN
 F 3 "~" H 8350 3350 50  0001 C CNN
 	1    8350 3150
@@
 F 0 "SW6" H 5800 4035 50  0000 C CNN
 F 1 "SW_Push" H 5800 3944 50  0000 C CNN
-F 2 "" H 5800 3950 50  0001 C CNN
+F 2 "Button_Switch_THT:SW_PUSH-12mm" H 5800 3950 50  0001 C CNN
 F 3 "~" H 5800 3950 50  0001 C CNN
 	1    5800 3750
@@
 F 0 "SW10" H 6650 4035 50  0000 C CNN
 F 1 "SW_Push" H 6650 3944 50  0000 C CNN
-F 2 "" H 6650 3950 50  0001 C CNN
+F 2 "Button_Switch_THT:SW_PUSH-12mm" H 6650 3950 50  0001 C CNN
 F 3 "~" H 6650 3950 50  0001 C CNN
 	1    6650 3750
@@
 F 0 "SW14" H 7500 4035 50  0000 C CNN
 F 1 "SW_Push" H 7500 3944 50  0000 C CNN
-F 2 "" H 7500 3950 50  0001 C CNN
+F 2 "Button_Switch_THT:SW_PUSH-12mm" H 7500 3950 50  0001 C CNN
 F 3 "~" H 7500 3950 50  0001 C CNN
 	1    7500 3750
@@
 F 0 "SW18" H 8350 4035 50  0000 C CNN
 F 1 "SW_Push" H 8350 3944 50  0000 C CNN
-F 2 "" H 8350 3950 50  0001 C CNN
+F 2 "Button_Switch_THT:SW_PUSH-12mm" H 8350 3950 50  0001 C CNN
 F 3 "~" H 8350 3950 50  0001 C CNN
 	1    8350 3750
@@
 F 0 "SW7" H 5800 4635 50  0000 C CNN
 F 1 "SW_Push" H 5800 4544 50  0000 C CNN
-F 2 "" H 5800 4550 50  0001 C CNN
+F 2 "Button_Switch_THT:SW_PUSH-12mm" H 5800 4550 50  0001 C CNN
 F 3 "~" H 5800 4550 50  0001 C CNN
 	1    5800 4350
@@
 F 0 "SW11" H 6650 4635 50  0000 C CNN
 F 1 "SW_Push" H 6650 4544 50  0000 C CNN
-F 2 "" H 6650 4550 50  0001 C CNN
+F 2 "Button_Switch_THT:SW_PUSH-12mm" H 6650 4550 50  0001 C CNN
 F 3 "~" H 6650 4550 50  0001 C CNN
 	1    6650 4350
@@
 F 0 "SW15" H 7500 4635 50  0000 C CNN
 F 1 "SW_Push" H 7500 4544 50  0000 C CNN
-F 2 "" H 7500 4550 50  0001 C CNN
+F 2 "Button_Switch_THT:SW_PUSH-12mm" H 7500 4550 50  0001 C CNN
 F 3 "~" H 7500 4550 50  0001 C CNN
 	1    7500 4350
@@
 F 0 "SW19" H 8350 4635 50  0000 C CNN
 F 1 "SW_Push" H 8350 4544 50  0000 C CNN
-F 2 "" H 8350 4550 50  0001 C CNN
+F 2 "Button_Switch_THT:SW_PUSH-12mm" H 8350 4550 50  0001 C CNN
 F 3 "~" H 8350 4550 50  0001 C CNN
 	1    8350 4350
@@
 F 0 "SW24" H 10000 3035 50  0000 C CNN
 F 1 "SW_Push" H 10000 2944 50  0000 C CNN
-F 2 "" H 10000 2950 50  0001 C CNN
+F 2 "Button_Switch_THT:SW_PUSH-12mm" H 10000 2950 50  0001 C CNN
 F 3 "~" H 10000 2950 50  0001 C CNN
 	1    10000 2750
@@
 F 0 "SW25" H 10050 4185 50  0000 C CNN
 F 1 "SW_Push" H 10050 4094 50  0000 C CNN
-F 2 "" H 10050 4100 50  0001 C CNN
+F 2 "Button_Switch_THT:SW_PUSH-12mm" H 10050 4100 50  0001 C CNN
 F 3 "~" H 10050 4100 50  0001 C CNN
 	1    10050 3900
@@
 F 0 "SW20" H 9200 2835 50  0000 C CNN
 F 1 "SW_Push" H 9200 2744 50  0000 C CNN
-F 2 "" H 9200 2750 50  0001 C CNN
+F 2 "Button_Switch_THT:SW_PUSH-12mm" H 9200 2750 50  0001 C CNN
 F 3 "~" H 9200 2750 50  0001 C CNN
 	1    9200 2550
@@
 F 0 "SW21" H 9200 3435 50  0000 C CNN
 F 1 "SW_Push" H 9200 3344 50  0000 C CNN
-F 2 "" H 9200 3350 50  0001 C CNN
+F 2 "Button_Switch_THT:SW_PUSH-12mm" H 9200 3350 50  0001 C CNN
 F 3 "~" H 9200 3350 50  0001 C CNN
 	1    9200 3150
@@
 F 0 "SW22" H 9200 4035 50  0000 C CNN
 F 1 "SW_Push" H 9200 3944 50  0000 C CNN
-F 2 "" H 9200 3950 50  0001 C CNN
+F 2 "Button_Switch_THT:SW_PUSH-12mm" H 9200 3950 50  0001 C CNN
 F 3 "~" H 9200 3950 50  0001 C CNN
 	1    9200 3750
@@
 F 0 "SW23" H 9200 4635 50  0000 C CNN
 F 1 "SW_Push" H 9200 4544 50  0000 C CNN
-F 2 "" H 9200 4550 50  0001 C CNN
+F 2 "Button_Switch_THT:SW_PUSH-12mm" H 9200 4550 50  0001 C CNN
 F 3 "~" H 9200 4550 50  0001 C CNN
 	1    9200 4350
@@
 F 0 "KeyboardSelector1" H 4900 7081 50  0000 C CNN
 F 1 "PAL16L8" H 4900 6990 50  0000 C CNN
-F 2 "" H 4900 6200 50  0001 C CNN
+F 2 "Package_DIP:DIP-20_W7.62mm" H 4900 6200 50  0001 C CNN
 F 3 "" H 4900 6200 50  0001 C CNN
 	1    4900 6200
