File: Final/Display(FIANL).sch (KiCad schematic (older format))
At the start: 25 parts

Commit message: Hopefully the board is here
Parts:
- D2, D3, D4, D5, D6, D7, D8, D9: footprint (none) -> LED_THT:LED_D1.8mm_W1.8mm_H2.4mm_Horizontal_O1.27mm_Z4.9mm
- Display1, Display2, Display3, Display_Decode1, Display_Decode2: footprint (none) -> Package_DIP:DIP-20_W7.62mm
- R10, R11, R12, R13, R4, R5, R6, R7, R8, R9: footprint (none) -> Resistor_THT:R_Axial_DIN0204_L3.6mm_D1.6mm_P2.54mm_Vertical
Changed lines of the file:
@@
 F 0 "Display1" H 7500 2431 50  0000 C CNN
 F 1 "74LS374" H 7500 2340 50  0000 C CNN
-F 2 "" H 7500 1450 50  0001 C CNN
+F 2 "Package_DIP:DIP-20_W7.62mm" H 7500 1450 50  0001 C CNN
 F 3 "http://www.ti.com/lit/gpn/sn74LS374" H 7500 1450 50  0001 C CNN
 	1    7500 1450
@@
 F 0 "Display2" H 7550 4481 50  0000 C CNN
 F 1 "74LS374" H 7550 4390 50  0000 C CNN
-F 2 "" H 7550 3500 50  0001 C CNN
+F 2 "Package_DIP:DIP-20_W7.62mm" H 7550 3500 50  0001 C CNN
 F 3 "http://www.ti.com/lit/gpn/sn74LS374" H 7550 3500 50  0001 C CNN
 	1    7550 3500
@@
 F 0 "Display3" H 7600 6481 50  0000 C CNN
 F 1 "74LS374" H 7600 6390 50  0000 C CNN
-F 2 "" H 7600 5500 50  0001 C CNN
+F 2 "Package_DIP:DIP-20_W7.62mm" H 7600 5500 50  0001 C CNN
 F 3 "http://www.ti.com/lit/gpn/sn74LS374" H 7600 5500 50  0001 C CNN
 	1    7600 5500
@@
 F 0 "Display_Decode2" H 3300 4231 50  0000 C CNN
 F 1 "PAL16L8" H 3300 4140 50  0000 C CNN
-F 2 "" H 3300 3350 50  0001 C CNN
+F 2 "Package_DIP:DIP-20_W7.62mm" H 3300 3350 50  0001 C CNN
 F 3 "" H 3300 3350 50  0001 C CNN
 	1    3300 3350
@@
 F 0 "Display_Decode1" H 3300 2381 50  0000 C CNN
 F 1 "PAL16L8" H 3300 2290 50  0000 C CNN
-F 2 "" H 3300 1500 50  0001 C CNN
+F 2 "Package_DIP:DIP-20_W7.62mm" H 3300 1500 50  0001 C CNN
 F 3 "" H 3300 1500 50  0001 C CNN
 	1    3300 1500
@@
 F 0 "R7" V 9845 4700 50  0000 C CNN
 F 1 "330" V 9936 4700 50  0000 C CNN
-F 2 "" H 10050 4700 50  0001 C CNN
+F 2 "Resistor_THT:R_Axial_DIN0204_L3.6mm_D1.6mm_P2.54mm_Vertical" H 10050 4700 50  0001 C CNN
 F 3 "~" H 10050 4700 50  0001 C CNN
 	1    10050 4700
@@
 F 0 "R13" V 10345 4950 50  0000 C CNN
 F 1 "330" V 10436 4950 50  0000 C CNN
-F 2 "" H 10550 4950 50  0001 C CNN
+F 2 "Resistor_THT:R_Axial_DIN0204_L3.6mm_D1.6mm_P2.54mm_Vertical" H 10550 4950 50  0001 C CNN
 F 3 "~" H 10550 4950 50  0001 C CNN
 	1    10550 4950
@@
 F 0 "R8" V 9845 5100 50  0000 C CNN
 F 1 "330" V 9936 5100 50  0000 C CNN
-F 2 "" H 10050 5100 50  0001 C CNN
+F 2 "Resistor_THT:R_Axial_DIN0204_L3.6mm_D1.6mm_P2.54mm_Vertical" H 10050 5100 50  0001 C CNN
 F 3 "~" H 10050 5100 50  0001 C CNN
 	1    10050 5100
@@
 F 0 "R10" V 10245 5350 50  0000 C CNN
 F 1 "330" V 10336 5350 50  0000 C CNN
-F 2 "" H 10450 5350 50  0001 C CNN
+F 2 "Resistor_THT:R_Axial_DIN0204_L3.6mm_D1.6mm_P2.54mm_Vertical" H 10450 5350 50  0001 C CNN
 F 3 "~" H 10450 5350 50  0001 C CNN
 	1    10450 5350
@@
 F 0 "R11" V 10245 5700 50  0000 C CNN
 F 1 "330" V 10336 5700 50  0000 C CNN
-F 2 "" H 10450 5700 50  0001 C CNN
+F 2 "Resistor_THT:R_Axial_DIN0204_L3.6mm_D1.6mm_P2.54mm_Vertical" H 10450 5700 50  0001 C CNN
 F 3 "~" H 10450 5700 50  0001 C CNN
 	1    10450 5700
@@
 F 0 "R6" V 9795 5500 50  0000 C CNN
 F 1 "330" V 9886 5500 50  0000 C CNN
-F 2 "" H 10000 5500 50  0001 C CNN
+F 2 "Resistor_THT:R_Axial_DIN0204_L3.6mm_D1.6mm_P2.54mm_Vertical" H 10000 5500 50  0001 C CNN
 F 3 "~" H 10000 5500 50  0001 C CNN
 	1    10000 5500
@@
 F 0 "R9" V 9845 5950 50  0000 C CNN
 F 1 "330" V 9936 5950 50  0000 C CNN
-F 2 "" H 10050 5950 50  0001 C CNN
+F 2 "Resistor_THT:R_Axial_DIN0204_L3.6mm_D1.6mm_P2.54mm_Vertical" H 10050 5950 50  0001 C CNN
 F 3 "~" H 10050 5950 50  0001 C CNN
 	1    10050 5950
@@
 F 0 "R12" V 10295 6150 50  0000 C CNN
 F 1 "330" V 10386 6150 50  0000 C CNN
-F 2 "" H 10500 6150 50  0001 C CNN
+F 2 "Resistor_THT:R_Axial_DIN0204_L3.6mm_D1.6mm_P2.54mm_Vertical" H 10500 6150 50  0001 C CNN
 F 3 "~" H 10500 6150 50  0001 C CNN
 	1    10500 6150
@@
 F 0 "D3" H 9343 4917 50  0000 C CNN
 F 1 "LED" H 9343 4826 50  0000 C CNN
-F 2 "" H 9350 4700 50  0001 C CNN
+F 2 "LED_THT:LED_D1.8mm_W1.8mm_H2.4mm_Horizontal_O1.27mm_Z4.9mm" H 9350 4700 50  0001 C CNN
 F 3 "~" H 9350 4700 50  0001 C CNN
 	1    9350 4700
@@
 F 0 "D5" H 9343 6167 50  0000 C CNN
 F 1 "LED" H 9343 6076 50  0000 C CNN
-F 2 "" H 9350 5950 50  0001 C CNN
+F 2 "LED_THT:LED_D1.8mm_W1.8mm_H2.4mm_Horizontal_O1.27mm_Z4.9mm" H 9350 5950 50  0001 C CNN
 F 3 "~" H 9350 5950 50  0001 C CNN
 	1    9350 5950
@@
 F 0 "D4" H 9343 5317 50  0000 C CNN
 F 1 "LED" H 9343 5226 50  0000 C CNN
-F 2 "" H 9350 5100 50  0001 C CNN
+F 2 "LED_THT:LED_D1.8mm_W1.8mm_H2.4mm_Horizontal_O1.27mm_Z4.9mm" H 9350 5100 50  0001 C CNN
 F 3 "~" H 9350 5100 50  0001 C CNN
 	1    9350 5100
@@
 F 0 "D8" H 9793 6367 50  0000 C CNN
 F 1 "LED" H 9793 6276 50  0000 C CNN
-F 2 "" H 9800 6150 50  0001 C CNN
+F 2 "LED_THT:LED_D1.8mm_W1.8mm_H2.4mm_Horizontal_O1.27mm_Z4.9mm" H 9800 6150 50  0001 C CNN
 F 3 "~" H 9800 6150 50  0001 C CNN
 	1    9800 6150
@@
 F 0 "D9" H 9843 5167 50  0000 C CNN
 F 1 "LED" H 9843 5076 50  0000 C CNN
-F 2 "" H 9850 4950 50  0001 C CNN
+F 2 "LED_THT:LED_D1.8mm_W1.8mm_H2.4mm_Horizontal_O1.27mm_Z4.9mm" H 9850 4950 50  0001 C CNN
 F 3 "~" H 9850 4950 50  0001 C CNN
 	1    9850 4950
@@
 F 0 "D7" H 9743 5917 50  0000 C CNN
 F 1 "LED" H 9743 5826 50  0000 C CNN
-F 2 "" H 9750 5700 50  0001 C CNN
+F 2 "LED_THT:LED_D1.8mm_W1.8mm_H2.4mm_Horizontal_O1.27mm_Z4.9mm" H 9750 5700 50  0001 C CNN
 F 3 "~" H 9750 5700 50  0001 C CNN
 	1    9750 5700
@@
 F 0 "D2" H 9293 5717 50  0000 C CNN
 F 1 "LED" H 9293 5626 50  0000 C CNN
-F 2 "" H 9300 5500 50  0001 C CNN
+F 2 "LED_THT:LED_D1.8mm_W1.8mm_H2.4mm_Horizontal_O1.27mm_Z4.9mm" H 9300 5500 50  0001 C CNN
 F 3 "~" H 9300 5500 50  0001 C CNN
 	1    9300 5500
@@
 F 0 "D6" H 9743 5567 50  0000 C CNN
 F 1 "LED" H 9743 5476 50  0000 C CNN
-F 2 "" H 9750 5350 50  0001 C CNN
+F 2 "LED_THT:LED_D1.8mm_W1.8mm_H2.4mm_Horizontal_O1.27mm_Z4.9mm" H 9750 5350 50  0001 C CNN
 F 3 "~" H 9750 5350 50  0001 C CNN
 	1    9750 5350
@@
 F 0 "R4" H 10070 1446 50  0000 L CNN
 F 1 "R" H 10070 1355 50  0000 L CNN
-F 2 "" V 9930 1400 50  0001 C CNN
+F 2 "Resistor_THT:R_Axial_DIN0204_L3.6mm_D1.6mm_P2.54mm_Vertical" V 9930 1400 50  0001 C CNN
 F 3 "~" H 10000 1400 50  0001 C CNN
 	1    10000 1400
@@
 F 0 "R5" H 10070 3446 50  0000 L CNN
 F 1 "R" H 10070 3355 50  0000 L CNN
-F 2 "" V 9930 3400 50  0001 C CNN
+F 2 "Resistor_THT:R_Axial_DIN0204_L3.6mm_D1.6mm_P2.54mm_Vertical" V 9930 3400 50  0001 C CNN
 F 3 "~" H 10000 3400 50  0001 C CNN
 	1    10000 3400
