File: Final/POWER(FINAL).sch (KiCad schematic (older format))
At the start: 26 parts

Commit message: New stuff
Parts:
- added J3: Conn_01x02_Female, symbol Connector:Conn_01x02_Female
- renumbered C25 to C10, C24 to C12, C10 to C13, C23 to C14, C9 to C15, C22 to C16, C8 to C17, C21 to C18, C7 to C19, C6 to C21, C19 to C22, C5 to C23, C18 to C24, C4 to C25, C17 to C26, C3 to C27, C16 to C28, C15 to C3, C28 to C4, C14 to C5, C27 to C6, C13 to C7, C26 to C8, C12 to C9
Connections:
- net VCC: now also J3.2 (Pin_2)
- net POWER: no longer names the net of C10.1, C11.1, C12.1, C13.1, C14.1, C15.1, C16.1, C17.1, C18.1, C19.1, C20.1, C21.1, C22.1, C23.1, C24.1, C25.1, C26.1, C27.1, C28.1, C3.1, C4.1, C5.1, C6.1, C7.1, C8.1, C9.1
- net POWER: now also J3.1 (Pin_1)
Changed lines of the file:
@@
 $EndDescr
 $Comp
-L Device:CP1_Small C13
+L Device:CP1_Small C7
 U 1 1 60786BAF
 P 2650 2750
-F 0 "C13" H 2741 2796 50  0000 L CNN
+F 0 "C7" H 2741 2796 50  0000 L CNN
 F 1 "CP1_Small" H 2741 2705 50  0000 L CNN
 F 2 "" H 2650 2750 50  0001 C CNN
@@
 $EndComp
 $Comp
-L Device:CP1_Small C12
+L Device:CP1_Small C9
 U 1 1 6078838C
 P 3250 2750
-F 0 "C12" H 3341 2796 50  0000 L CNN
+F 0 "C9" H 3341 2796 50  0000 L CNN
 F 1 "CP1_Small" H 3341 2705 50  0000 L CNN
 F 2 "" H 3250 2750 50  0001 C CNN
@@
 $EndComp
 $Comp
-L Device:CP1_Small C10
+L Device:CP1_Small C13
 U 1 1 607889E2
 P 4450 2750
-F 0 "C10" H 4541 2796 50  0000 L CNN
+F 0 "C13" H 4541 2796 50  0000 L CNN
 F 1 "CP1_Small" H 4541 2705 50  0000 L CNN
 F 2 "" H 4450 2750 50  0001 C CNN
@@
 $EndComp
 $Comp
-L Device:CP1_Small C9
+L Device:CP1_Small C15
 U 1 1 6078E574
 P 5050 2750
-F 0 "C9" H 5141 2796 50  0000 L CNN
+F 0 "C15" H 5141 2796 50  0000 L CNN
 F 1 "CP1_Small" H 5141 2705 50  0000 L CNN
 F 2 "" H 5050 2750 50  0001 C CNN
@@
 $EndComp
 $Comp
-L Device:CP1_Small C8
+L Device:CP1_Small C17
 U 1 1 6078E57A
 P 5650 2750
-F 0 "C8" H 5741 2796 50  0000 L CNN
+F 0 "C17" H 5741 2796 50  0000 L CNN
 F 1 "CP1_Small" H 5741 2705 50  0000 L CNN
 F 2 "" H 5650 2750 50  0001 C CNN
@@
 $EndComp
 $Comp
-L Device:CP1_Small C7
+L Device:CP1_Small C19
 U 1 1 6078E580
 P 6250 2750
-F 0 "C7" H 6341 2796 50  0000 L CNN
+F 0 "C19" H 6341 2796 50  0000 L CNN
 F 1 "CP1_Small" H 6341 2705 50  0000 L CNN
 F 2 "" H 6250 2750 50  0001 C CNN
@@
 $EndComp
 $Comp
-L Device:CP1_Small C6
+L Device:CP1_Small C21
 U 1 1 6078E586
 P 6850 2750
-F 0 "C6" H 6941 2796 50  0000 L CNN
+F 0 "C21" H 6941 2796 50  0000 L CNN
 F 1 "CP1_Small" H 6941 2705 50  0000 L CNN
 F 2 "" H 6850 2750 50  0001 C CNN
@@
 $EndComp
 $Comp
-L Device:CP1_Small C5
+L Device:CP1_Small C23
 U 1 1 6078F9B2
 P 7450 2750
-F 0 "C5" H 7541 2796 50  0000 L CNN
+F 0 "C23" H 7541 2796 50  0000 L CNN
 F 1 "CP1_Small" H 7541 2705 50  0000 L CNN
 F 2 "" H 7450 2750 50  0001 C CNN
@@
 $EndComp
 $Comp
-L Device:CP1_Small C4
+L Device:CP1_Small C25
 U 1 1 6078F9B8
 P 8050 2750
-F 0 "C4" H 8141 2796 50  0000 L CNN
+F 0 "C25" H 8141 2796 50  0000 L CNN
 F 1 "CP1_Small" H 8141 2705 50  0000 L CNN
 F 2 "" H 8050 2750 50  0001 C CNN
@@
 $EndComp
 $Comp
-L Device:CP1_Small C3
+L Device:CP1_Small C27
 U 1 1 6078F9BE
 P 8650 2750
-F 0 "C3" H 8741 2796 50  0000 L CNN
+F 0 "C27" H 8741 2796 50  0000 L CNN
 F 1 "CP1_Small" H 8741 2705 50  0000 L CNN
 F 2 "" H 8650 2750 50  0001 C CNN
@@
 $EndComp
 $Comp
-L Device:CP1_Small C15
+L Device:CP1_Small C3
 U 1 1 607906C5
 P 1450 2750
-F 0 "C15" H 1541 2796 50  0000 L CNN
+F 0 "C3" H 1541 2796 50  0000 L CNN
 F 1 "CP1_Small" H 1541 2705 50  0000 L CNN
 F 2 "" H 1450 2750 50  0001 C CNN
@@
 $EndComp
 $Comp
-L Device:CP1_Small C14
+L Device:CP1_Small C5
 U 1 1 607906CB
 P 2050 2750
-F 0 "C14" H 2141 2796 50  0000 L CNN
+F 0 "C5" H 2141 2796 50  0000 L CNN
 F 1 "CP1_Small" H 2141 2705 50  0000 L CNN
 F 2 "" H 2050 2750 50  0001 C CNN
@@
 $EndComp
 $Comp
-L Device:CP1_Small C26
+L Device:CP1_Small C8
 U 1 1 60797042
 P 2650 3450
-F 0 "C26" H 2741 3496 50  0000 L CNN
+F 0 "C8" H 2741 3496 50  0000 L CNN
 F 1 "CP1_Small" H 2741 3405 50  0000 L CNN
 F 2 "" H 2650 3450 50  0001 C CNN
@@
 $EndComp
 $Comp
-L Device:CP1_Small C25
+L Device:CP1_Small C10
 U 1 1 60797048
 P 3250 3450
-F 0 "C25" H 3341 3496 50  0000 L CNN
+F 0 "C10" H 3341 3496 50  0000 L CNN
 F 1 "CP1_Small" H 3341 3405 50  0000 L CNN
 F 2 "" H 3250 3450 50  0001 C CNN
@@
 $EndComp
 $Comp
-L Device:CP1_Small C24
+L Device:CP1_Small C12
 U 1 1 6079704E
 P 3850 3450
-F 0 "C24" H 3941 3496 50  0000 L CNN
+F 0 "C12" H 3941 3496 50  0000 L CNN
 F 1 "CP1_Small" H 3941 3405 50  0000 L CNN
 F 2 "" H 3850 3450 50  0001 C CNN
@@
 $EndComp
 $Comp
-L Device:CP1_Small C23
+L Device:CP1_Small C14
 U 1 1 60797054
 P 4450 3450
-F 0 "C23" H 4541 3496 50  0000 L CNN
+F 0 "C14" H 4541 3496 50  0000 L CNN
 F 1 "CP1_Small" H 4541 3405 50  0000 L CNN
 F 2 "" H 4450 3450 50  0001 C CNN
@@
 $EndComp
 $Comp
-L Device:CP1_Small C22
+L Device:CP1_Small C16
 U 1 1 6079705A
 P 5050 3450
-F 0 "C22" H 5141 3496 50  0000 L CNN
+F 0 "C16" H 5141 3496 50  0000 L CNN
 F 1 "CP1_Small" H 5141 3405 50  0000 L CNN
 F 2 "" H 5050 3450 50  0001 C CNN
@@
 $EndComp
 $Comp
-L Device:CP1_Small C21
+L Device:CP1_Small C18
 U 1 1 60797060
 P 5650 3450
-F 0 "C21" H 5741 3496 50  0000 L CNN
+F 0 "C18" H 5741 3496 50  0000 L CNN
 F 1 "CP1_Small" H 5741 3405 50  0000 L CNN
 F 2 "" H 5650 3450 50  0001 C CNN
@@
 $EndComp
 $Comp
-L Device:CP1_Small C19
+L Device:CP1_Small C22
 U 1 1 6079706C
 P 6850 3450
-F 0 "C19" H 6941 3496 50  0000 L CNN
+F 0 "C22" H 6941 3496 50  0000 L CNN
 F 1 "CP1_Small" H 6941 3405 50  0000 L CNN
 F 2 "" H 6850 3450 50  0001 C CNN
@@
 $EndComp
 $Comp
-L Device:CP1_Small C18
+L Device:CP1_Small C24
 U 1 1 60797072
 P 7450 3450
-F 0 "C18" H 7541 3496 50  0000 L CNN
+F 0 "C24" H 7541 3496 50  0000 L CNN
 F 1 "CP1_Small" H 7541 3405 50  0000 L CNN
 F 2 "" H 7450 3450 50  0001 C CNN
@@
 $EndComp
 $Comp
-L Device:CP1_Small C17
+L Device:CP1_Small C26
 U 1 1 60797078
 P 8050 3450
-F 0 "C17" H 8141 3496 50  0000 L CNN
+F 0 "C26" H 8141 3496 50  0000 L CNN
 F 1 "CP1_Small" H 8141 3405 50  0000 L CNN
 F 2 "" H 8050 3450 50  0001 C CNN
@@
 $EndComp
 $Comp
-L Device:CP1_Small C16
+L Device:CP1_Small C28
 U 1 1 6079707E
 P 8650 3450
-F 0 "C16" H 8741 3496 50  0000 L CNN
+F 0 "C28" H 8741 3496 50  0000 L CNN
 F 1 "CP1_Small" H 8741 3405 50  0000 L CNN
 F 2 "" H 8650 3450 50  0001 C CNN
@@
 $EndComp
 $Comp
-L Device:CP1_Small C28
+L Device:CP1_Small C4
 U 1 1 60797084
 P 1450 3450
-F 0 "C28" H 1541 3496 50  0000 L CNN
+F 0 "C4" H 1541 3496 50  0000 L CNN
 F 1 "CP1_Small" H 1541 3405 50  0000 L CNN
 F 2 "" H 1450 3450 50  0001 C CNN
@@
 $EndComp
 $Comp
-L Device:CP1_Small C27
+L Device:CP1_Small C6
 U 1 1 6079708A
 P 2050 3450
-F 0 "C27" H 2141 3496 50  0000 L CNN
+F 0 "C6" H 2141 3496 50  0000 L CNN
 F 1 "CP1_Small" H 2141 3405 50  0000 L CNN
 F 2 "" H 2050 3450 50  0001 C CNN
@@
 	8650 2850 8650 3050
 Wire Wire Line
-	8650 3050 9350 3050
+	8650 3050 9200 3050
 Connection ~ 8650 2850
 Wire Wire Line
@@
 Connection ~ 8650 2650
 $Comp
-L power:VCC #PWR0101
+L power:VCC #PWR068
 U 1 1 6079D049
 P 9350 3050
-F 0 "#PWR0101" H 9350 2900 50  0001 C CNN
+F 0 "#PWR068" H 9350 2900 50  0001 C CNN
 F 1 "VCC" V 9365 3178 50  0000 L CNN
 F 2 "" H 9350 3050 50  0001 C CNN
@@
 	0    1    1    0
 $EndComp
-Text HLabel 9350 2300 2    50   Output ~ 0
-POWER
+$Comp
+L Connector:Conn_01x02_Female J3
+U 1 1 60B637C0
+P 9550 2300
+F 0 "J3" H 9578 2276 50  0000 L CNN
+F 1 "Conn_01x02_Female" H 9578 2185 50  0000 L CNN
+F 2 "" H 9550 2300 50  0001 C CNN
+F 3 "~" H 9550 2300 50  0001 C CNN
+	1    9550 2300
+	1    0    0    -1
+$EndComp
+Wire Wire Line
+	9200 3050 9200 2400
+Wire Wire Line
+	9200 2400 9350 2400
+Connection ~ 9200 3050
+Wire Wire Line
+	9200 3050 9350 3050
 $EndSCHEMATC

Commit message: Final?
Parts:
- renumbered J3 to Power_1
Changed lines of the file:
@@
 $EndComp
 $Comp
-L Connector:Conn_01x02_Female J3
+L Connector:Conn_01x02_Female Power_1
 U 1 1 60B637C0
 P 9550 2300
-F 0 "J3" H 9578 2276 50  0000 L CNN
+F 0 "Power_1" H 9578 2276 50  0000 L CNN
 F 1 "Conn_01x02_Female" H 9578 2185 50  0000 L CNN
 F 2 "" H 9550 2300 50  0001 C CNN

Commit message: Hopefully the board is here
Parts:
- C10, C11, C12, C13, C14, C15, C16, C17, C18, C19, C20, C21, C22, C23, C24, C25, C26, C27, C28, C3, C4, C5, C6, C7, C8, C9: footprint (none) -> Capacitor_THT:CP_Axial_L10.0mm_D4.5mm_P15.00mm_Horizontal
- Power_1: footprint (none) -> Connector_PinHeader_1.00mm:PinHeader_1x02_P1.00mm_Horizontal
Changed lines of the file:
@@
 F 0 "C7" H 2741 2796 50  0000 L CNN
 F 1 "CP1_Small" H 2741 2705 50  0000 L CNN
-F 2 "" H 2650 2750 50  0001 C CNN
+F 2 "Capacitor_THT:CP_Axial_L10.0mm_D4.5mm_P15.00mm_Horizontal" H 2650 2750 50  0001 C CNN
 F 3 "~" H 2650 2750 50  0001 C CNN
 	1    2650 2750
@@
 F 0 "C9" H 3341 2796 50  0000 L CNN
 F 1 "CP1_Small" H 3341 2705 50  0000 L CNN
-F 2 "" H 3250 2750 50  0001 C CNN
+F 2 "Capacitor_THT:CP_Axial_L10.0mm_D4.5mm_P15.00mm_Horizontal" H 3250 2750 50  0001 C CNN
 F 3 "~" H 3250 2750 50  0001 C CNN
 	1    3250 2750
@@
 F 0 "C11" H 3941 2796 50  0000 L CNN
 F 1 "CP1_Small" H 3941 2705 50  0000 L CNN
-F 2 "" H 3850 2750 50  0001 C CNN
+F 2 "Capacitor_THT:CP_Axial_L10.0mm_D4.5mm_P15.00mm_Horizontal" H 3850 2750 50  0001 C CNN
 F 3 "~" H 3850 2750 50  0001 C CNN
 	1    3850 2750
@@
 F 0 "C13" H 4541 2796 50  0000 L CNN
 F 1 "CP1_Small" H 4541 2705 50  0000 L CNN
-F 2 "" H 4450 2750 50  0001 C CNN
+F 2 "Capacitor_THT:CP_Axial_L10.0mm_D4.5mm_P15.00mm_Horizontal" H 4450 2750 50  0001 C CNN
 F 3 "~" H 4450 2750 50  0001 C CNN
 	1    4450 2750
@@
 F 0 "C15" H 5141 2796 50  0000 L CNN
 F 1 "CP1_Small" H 5141 2705 50  0000 L CNN
-F 2 "" H 5050 2750 50  0001 C CNN
+F 2 "Capacitor_THT:CP_Axial_L10.0mm_D4.5mm_P15.00mm_Horizontal" H 5050 2750 50  0001 C CNN
 F 3 "~" H 5050 2750 50  0001 C CNN
 	1    5050 2750
@@
 F 0 "C17" H 5741 2796 50  0000 L CNN
 F 1 "CP1_Small" H 5741 2705 50  0000 L CNN
-F 2 "" H 5650 2750 50  0001 C CNN
+F 2 "Capacitor_THT:CP_Axial_L10.0mm_D4.5mm_P15.00mm_Horizontal" H 5650 2750 50  0001 C CNN
 F 3 "~" H 5650 2750 50  0001 C CNN
 	1    5650 2750
@@
 F 0 "C19" H 6341 2796 50  0000 L CNN
 F 1 "CP1_Small" H 6341 2705 50  0000 L CNN
-F 2 "" H 6250 2750 50  0001 C CNN
+F 2 "Capacitor_THT:CP_Axial_L10.0mm_D4.5mm_P15.00mm_Horizontal" H 6250 2750 50  0001 C CNN
 F 3 "~" H 6250 2750 50  0001 C CNN
 	1    6250 2750
@@
 F 0 "C21" H 6941 2796 50  0000 L CNN
 F 1 "CP1_Small" H 6941 2705 50  0000 L CNN
-F 2 "" H 6850 2750 50  0001 C CNN
+F 2 "Capacitor_THT:CP_Axial_L10.0mm_D4.5mm_P15.00mm_Horizontal" H 6850 2750 50  0001 C CNN
 F 3 "~" H 6850 2750 50  0001 C CNN
 	1    6850 2750
@@
 F 0 "C23" H 7541 2796 50  0000 L CNN
 F 1 "CP1_Small" H 7541 2705 50  0000 L CNN
-F 2 "" H 7450 2750 50  0001 C CNN
+F 2 "Capacitor_THT:CP_Axial_L10.0mm_D4.5mm_P15.00mm_Horizontal" H 7450 2750 50  0001 C CNN
 F 3 "~" H 7450 2750 50  0001 C CNN
 	1    7450 2750
@@
 F 0 "C25" H 8141 2796 50  0000 L CNN
 F 1 "CP1_Small" H 8141 2705 50  0000 L CNN
-F 2 "" H 8050 2750 50  0001 C CNN
+F 2 "Capacitor_THT:CP_Axial_L10.0mm_D4.5mm_P15.00mm_Horizontal" H 8050 2750 50  0001 C CNN
 F 3 "~" H 8050 2750 50  0001 C CNN
 	1    8050 2750
@@
 F 0 "C27" H 8741 2796 50  0000 L CNN
 F 1 "CP1_Small" H 8741 2705 50  0000 L CNN
-F 2 "" H 8650 2750 50  0001 C CNN
+F 2 "Capacitor_THT:CP_Axial_L10.0mm_D4.5mm_P15.00mm_Horizontal" H 8650 2750 50  0001 C CNN
 F 3 "~" H 8650 2750 50  0001 C CNN
 	1    8650 2750
@@
 F 0 "C3" H 1541 2796 50  0000 L CNN
 F 1 "CP1_Small" H 1541 2705 50  0000 L CNN
-F 2 "" H 1450 2750 50  0001 C CNN
+F 2 "Capacitor_THT:CP_Axial_L10.0mm_D4.5mm_P15.00mm_Horizontal" H 1450 2750 50  0001 C CNN
 F 3 "~" H 1450 2750 50  0001 C CNN
 	1    1450 2750
@@
 F 0 "C5" H 2141 2796 50  0000 L CNN
 F 1 "CP1_Small" H 2141 2705 50  0000 L CNN
-F 2 "" H 2050 2750 50  0001 C CNN
+F 2 "Capacitor_THT:CP_Axial_L10.0mm_D4.5mm_P15.00mm_Horizontal" H 2050 2750 50  0001 C CNN
 F 3 "~" H 2050 2750 50  0001 C CNN
 	1    2050 2750
@@
 F 0 "C8" H 2741 3496 50  0000 L CNN
 F 1 "CP1_Small" H 2741 3405 50  0000 L CNN
-F 2 "" H 2650 3450 50  0001 C CNN
+F 2 "Capacitor_THT:CP_Axial_L10.0mm_D4.5mm_P15.00mm_Horizontal" H 2650 3450 50  0001 C CNN
 F 3 "~" H 2650 3450 50  0001 C CNN
 	1    2650 3450
@@
 F 0 "C10" H 3341 3496 50  0000 L CNN
 F 1 "CP1_Small" H 3341 3405 50  0000 L CNN
-F 2 "" H 3250 3450 50  0001 C CNN
+F 2 "Capacitor_THT:CP_Axial_L10.0mm_D4.5mm_P15.00mm_Horizontal" H 3250 3450 50  0001 C CNN
 F 3 "~" H 3250 3450 50  0001 C CNN
 	1    3250 3450
@@
 F 0 "C12" H 3941 3496 50  0000 L CNN
 F 1 "CP1_Small" H 3941 3405 50  0000 L CNN
-F 2 "" H 3850 3450 50  0001 C CNN
+F 2 "Capacitor_THT:CP_Axial_L10.0mm_D4.5mm_P15.00mm_Horizontal" H 3850 3450 50  0001 C CNN
 F 3 "~" H 3850 3450 50  0001 C CNN
 	1    3850 3450
@@
 F 0 "C14" H 4541 3496 50  0000 L CNN
 F 1 "CP1_Small" H 4541 3405 50  0000 L CNN
-F 2 "" H 4450 3450 50  0001 C CNN
+F 2 "Capacitor_THT:CP_Axial_L10.0mm_D4.5mm_P15.00mm_Horizontal" H 4450 3450 50  0001 C CNN
 F 3 "~" H 4450 3450 50  0001 C CNN
 	1    4450 3450
@@
 F 0 "C16" H 5141 3496 50  0000 L CNN
 F 1 "CP1_Small" H 5141 3405 50  0000 L CNN
-F 2 "" H 5050 3450 50  0001 C CNN
+F 2 "Capacitor_THT:CP_Axial_L10.0mm_D4.5mm_P15.00mm_Horizontal" H 5050 3450 50  0001 C CNN
 F 3 "~" H 5050 3450 50  0001 C CNN
 	1    5050 3450
@@
 F 0 "C18" H 5741 3496 50  0000 L CNN
 F 1 "CP1_Small" H 5741 3405 50  0000 L CNN
-F 2 "" H 5650 3450 50  0001 C CNN
+F 2 "Capacitor_THT:CP_Axial_L10.0mm_D4.5mm_P15.00mm_Horizontal" H 5650 3450 50  0001 C CNN
 F 3 "~" H 5650 3450 50  0001 C CNN
 	1    5650 3450
@@
 F 0 "C20" H 6341 3496 50  0000 L CNN
 F 1 "CP1_Small" H 6341 3405 50  0000 L CNN
-F 2 "" H 6250 3450 50  0001 C CNN
+F 2 "Capacitor_THT:CP_Axial_L10.0mm_D4.5mm_P15.00mm_Horizontal" H 6250 3450 50  0001 C CNN
 F 3 "~" H 6250 3450 50  0001 C CNN
 	1    6250 3450
@@
 F 0 "C22" H 6941 3496 50  0000 L CNN
 F 1 "CP1_Small" H 6941 3405 50  0000 L CNN
-F 2 "" H 6850 3450 50  0001 C CNN
+F 2 "Capacitor_THT:CP_Axial_L10.0mm_D4.5mm_P15.00mm_Horizontal" H 6850 3450 50  0001 C CNN
 F 3 "~" H 6850 3450 50  0001 C CNN
 	1    6850 3450
@@
 F 0 "C24" H 7541 3496 50  0000 L CNN
 F 1 "CP1_Small" H 7541 3405 50  0000 L CNN
-F 2 "" H 7450 3450 50  0001 C CNN
+F 2 "Capacitor_THT:CP_Axial_L10.0mm_D4.5mm_P15.00mm_Horizontal" H 7450 3450 50  0001 C CNN
 F 3 "~" H 7450 3450 50  0001 C CNN
 	1    7450 3450
@@
 F 0 "C26" H 8141 3496 50  0000 L CNN
 F 1 "CP1_Small" H 8141 3405 50  0000 L CNN
-F 2 "" H 8050 3450 50  0001 C CNN
+F 2 "Capacitor_THT:CP_Axial_L10.0mm_D4.5mm_P15.00mm_Horizontal" H 8050 3450 50  0001 C CNN
 F 3 "~" H 8050 3450 50  0001 C CNN
 	1    8050 3450
@@
 F 0 "C28" H 8741 3496 50  0000 L CNN
 F 1 "CP1_Small" H 8741 3405 50  0000 L CNN
-F 2 "" H 8650 3450 50  0001 C CNN
+F 2 "Capacitor_THT:CP_Axial_L10.0mm_D4.5mm_P15.00mm_Horizontal" H 8650 3450 50  0001 C CNN
 F 3 "~" H 8650 3450 50  0001 C CNN
 	1    8650 3450
@@
 F 0 "C4" H 1541 3496 50  0000 L CNN
 F 1 "CP1_Small" H 1541 3405 50  0000 L CNN
-F 2 "" H 1450 3450 50  0001 C CNN
+F 2 "Capacitor_THT:CP_Axial_L10.0mm_D4.5mm_P15.00mm_Horizontal" H 1450 3450 50  0001 C CNN
 F 3 "~" H 1450 3450 50  0001 C CNN
 	1    1450 3450
@@
 F 0 "C6" H 2141 3496 50  0000 L CNN
 F 1 "CP1_Small" H 2141 3405 50  0000 L CNN
-F 2 "" H 2050 3450 50  0001 C CNN
+F 2 "Capacitor_THT:CP_Axial_L10.0mm_D4.5mm_P15.00mm_Horizontal" H 2050 3450 50  0001 C CNN
 F 3 "~" H 2050 3450 50  0001 C CNN
 	1    2050 3450
@@
 F 0 "Power_1" H 9578 2276 50  0000 L CNN
 F 1 "Conn_01x02_Female" H 9578 2185 50  0000 L CNN
-F 2 "" H 9550 2300 50  0001 C CNN
+F 2 "Connector_PinHeader_1.00mm:PinHeader_1x02_P1.00mm_Horizontal" H 9550 2300 50  0001 C CNN
 F 3 "~" H 9550 2300 50  0001 C CNN
 	1    9550 2300

Commit message: Added some final touches
Parts:
- Power_1: footprint Connector_PinHeader_1.00mm:PinHeader_1x02_P1.00mm_Horizontal -> Connector_PinHeader_1.00mm:PinHeader_1x02_P1.00mm_Vertical
Changed lines of the file:
@@
 encoding utf-8
 Sheet 14 16
-Title ""
+Title "Power"
 Date ""
 Rev ""
-Comp ""
-Comment1 ""
+Comp "UMBC 2021"
+Comment1 "Christian Lostoski"
 Comment2 ""
 Comment3 ""
@@
 F 0 "Power_1" H 9578 2276 50  0000 L CNN
 F 1 "Conn_01x02_Female" H 9578 2185 50  0000 L CNN
-F 2 "Connector_PinHeader_1.00mm:PinHeader_1x02_P1.00mm_Horizontal" H 9550 2300 50  0001 C CNN
+F 2 "Connector_PinHeader_1.00mm:PinHeader_1x02_P1.00mm_Vertical" H 9550 2300 50  0001 C CNN
 F 3 "~" H 9550 2300 50  0001 C CNN
 	1    9550 2300
